File: minimal_ad74416h/minimal_ad74416h.kicad_pcb (KiCad board)
At the start: 4 copper layers, 25.4 x 25.4 mm, 1 part, among them U1 AD74416HBCPZ-RL7

Commit message: minor changes
Routing:
- added copper zone on B.Cu, net (none)
- added copper zone on F.Cu, net (none)
- added copper zone on In1.Cu, net (none)
- added copper zone on In2.Cu, net (none)
Other:
- outline, holes or cut-outs redrawn
Changed lines of the file:
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@@
 		)
 	)
-	(gr_rect
-		(start 122.682 100.624087)
-		(end 148.082 126.024087)
+	(gr_arc
+		(start 147.066 100.624087)
+		(mid 147.784425 100.921666)
+		(end 148.082 101.640087)
 		(stroke
 			(width 0.05)
-			(type solid)
+			(type default)
 		)
-		(fill no)
 		(layer "Edge.Cuts")
 	)
+	(gr_line
+		(start 122.682 125.008087)
+		(end 122.682 101.640087)
+		(stroke
+			(width 0.05)
+			(type default)
+		)
+		(layer "Edge.Cuts")
+	)
+	(gr_line
+		(start 148.082 101.640087)
+		(end 148.082 125.008087)
+		(stroke
+			(width 0.05)
+			(type default)
+		)
+		(layer "Edge.Cuts")
+	)
+	(gr_arc
+		(start 123.698 126.024087)
+		(mid 122.979584 125.726507)
+		(end 122.682 125.008087)
+		(stroke
+			(width 0.05)
+			(type default)
+		)
+		(layer "Edge.Cuts")
+	)
+	(gr_arc
+		(start 122.682 101.640087)
+		(mid 122.97958 100.921667)
+		(end 123.698 100.624087)
+		(stroke
+			(width 0.05)
+			(type default)
+		)
+		(layer "Edge.Cuts")
+	)
+	(gr_line
+		(start 147.066 126.024087)
+		(end 123.698 126.024087)
+		(stroke
+			(width 0.05)
+			(type default)
+		)
+		(layer "Edge.Cuts")
+	)
+	(gr_arc
+		(start 148.082 125.008087)
+		(mid 147.78442 125.726507)
+		(end 147.066 126.024087)
+		(stroke
+			(width 0.05)
+			(type default)
+		)
+		(layer "Edge.Cuts")
+	)
+	(gr_line
+		(start 123.698 100.624087)
+		(end 147.066 100.624087)
+		(stroke
+			(width 0.05)
+			(type default)
+		)
+		(layer "Edge.Cuts")
+	)
+	(zone
+		(net 0)
+		(net_name "")
+		(layers "F.Cu" "B.Cu" "In1.Cu" "In2.Cu")
+		(hatch none 0.508)
+		(connect_pads
+			(clearance 0.508)
+		)
+		(min_thickness 0.508)
+		(filled_areas_thickness no)
+		(fill yes
+			(thermal_gap 0.508)
+			(thermal_bridge_width 0.508)
+			(smoothing fillet)
+			(radius 0.508)
+			(island_removal_mode 1)
+			(island_area_min 9.999999)
+		)
+		(polygon
+			(pts
+				(xy 122.682 100.6348) (xy 148.082 100.6348) (xy 148.082 126.0348) (xy 122.682 126.0348)
+			)
+		)
+	)
 	(embedded_fonts no)

Commit message: backup
Parts:
- added C1: 10 µF, capacitor_footprints:C_1206_3216Metric, F.Cu at (127.3, 113.4)
- added C10: 100 nF, capacitor_footprints:C_0402_1005Metric, F.Cu at (131.6, 107.1)
- added C11: 10 µF, capacitor_footprints:C_1210_250_3225Metric, F.Cu at (138.2, 120.9)
- added C12: 2.2 µF, capacitor_footprints:C_0805_2012Metric, F.Cu at (134.1, 104.7)
- added C13: 39 nF, capacitor_footprints:C_0603_1608Metric, F.Cu at (130.2, 119.5)
- added C2: 100 nF, capacitor_footprints:C_0402_1005Metric, F.Cu at (129.1, 113.4)
- added C3: 10 µF, capacitor_footprints:C_1206_3216Metric, F.Cu at (143.7, 113.4)
- added C4: 100 nF, capacitor_footprints:C_0402_1005Metric, F.Cu at (141.8, 113.4)
- added C5: 10 µF, capacitor_footprints:C_1206_3216Metric, F.Cu at (130.7, 123.9)
- added C6: 100 nF, capacitor_footprints:C_0402_1005Metric, F.Cu at (131.7, 122.0)
- added C7: 10 µF, capacitor_footprints:C_1206_3216Metric, F.Cu at (135.7, 123.9)
- added C8: 100 nF, capacitor_footprints:C_0402_1005Metric, F.Cu at (134.7, 122.0)
- added C9: 10 µF, capacitor_footprints:C_1206_3216Metric, F.Cu at (130.6, 105.2)
- added R1: 10 kΩ, resistor_footprints:R_0402_1005Metric, F.Cu at (138.0, 104.0)
- added R12: 10 kΩ, resistor_footprints:R_0402_1005Metric, F.Cu at (136.7, 103.9)
- added R2: 10 kΩ, resistor_footprints:R_0402_1005Metric, F.Cu at (139.3, 106.4)
Connections:
- U1 pad 17: unconnected-(U1-REFIO1-Pad17) -> Net-(U1-REFIO1)
- U1 pad 19: unconnected-(U1-AVCC-Pad19) -> Net-(U1-AVCC)
- U1 pad 20: unconnected-(U1-AGND-Pad20) -> GNDA
- U1 pad 21: unconnected-(U1-AVSS-Pad21) -> /AVSS
- U1 pad 26: unconnected-(U1-DO_VDD-Pad26) -> Net-(U1-DO_VDD)
- U1 pad 40: unconnected-(U1-AGND-Pad40) -> GNDA
- U1 pad 41: unconnected-(U1-AVDD_LO-Pad41) -> Net-(U1-AVDD_LO)
- U1 pad 49: unconnected-(U1-~{RESET}-Pad49) -> Net-(U1-~{RESET})
- U1 pad 54: unconnected-(U1-DGND-Pad54) -> GNDA
- U1 pad 55: unconnected-(U1-~{ALERT}-Pad55) -> Net-(U1-~{ALERT})
- U1 pad 56: unconnected-(U1-~{ADC_RDY}-Pad56) -> Net-(U1-~{ADC_RDY})
- U1 pad 61: unconnected-(U1-LDO1V8-Pad61) -> Net-(U1-LDO1V8)
- U1 pad 62: unconnected-(U1-DVCC-Pad62) -> Net-(U1-DVCC)
- U1 pad 8: unconnected-(U1-AVDD_HI-Pad8) -> Net-(U1-AVDD_HI)
- U1 pad 9: unconnected-(U1-AGND-Pad9) -> GNDA
- U1 pad PAD: (no net) -> /AVSS
Routing:
- net Net-(U1-AVCC): track 0.00 -> 6.21 mm
- net /AVSS: track 0.00 -> 6.21 mm
- net Net-(U1-AVDD_HI): track 0.00 -> 4.09 mm
- net Net-(U1-AVDD_LO): track 0.00 -> 4.09 mm
- net Net-(U1-DVCC): track 0.00 -> 3.88 mm
- net Net-(U1-LDO1V8): track 0.00 -> 3.70 mm
- net Net-(U1-DO_VDD): track 0.00 -> 3.11 mm
- net Net-(U1-~{ADC_RDY}): track 0.00 -> 2.18 mm, vias 0 -> 1
- net unconnected-(U1-GPIO_B-Pad58): track 0.00 -> 2.13 mm, vias 0 -> 1
- net unconnected-(U1-GPIO_D-Pad60): track 0.00 -> 2.08 mm, vias 0 -> 1
- net Net-(U1-REFIO1): track 0.00 -> 1.92 mm
- net Net-(U1-~{ALERT}): track 0.00 -> 1.70 mm, vias 0 -> 1
- net unconnected-(U1-GPIO_A-Pad57): track 0.00 -> 1.65 mm, vias 0 -> 1
- net unconnected-(U1-GPIO_C-Pad59): track 0.00 -> 1.60 mm, vias 0 -> 1
- net GNDA: vias 0 -> 1
- added copper zone on B.Cu, net GNDA
- added copper zone on F.Cu, net GNDA
- added copper zone on In1.Cu, net GNDA
- added copper zone on In2.Cu, net GNDA
- removed copper zone on B.Cu, net (none)
- removed copper zone on F.Cu, net (none)
- removed copper zone on In1.Cu, net (none)
- removed copper zone on In2.Cu, net (none)

Commit message: backup
Parts:
- added C14: 4.7 nF, capacitor_footprints:C_0603_1608Metric, F.Cu at (127.3, 106.0)
- added C15: 4.7 nF, capacitor_footprints:C_0603_1608Metric, F.Cu at (127.3, 120.8)
- added C16: 4.7 nF, capacitor_footprints:C_0603_1608Metric, F.Cu at (143.7, 120.8)
- added C17: 4.7 nF, capacitor_footprints:C_0603_1608Metric, F.Cu at (143.7, 106.0)
- added C18: 4.7 nF, capacitor_footprints:C_0603_1608Metric, F.Cu at (129.0, 107.6)
- added C19: 4.7 nF, capacitor_footprints:C_0603_1608Metric, F.Cu at (129.0, 119.2)
- added C20: 4.7 nF, capacitor_footprints:C_0603_1608Metric, F.Cu at (142.0, 119.1)
- added C21: 4.7 nF, capacitor_footprints:C_0603_1608Metric, F.Cu at (142.0, 107.5)
- added C22: 220 pF, capacitor_footprints:C_0603_1608Metric, F.Cu at (126.8, 110.9)
- added C23: 220 pF, capacitor_footprints:C_0603_1608Metric, F.Cu at (126.8, 116.0)
- added C24: 220 pF, capacitor_footprints:C_0603_1608Metric, F.Cu at (144.2, 116.0)
- added C25: 220 pF, capacitor_footprints:C_0603_1608Metric, F.Cu at (144.2, 110.9)
- added R10: 12 Ω, resistor_footprints:R_0805_2012Metric, F.Cu at (146.3, 109.1)
- added R11: 2 kΩ, resistor_footprints:R_0402_1005Metric, F.Cu at (144.2, 108.2)
- added R4: 12 Ω, resistor_footprints:R_0805_2012Metric, F.Cu at (124.6, 109.1)
- added R5: 2 kΩ, resistor_footprints:R_0402_1005Metric, F.Cu at (126.8, 108.2)
- added R6: 12 Ω, resistor_footprints:R_0805_2012Metric, F.Cu at (124.6, 117.7)
- added R7: 2 kΩ, resistor_footprints:R_0402_1005Metric, F.Cu at (126.8, 118.6)
- added R8: 12 Ω, resistor_footprints:R_0805_2012Metric, F.Cu at (146.3, 117.7)
- added R9: 2 kΩ, resistor_footprints:R_0402_1005Metric, F.Cu at (144.2, 118.6)
- moved C5 2.65 mm to (146.3, 113.4)
- moved C9 2.65 mm to (124.6, 113.4)
- moved R1 1.66 mm to (140.0, 104.9)
- moved C7 1.45 mm to (143.2, 113.4)
- moved C11 1.44 mm to (127.7, 113.4)
- moved R2 1.38 mm to (137.0, 104.9)
- moved R3 1.34 mm to (135.8, 104.9)
- moved C13 0.92 mm to (131.0, 120.0), turned to -90 degrees
- moved C1 0.53 mm to (134.1, 104.1)
- moved C2 0.53 mm to (130.6, 104.7)
- moved C3 0.53 mm to (131.6, 106.6)
- renumbered C12 to C1, C7 to C10, C2 to C11, C8 to C12, C9 to C2, C10 to C3, C11 to C4, C3 to C5, C5 to C6, C4 to C7, C6 to C8, C1 to C9, R2 to R1, R1 to R2, R12 to R3
Connections:
- U1 pad 1: unconnected-(U1-VIOUT_A-Pad1) -> /VIOUT_A
- U1 pad 10: unconnected-(U1-CCOMP_B-Pad10) -> /CCOMP_B
- U1 pad 12: unconnected-(U1-SENSELF_B-Pad12) -> /SENSELF_B
- U1 pad 13: unconnected-(U1-SENSEHF_B-Pad13) -> /SENSEHF_B
- U1 pad 16: unconnected-(U1-VIOUT_B-Pad16) -> /VIOUT_B
- U1 pad 33: unconnected-(U1-VIOUT_C-Pad33) -> /VIOUT_C
- U1 pad 36: unconnected-(U1-SENSEHF_C-Pad36) -> /SENSEHF_C
- U1 pad 37: unconnected-(U1-SENSELF_C-Pad37) -> /SENSELF_C
- U1 pad 39: unconnected-(U1-CCOMP_C-Pad39) -> /CCOMP_C
- U1 pad 4: unconnected-(U1-SENSEHF_A-Pad4) -> /SENSEHF_A
- U1 pad 42: unconnected-(U1-CCOMP_D-Pad42) -> /CCOMP_D
- U1 pad 44: unconnected-(U1-SENSELF_D-Pad44) -> /SENSELF_D
- U1 pad 45: unconnected-(U1-SENSEHF_D-Pad45) -> /SENSEHF_D
- U1 pad 48: unconnected-(U1-VIOUT_D-Pad48) -> /VIOUT_D
- U1 pad 5: unconnected-(U1-SENSELF_A-Pad5) -> /SENSELF_A
- U1 pad 7: unconnected-(U1-CCOMP_A-Pad7) -> /CCOMP_A
Routing:
- net unconnected-(U1-VSENSEN_A-Pad6): track 0.00 -> 9.19 mm
- net unconnected-(U1-VSENSEN_D-Pad43): track 0.00 -> 9.02 mm
- net unconnected-(U1-VSENSEN_B-Pad11): track 0.00 -> 8.75 mm
- net unconnected-(U1-VSENSEN_C-Pad38): track 0.00 -> 8.71 mm
- net /SENSELF_A: track 0.00 -> 7.33 mm
- net /SENSELF_B: track 0.00 -> 7.31 mm
- net /SENSELF_D: track 0.00 -> 7.29 mm
- net /SENSELF_C: track 0.00 -> 7.27 mm
- net /AVSS: track 6.21 -> 11.4 mm
- net /CCOMP_B: track 0.00 -> 4.70 mm
- net /CCOMP_A: track 0.00 -> 4.70 mm
- net /CCOMP_D: track 0.00 -> 4.66 mm
- net /CCOMP_C: track 0.00 -> 4.66 mm
- net /SENSEHF_D: track 0.00 -> 4.34 mm
- net /SENSEHF_B: track 0.00 -> 4.31 mm
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- added copper zone on F.Cu, net /VIOUT_A
- added copper zone on F.Cu, net /VIOUT_B
- added copper zone on F.Cu, net /VIOUT_C
- added copper zone on F.Cu, net /VIOUT_D
- added copper zone on F.Cu, net Net-(U1-AVDD_HI)
- added copper zone on F.Cu, net Net-(U1-AVDD_LO)
Other:
- board size 25.4 x 25.4 mm -> 30.5 x 25.4 mm

Commit message: backup
Parts:
- added C26: 4.7 nF, capacitor_footprints:C_0603_1608Metric, F.Cu at (123.4, 105.3)
- added C27: 4.7 nF, capacitor_footprints:C_0603_1608Metric, F.Cu at (123.4, 121.7)
- added C28: 4.7 nF, capacitor_footprints:C_0603_1608Metric, F.Cu at (147.6, 121.7)
- added C29: 4.7 nF, capacitor_footprints:C_0603_1608Metric, F.Cu at (147.6, 105.3)
- added D1: 36 V, diode_footprints:DO-214AA, F.Cu at (119.6, 105.9)
- added D2: 36 V, diode_footprints:DO-214AA, F.Cu at (119.6, 120.8)
- added D3: 36 V, diode_footprints:DO-214AA, F.Cu at (151.4, 121.8)
- added D4: 36 V, diode_footprints:DO-214AA, F.Cu at (151.4, 105.0)
- added D5: 36 V, diode_footprints:DO-214AA, F.Cu at (115.3, 109.4)
- added D6: 36 V, diode_footprints:DO-214AA, F.Cu at (115.3, 117.4)
- added D7: 36 V, diode_footprints:DO-214AA, F.Cu at (155.6, 117.4)
- added D8: 36 V, diode_footprints:DO-214AA, F.Cu at (155.6, 109.4)
- added R12: 2 kΩ, resistor_footprints:R_0603_1608Metric, F.Cu at (127.4, 108.4)
- added R13: 2 kΩ, resistor_footprints:R_0603_1608Metric, F.Cu at (127.4, 118.4)
- added R14: 2 kΩ, resistor_footprints:R_0603_1608Metric, F.Cu at (143.6, 118.4)
- added R15: 2 kΩ, resistor_footprints:R_0603_1608Metric, F.Cu at (143.6, 108.4)
- added R16: 2 kΩ, resistor_footprints:R_0402_1005Metric, F.Cu at (129.6, 107.9)
- added R17: 2 kΩ, resistor_footprints:R_0402_1005Metric, F.Cu at (129.6, 118.9)
- added R18: 2 kΩ, resistor_footprints:R_0402_1005Metric, F.Cu at (141.3, 118.9)
- added R19: 2 kΩ, resistor_footprints:R_0402_1005Metric, F.Cu at (141.3, 107.7)
- moved R11 3.94 mm to (147.8, 106.7)
- moved R5 3.94 mm to (123.1, 106.7)
- moved R9 3.94 mm to (147.8, 120.1)
- moved R7 3.94 mm to (123.1, 120.1)
- moved C20 1.96 mm to (142.8, 120.9)
- moved C18 1.87 mm to (128.2, 105.9)
- moved C19 1.86 mm to (128.2, 120.9)
- moved C21 1.80 mm to (142.8, 105.9)
- moved C2 1.63 mm to (131.7, 103.5), turned to 90 degrees
- moved R4 1.32 mm to (123.5, 108.4), turned to 180 degrees
- moved R10 1.32 mm to (147.4, 108.4), turned to 0 degrees
- moved R6 1.30 mm to (123.5, 118.4), turned to 180 degrees
- moved R8 1.30 mm to (147.4, 118.4), turned to 0 degrees
- moved C17 0.80 mm to (144.5, 105.9)
- moved C16 0.80 mm to (144.5, 120.9)
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Connections:
- net Net-(R10-Pad2) renamed /I/OP_D
- net Net-(R4-Pad2) renamed /I/OP_A
- net Net-(R6-Pad2) renamed /I/OP_B
- net Net-(R8-Pad2) renamed /I/OP_C
- U1 pad 11: unconnected-(U1-VSENSEN_B-Pad11) -> /VSENSEN_B
- U1 pad 14: unconnected-(U1-VSENSEP_B-Pad14) -> /VSENSEP_B
- U1 pad 3: unconnected-(U1-VSENSEP_A-Pad3) -> /VSENSEP_A
- U1 pad 35: unconnected-(U1-VSENSEP_C-Pad35) -> /VSENSEP_C
- U1 pad 38: unconnected-(U1-VSENSEN_C-Pad38) -> /VSENSEN_C
- U1 pad 43: unconnected-(U1-VSENSEN_D-Pad43) -> /VSENSEN_D
- U1 pad 46: unconnected-(U1-VSENSEP_D-Pad46) -> /VSENSEP_D
- U1 pad 6: unconnected-(U1-VSENSEN_A-Pad6) -> /VSENSEN_A
Routing:
- net /VSENSEN_A: track 0.00 -> 16.6 mm
- net /VSENSEN_B: track 0.00 -> 16.6 mm
- net /VSENSEN_C: track 0.00 -> 16.6 mm
- net /VSENSEN_D: track 0.00 -> 16.6 mm
- net unconnected-(U1-VSENSEN_A-Pad6): track 9.19 -> 0.00 mm
- net unconnected-(U1-VSENSEN_D-Pad43): track 9.02 -> 0.00 mm
- net unconnected-(U1-VSENSEN_B-Pad11): track 8.75 -> 0.00 mm
- net unconnected-(U1-VSENSEN_C-Pad38): track 8.71 -> 0.00 mm
- net /VSENSEP_D: track 0.00 -> 3.43 mm
- net /SENSELF_C: track 7.27 -> 10.5 mm
- net /SENSELF_D: track 7.29 -> 10.6 mm
- net /SENSELF_A: track 7.33 -> 10.6 mm
- net /VSENSEP_A: track 0.00 -> 3.22 mm
- net /VSENSEP_C: track 0.00 -> 3.19 mm
- net /VSENSEP_B: track 0.00 -> 3.19 mm
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- added copper zone on F.Cu, net /I/OP_A
- added copper zone on F.Cu, net /I/OP_B
- added copper zone on F.Cu, net /I/OP_C
- added copper zone on F.Cu, net /I/OP_D
Other:
- board size 30.5 x 25.4 mm -> 45.7 x 25.4 mm

Commit message: backup
Parts:
- added J5: MTMM-101-04-L-D-196, connector_footprints:MTMM-101-04-L-D-196, F.Cu at (128.3, 106.6)
- added J6: MTMM-101-04-L-D-196, connector_footprints:MTMM-101-04-L-D-196, F.Cu at (128.3, 120.2)
- added J7: MTMM-101-04-L-D-196, connector_footprints:MTMM-101-04-L-D-196, F.Cu at (142.7, 120.2)
- added J8: MTMM-101-04-L-D-196, connector_footprints:MTMM-101-04-L-D-196, F.Cu at (142.7, 106.6)
- added Q1: -100.0 V, transistor_footprints:PowerPAK 1212-8, F.Cu at (118.4, 102.0)
- added Q2: -100.0 V, transistor_footprints:PowerPAK 1212-8, F.Cu at (118.4, 124.9)
- added Q3: -100.0 V, transistor_footprints:PowerPAK 1212-8, F.Cu at (152.6, 124.9)
- added Q4: -100.0 V, transistor_footprints:PowerPAK 1212-8, F.Cu at (152.6, 102.0)
- added Q5: -100.0 V, transistor_footprints:PowerPAK 1212-8, F.Cu at (114.2, 101.1)
- added Q6: -100.0 V, transistor_footprints:PowerPAK 1212-8, F.Cu at (114.2, 125.8)
- added Q7: -100.0 V, transistor_footprints:PowerPAK 1212-8, F.Cu at (156.8, 125.8)
- added Q8: -100.0 V, transistor_footprints:PowerPAK 1212-8, F.Cu at (156.8, 101.1)
- added R20: 100 kΩ, resistor_footprints:R_0402_1005Metric, F.Cu at (117.9, 111.4)
- added R21: 100 kΩ, resistor_footprints:R_0402_1005Metric, F.Cu at (117.9, 115.4)
- added R22: 100 kΩ, resistor_footprints:R_0402_1005Metric, F.Cu at (153.0, 115.4)
- added R23: 100 kΩ, resistor_footprints:R_0402_1005Metric, F.Cu at (153.0, 111.4)
- added R24: 10 kΩ, resistor_footprints:R_0402_1005Metric, F.Cu at (128.3, 109.0)
- added R25: 10 kΩ, resistor_footprints:R_0402_1005Metric, F.Cu at (128.3, 117.9)
- added R26: 10 kΩ, resistor_footprints:R_0402_1005Metric, F.Cu at (142.7, 117.9)
- added R27: 10 kΩ, resistor_footprints:R_0402_1005Metric, F.Cu at (142.7, 109.0)
- moved D4 6.49 mm to (157.6, 106.6), turned to 180 degrees
- moved D3 6.46 mm to (157.6, 120.3), turned to 180 degrees
- moved D1 6.31 mm to (113.3, 106.6), turned to 0 degrees
- moved D2 6.30 mm to (113.3, 120.3), turned to 0 degrees
- moved C16 3.30 mm to (147.8, 120.9)
- moved C17 3.30 mm to (147.8, 105.9)
- moved C20 3.30 mm to (146.0, 120.9)
- moved C21 3.30 mm to (146.0, 105.9)
- moved R14 3.30 mm to (146.9, 118.4)
- moved R15 3.30 mm to (146.9, 108.4)
- moved C11 3.01 mm to (124.1, 113.4)
- moved C14 3.01 mm to (123.5, 105.9)
- moved C15 3.01 mm to (123.5, 120.9)
- moved C26 3.01 mm to (120.4, 105.3)
- moved C27 3.01 mm to (120.4, 121.7)
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Connections:
- net /VSENSEN_A renamed /ISN_A
- net /VSENSEN_B renamed /ISN_B
- net /VSENSEN_C renamed /ISN_C
- net /VSENSEN_D renamed /ISN_D
- R16 pad 2: unconnected-(R16-Pad2) -> /ISP_A
- R17 pad 2: unconnected-(R17-Pad2) -> /ISP_B
- R18 pad 2: unconnected-(R18-Pad2) -> /ISP_C
- R19 pad 2: unconnected-(R19-Pad2) -> /ISP_D
- U1 pad 15: unconnected-(U1-LKG_COMP_B-Pad15) -> /LKG_COMP_B
- U1 pad 2: unconnected-(U1-LKG_COMP_A-Pad2) -> /LKG_COMP_A
- U1 pad 34: unconnected-(U1-LKG_COMP_C-Pad34) -> /LKG_COMP_C
- U1 pad 47: unconnected-(U1-LKG_COMP_D-Pad47) -> /LKG_COMP_D
Routing:
- net /ISP_B: track 0.00 -> 3.65 mm
- net /ISP_D: track 0.00 -> 3.65 mm
- net /ISP_C: track 0.00 -> 3.65 mm
- net /ISP_A: track 0.00 -> 3.65 mm
- net /SENSELF_B: track 10.2 -> 13.2 mm
- net /SENSELF_A: track 10.6 -> 13.6 mm
- net /SENSEHF_A: track 6.35 -> 9.36 mm
- net /SENSEHF_B: track 6.35 -> 9.36 mm
- net /CCOMP_B: track 5.28 -> 8.29 mm
- net /CCOMP_A: track 5.28 -> 8.29 mm
- net /CCOMP_C: track 5.24 -> 8.24 mm
- net /CCOMP_D: track 5.24 -> 8.24 mm
- net /SENSELF_D: track 10.6 -> 13.5 mm
- net /SENSEHF_C: track 6.36 -> 8.96 mm
- net /SENSELF_C: track 10.5 -> 13.1 mm
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Other:
- board size 45.7 x 25.4 mm -> 53.3 x 30.5 mm

Commit message: backup
Parts:
- added R28: 0 Ω, resistor_footprints:R_0402_1005Metric, F.Cu at (125.7, 99.6)
- added R29: 0 Ω, resistor_footprints:R_0402_1005Metric, F.Cu at (125.7, 124.3)
- added R30: 0 Ω, resistor_footprints:R_0402_1005Metric, F.Cu at (145.2, 127.3)
- added R31: 0 Ω, resistor_footprints:R_0402_1005Metric, F.Cu at (145.2, 102.6)
- added R32: 0.15 Ω, resistor_footprints:R_1206_3216Metric, F.Cu at (127.1, 101.5)
- added R33: 0.15 Ω, resistor_footprints:R_1206_3216Metric, F.Cu at (127.1, 126.1)
- added R34: 0.15 Ω, resistor_footprints:R_1206_3216Metric, F.Cu at (143.8, 125.5)
- added R35: 0.15 Ω, resistor_footprints:R_1206_3216Metric, F.Cu at (143.8, 100.8)
- moved Q7 8.41 mm to (148.4, 125.8), turned to 0 degrees
- moved Q8 8.41 mm to (148.4, 101.1), turned to 0 degrees
- moved Q5 8.41 mm to (122.6, 101.1), turned to 180 degrees
- moved Q6 8.41 mm to (122.6, 125.8), turned to 180 degrees
- moved C6 1.37 mm to (130.8, 123.1)
- moved C14 0.29 mm to (123.2, 105.9)
- moved C15 0.29 mm to (123.2, 120.9)
- moved C18 0.29 mm to (124.9, 105.9)
- moved C19 0.29 mm to (124.9, 120.9)
- moved R12 0.29 mm to (124.1, 108.4)
- moved R13 0.29 mm to (124.1, 118.4)
Connections:
- Q5 pad 1: unconnected-(Q5-S-Pad1) -> /DO_SRC_SNS_A
- Q5 pad 2: unconnected-(Q5-S-Pad2) -> /DO_SRC_SNS_A
- Q5 pad 3: unconnected-(Q5-S-Pad3) -> /DO_SRC_SNS_A
- Q5 pad 4: unconnected-(Q5-G-Pad4) -> Net-(Q5-G)
- Q6 pad 1: unconnected-(Q6-S-Pad1) -> /DO_SRC_SNS_B
- Q6 pad 2: unconnected-(Q6-S-Pad2) -> /DO_SRC_SNS_B
- Q6 pad 3: unconnected-(Q6-S-Pad3) -> /DO_SRC_SNS_B
- Q6 pad 4: unconnected-(Q6-G-Pad4) -> Net-(Q6-G)
- Q7 pad 1: unconnected-(Q7-S-Pad1) -> /DO_SRC_SNS_C
- Q7 pad 2: unconnected-(Q7-S-Pad2) -> /DO_SRC_SNS_C
- Q7 pad 3: unconnected-(Q7-S-Pad3) -> /DO_SRC_SNS_C
- Q7 pad 4: unconnected-(Q7-G-Pad4) -> Net-(Q7-G)
- Q8 pad 1: unconnected-(Q8-S-Pad1) -> /DO_SRC_SNS_D
- Q8 pad 2: unconnected-(Q8-S-Pad2) -> /DO_SRC_SNS_D
- Q8 pad 3: unconnected-(Q8-S-Pad3) -> /DO_SRC_SNS_D
- Q8 pad 4: unconnected-(Q8-G-Pad4) -> Net-(Q8-G)
- U1 pad 22: unconnected-(U1-DO_SRC_GATE_A-Pad22) -> /DO_SRC_GATE_A
- U1 pad 23: unconnected-(U1-DO_SRC_SNS_A-Pad23) -> /DO_SRC_SNS_A
- U1 pad 24: unconnected-(U1-DO_SRC_GATE_B-Pad24) -> /DO_SRC_GATE_B
- U1 pad 25: unconnected-(U1-DO_SRC_SNS_B-Pad25) -> /DO_SRC_SNS_B
- U1 pad 27: unconnected-(U1-DO_SRC_SNS_C-Pad27) -> /DO_SRC_SNS_C
- U1 pad 28: unconnected-(U1-DO_SRC_GATE_C-Pad28) -> /DO_SRC_GATE_C
- U1 pad 29: unconnected-(U1-DO_SRC_SNS_D-Pad29) -> /DO_SRC_SNS_D
- U1 pad 30: unconnected-(U1-DO_SRC_GATE_D-Pad30) -> /DO_SRC_GATE_D
Routing:
- net /SENSEHF_A: track 9.36 -> 7.26 mm
- net Net-(Q7-G): track 0.00 -> 1.44 mm
- net Net-(Q5-G): track 0.00 -> 1.44 mm
- net Net-(Q8-G): track 0.00 -> 1.44 mm
- net Net-(Q6-G): track 0.00 -> 1.44 mm
- net Net-(U1-AVCC): track 6.53 -> 5.37 mm

Commit message: backup
Parts:
- C13: footprint capacitor_footprints:C_0603_1608Metric -> capacitor_footprints:C_0402_1005Metric
- moved C4 4.15 mm to (138.8, 124.9), turned to 90 degrees
- moved C11 2.54 mm to (126.7, 113.4)
- moved C7 2.54 mm to (144.3, 113.4)
- moved C6 1.89 mm to (131.4, 124.9), turned to -90 degrees
- moved C13 1.35 mm to (130.5, 119.2), turned to 180 degrees
- moved C8 1.24 mm to (132.3, 121.3)
- moved R11 1.08 mm to (150.2, 107.6)
- moved R5 1.08 mm to (120.7, 107.6)
- moved R9 1.04 mm to (150.2, 119.3)
- moved R7 1.04 mm to (120.7, 119.3)
- moved C10 1.04 mm to (135.3, 124.9), turned to -90 degrees
- moved J6 0.97 mm to (128.3, 121.2), turned to -90 degrees
- moved J7 0.97 mm to (142.7, 121.2), turned to 90 degrees
- moved R25 0.97 mm to (128.3, 118.8), turned to 0 degrees
- moved R26 0.97 mm to (142.7, 118.8), turned to 180 degrees
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Routing:
- net /DO_SRC_GATE_A: track 0.00 -> 30.0 mm, vias 0 -> 2
- net /DO_SRC_GATE_D: track 0.00 -> 27.1 mm, vias 0 -> 2
- net /DO_SRC_SNS_D: track 0.00 -> 26.6 mm, vias 0 -> 2
- net /DO_SRC_SNS_A: track 0.00 -> 25.2 mm, vias 0 -> 2
- net /DO_SRC_SNS_B: track 0.00 -> 15.0 mm, vias 0 -> 2
- net /LKG_COMP_B: track 1.05 -> 15.0 mm, vias 1 -> 2
- net /LKG_COMP_C: track 1.05 -> 15.0 mm, vias 1 -> 2
- net /LKG_COMP_D: track 1.05 -> 14.9 mm, vias 1 -> 2
- net /LKG_COMP_A: track 1.05 -> 14.9 mm, vias 1 -> 2
- net /DO_SRC_GATE_B: track 0.00 -> 13.5 mm, vias 0 -> 2
- net /DO_SRC_GATE_C: track 0.00 -> 13.3 mm, vias 0 -> 2
- net /AVSS: track 12.1 -> 0.00 mm
- net /DO_SRC_SNS_C: track 0.00 -> 11.4 mm, vias 0 -> 2
- net GNDA: track 0.00 -> 11.2 mm, vias 8 -> 20
- net /VIOUT_B: track 1.16 -> 9.27 mm
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- added copper zone on F.Cu, net /AVSS
- added copper zone on F.Cu, net /DO_SRC_SNS_A
- added copper zone on F.Cu, net /DO_SRC_SNS_B
- added copper zone on F.Cu, net /DO_SRC_SNS_C
- added copper zone on F.Cu, net /DO_SRC_SNS_D
- added copper zone on F.Cu, net /LKG_COMP_A
- added copper zone on F.Cu, net /LKG_COMP_B
- added copper zone on F.Cu, net /LKG_COMP_C
- added copper zone on F.Cu, net /LKG_COMP_D
- added copper zone on F.Cu, net Net-(U1-AVCC)
- added copper zone on F.Cu, net Net-(U1-DO_VDD)
Other:
- board size 53.3 x 30.5 mm -> 53.4 x 35.6 mm
