File: minimal_ad74416h/minimal_ad74416h.kicad_pcb (KiCad board)
At the start: 4 copper layers, 53.4 x 35.6 mm, 85 parts, among them J5 MTMM-101-04-L-D-196, J6 MTMM-101-04-L-D-196, J7 MTMM-101-04-L-D-196, J8 MTMM-101-04-L-D-196, Q1 -100.0 V, Q2 -100.0 V, Q3 -100.0 V, Q4 -100.0 V, Q5 -100.0 V, Q6 -100.0 V, Q7 -100.0 V, Q8 -100.0 V, U1 AD74416HBCPZ-RL7

Commit message: backup
Parts:
- added R36: 10 kΩ, resistor_footprints:R_0402_1005Metric, F.Cu at (115.3, 101.6)
- added R37: 10 kΩ, resistor_footprints:R_0402_1005Metric, F.Cu at (115.3, 126.3)
- added R38: 10 kΩ, resistor_footprints:R_0402_1005Metric, F.Cu at (155.6, 125.3)
- added R39: 10 kΩ, resistor_footprints:R_0402_1005Metric, F.Cu at (155.6, 100.7)
- moved C13 0.62 mm to (131.1, 119.2)
- moved J5 0.49 mm to (128.3, 105.2), turned to 180 degrees
- moved J8 0.49 mm to (142.7, 105.2), turned to 180 degrees
- moved J6 0.49 mm to (128.3, 121.6), turned to 0 degrees
- moved J7 0.49 mm to (142.7, 121.6), turned to 0 degrees
- moved C4 0.13 mm to (138.7, 124.9)
Connections:
- C4 pad 2: Net-(U1-DO_VDD) -> /DO_VDD
- Q1 pad 4: unconnected-(Q1-G-Pad4) -> Net-(Q1-G)
- Q2 pad 4: unconnected-(Q2-G-Pad4) -> Net-(Q2-G)
- Q3 pad 4: unconnected-(Q3-G-Pad4) -> Net-(Q3-G)
- Q4 pad 4: unconnected-(Q4-G-Pad4) -> Net-(Q4-G)
- R32 pad 1: unconnected-(R32-Pad1) -> /DO_VDD
- R33 pad 1: unconnected-(R33-Pad1) -> /DO_VDD
- R34 pad 1: unconnected-(R34-Pad1) -> /DO_VDD
- R35 pad 1: unconnected-(R35-Pad1) -> /DO_VDD
- U1 pad 26: Net-(U1-DO_VDD) -> /DO_VDD
Routing:
- net /DO_SRC_GATE_B: track 13.5 -> 22.1 mm
- net /DO_SRC_SNS_D: track 26.6 -> 23.3 mm
- net /DO_SRC_GATE_D: track 27.1 -> 24.2 mm
- net /DO_SRC_SNS_A: track 25.2 -> 22.8 mm
- net /VIOUT_B: track 9.27 -> 11.1 mm
- net /VIOUT_A: track 9.27 -> 11.1 mm
- net /VIOUT_D: track 9.27 -> 11.1 mm
- net /VIOUT_C: track 9.27 -> 11.0 mm
- net Net-(Q4-G): track 0.00 -> 1.54 mm
- net Net-(Q3-G): track 0.00 -> 1.54 mm
- net Net-(Q2-G): track 0.00 -> 1.54 mm
- net Net-(Q1-G): track 0.00 -> 1.54 mm
- net /LKG_COMP_B: track 15.0 -> 13.6 mm
- net /DO_SRC_GATE_A: track 30.0 -> 28.7 mm
- net /LKG_COMP_C: track 15.0 -> 13.6 mm
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- added copper zone on F.Cu, net /DO_VDD
- added copper zone on In1.Cu, net /DO_VDD
- removed copper zone on F.Cu, net Net-(U1-DO_VDD)
