File: minimal_ad74416h/minimal_ad74416h.kicad_pcb (KiCad board)
At the start: 4 copper layers, 53.4 x 35.6 mm, 89 parts, among them J5 MTMM-101-04-L-D-196, J6 MTMM-101-04-L-D-196, J7 MTMM-101-04-L-D-196, J8 MTMM-101-04-L-D-196, Q1 -100.0 V, Q2 -100.0 V, Q3 -100.0 V, Q4 -100.0 V, Q5 -100.0 V, Q6 -100.0 V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

Commit message: backup
Parts:
- added D10: 5.0 V, diode_footprints:SOD323, F.Cu at (114.2, 125.3)
- added D11: 5.0 V, diode_footprints:SOD323, F.Cu at (156.7, 126.3)
- added D12: 5.0 V, diode_footprints:SOD323, F.Cu at (156.7, 101.6)
- added D13: 100.0 V, diode_footprints:DO-219AD, F.Cu at (116.6, 97.4)
- added D14: 100.0 V, diode_footprints:DO-219AD, F.Cu at (116.6, 129.5)
- added D15: 100.0 V, diode_footprints:DO-219AD, F.Cu at (154.3, 129.5)
- added D16: 100.0 V, diode_footprints:DO-219AD, F.Cu at (154.3, 97.4)
- added D9: 5.0 V, diode_footprints:SOD323, F.Cu at (114.2, 100.6)
- added Q10: 50 V, transistor_footprints:SOT23-3, F.Cu at (120.4, 129.5)
- added Q11: 50 V, transistor_footprints:SOT23-3, F.Cu at (150.5, 129.5)
- added Q12: 50 V, transistor_footprints:SOT23-3, F.Cu at (150.5, 97.4)
- added Q9: 50 V, transistor_footprints:SOT23-3, F.Cu at (120.4, 97.4)
- added R40: 100 kΩ, resistor_footprints:R_0402_1005Metric, F.Cu at (123.2, 98.2)
- added R41: 100 kΩ, resistor_footprints:R_0402_1005Metric, F.Cu at (123.2, 130.2)
- added R42: 100 kΩ, resistor_footprints:R_0402_1005Metric, F.Cu at (147.8, 128.8)
- added R43: 100 kΩ, resistor_footprints:R_0402_1005Metric, F.Cu at (147.8, 96.7)
- added R44: 3.9 kΩ, resistor_footprints:R_0402_1005Metric, F.Cu at (123.2, 96.7)
- added R45: 3.9 kΩ, resistor_footprints:R_0402_1005Metric, F.Cu at (123.2, 128.8)
- added R46: 3.9 kΩ, resistor_footprints:R_0402_1005Metric, F.Cu at (147.8, 130.2)
- added R47: 3.9 kΩ, resistor_footprints:R_0402_1005Metric, F.Cu at (147.8, 98.2)
- moved R20 0.76 mm to (118.7, 111.4)
- moved R21 0.76 mm to (118.7, 115.4)
- moved D1 0.75 mm to (114.1, 106.6)
- moved D2 0.75 mm to (114.1, 120.3)
- moved D5 0.75 mm to (114.1, 110.9)
- moved D6 0.75 mm to (114.1, 116.0)
- moved R36 0.69 mm to (114.9, 102.1), turned to 180 degrees
- moved R37 0.69 mm to (114.9, 126.8), turned to 180 degrees
- moved R38 0.69 mm to (156.1, 124.8), turned to 0 degrees
- moved R39 0.69 mm to (156.1, 100.1), turned to 0 degrees
- moved D4 0.12 mm to (156.9, 106.6)
- moved D8 0.12 mm to (156.9, 110.9)
- moved R22 0.12 mm to (152.3, 115.4)
- moved R23 0.12 mm to (152.3, 111.4)
Routing:
- net Net-(Q3-G): track 1.54 -> 6.19 mm
- net Net-(Q1-G): track 1.54 -> 6.19 mm
- net Net-(Q2-G): track 1.54 -> 5.69 mm
- net Net-(Q4-G): track 1.54 -> 5.68 mm
- net Net-(Q12-D): track 0.00 -> 2.10 mm
- net Net-(Q11-D): track 0.00 -> 2.10 mm
- net Net-(Q9-D): track 0.00 -> 2.10 mm
- net Net-(Q10-D): track 0.00 -> 2.10 mm
- net Net-(Q9-G): track 0.00 -> 1.33 mm
- net Net-(Q10-S): track 0.00 -> 1.33 mm
- net Net-(Q10-G): track 0.00 -> 1.33 mm
- net Net-(Q9-S): track 0.00 -> 1.33 mm
- net Net-(Q11-S): track 0.00 -> 1.33 mm
- net Net-(Q12-G): track 0.00 -> 1.33 mm
- net Net-(Q12-S): track 0.00 -> 1.33 mm
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Other:
- board size 53.4 x 35.6 mm -> 53.4 x 38.1 mm

Commit message: backup
Parts:
- added J1: MTMM-101-04-L-D-196, connector_footprints:MTMM-101-04-L-D-196, F.Cu at (128.3, 96.5)
- added J2: MTMM-101-04-L-D-196, connector_footprints:MTMM-101-04-L-D-196, F.Cu at (128.3, 130.4)
- added J3: MTMM-101-04-L-D-196, connector_footprints:MTMM-101-04-L-D-196, F.Cu at (142.7, 130.4)
- added J4: MTMM-101-04-L-D-196, connector_footprints:MTMM-101-04-L-D-196, F.Cu at (142.7, 96.5)
- C10, C2, C5, C6, C9: footprint capacitor_footprints:C_1206_3216Metric -> capacitor_footprints:C_0805_125_2012Metric
- moved C1 1.52 mm to (133.8, 102.7)
- moved R1 1.35 mm to (138.7, 103.9), turned to -90 degrees
- moved R2 1.26 mm to (137.4, 103.9), turned to -90 degrees
- moved R41 0.91 mm to (124.0, 129.9), turned to 90 degrees
- moved R44 0.91 mm to (124.0, 97.0), turned to -90 degrees
- moved R43 0.91 mm to (146.9, 97.0), turned to -90 degrees
- moved R46 0.91 mm to (146.9, 129.9), turned to 90 degrees
- moved R16 0.69 mm to (128.3, 109.2), turned to 0 degrees
- moved R17 0.69 mm to (128.3, 117.6), turned to 0 degrees
- moved R18 0.69 mm to (142.7, 117.6), turned to 180 degrees
- moved R19 0.69 mm to (142.7, 109.2), turned to 180 degrees
- moved C3 0.54 mm to (131.6, 105.1)
- moved R3 0.51 mm to (136.1, 103.9), turned to -90 degrees
- moved C4 0.51 mm to (138.2, 124.9)
- moved R45 0.49 mm to (122.7, 128.9), turned to -90 degrees
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Connections:
- U1 pad 57: unconnected-(U1-GPIO_A-Pad57) -> /GPIO_A
- U1 pad 58: unconnected-(U1-GPIO_B-Pad58) -> /GPIO_B
- U1 pad 59: unconnected-(U1-GPIO_C-Pad59) -> /GPIO_C
- U1 pad 60: unconnected-(U1-GPIO_D-Pad60) -> /GPIO_D
Routing:
- net /GPIO_B: track 0.00 -> 36.0 mm, vias 0 -> 1
- net /GPIO_C: track 0.00 -> 34.8 mm, vias 0 -> 1
- net /GPIO_D: track 0.00 -> 15.9 mm, vias 0 -> 1
- net /GPIO_A: track 0.00 -> 15.1 mm, vias 0 -> 1
- net Net-(Q9-G): track 1.33 -> 6.61 mm
- net Net-(Q11-G): track 1.33 -> 6.61 mm
- net Net-(Q10-G): track 1.33 -> 5.88 mm
- net Net-(Q12-G): track 1.33 -> 5.75 mm
- net unconnected-(U1-GPIO_A-Pad57): track 2.62 -> 0.00 mm, vias 1 -> 0
- net unconnected-(U1-GPIO_C-Pad59): track 2.59 -> 0.00 mm, vias 1 -> 0
- net /DO_SRC_GATE_D: track 24.2 -> 26.4 mm
- net unconnected-(U1-GPIO_B-Pad58): track 2.11 -> 0.00 mm, vias 1 -> 0
- net unconnected-(U1-GPIO_D-Pad60): track 2.06 -> 0.00 mm, vias 1 -> 0
- net /VSENSEP_A: track 2.35 -> 3.81 mm
- net /VSENSEP_D: track 2.35 -> 3.81 mm
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
Commit message: backup
Parts:
- added D17: 1.8 V, diode_footprints:LED_GREEN_0402_1005Metric, F.Cu at (125.9, 94.1)
- added D18: 1.8 V, diode_footprints:LED_GREEN_0402_1005Metric, F.Cu at (125.9, 132.8)
- added D19: 1.8 V, diode_footprints:LED_GREEN_0402_1005Metric, F.Cu at (145.0, 132.8)
- added D20: 1.8 V, diode_footprints:LED_GREEN_0402_1005Metric, F.Cu at (145.0, 94.1)
- added R48: 10 kΩ, resistor_footprints:R_0402_1005Metric, F.Cu at (128.1, 94.1)
- added R49: 10 kΩ, resistor_footprints:R_0402_1005Metric, F.Cu at (128.1, 132.8)
- added R50: 10 kΩ, resistor_footprints:R_0402_1005Metric, F.Cu at (142.8, 132.8)
- added R51: 10 kΩ, resistor_footprints:R_0402_1005Metric, F.Cu at (142.8, 94.1)
- added S1: TS21-34-035-BK-160-SMT-TR, tactile_switches_footprints:TS21, F.Cu at (138.1, 100.4)
- added TP1: TestPoint, test_point_footprints:TestPoint_THTPad_Castelated, F.Cu at (132.9, 91.8)
- added TP2: TestPoint, test_point_footprints:TestPoint_THTPad_Castelated, F.Cu at (134.2, 91.8)
- added TP3: TestPoint, test_point_footprints:TestPoint_THTPad_Castelated, F.Cu at (135.5, 91.8)
- added TP4: TestPoint, test_point_footprints:TestPoint_THTPad_Castelated, F.Cu at (136.7, 91.8)
- added TP5: TestPoint, test_point_footprints:TestPoint_THTPad_Castelated, F.Cu at (138.0, 91.8)
- added TP6: TestPoint, test_point_footprints:TestPoint_THTPad_Castelated, F.Cu at (139.3, 91.8)
- added TP7: TestPoint, test_point_footprints:TestPoint_THTPad_Castelated, F.Cu at (140.5, 91.8)
- added TP8: TestPoint, test_point_footprints:TestPoint_THTPad_Castelated, F.Cu at (131.7, 91.8)
- added TP9: TestPoint, test_point_footprints:TestPoint_THTPad_Castelated, F.Cu at (130.4, 91.8)
- moved R1 1.41 mm to (140.0, 104.5)
- moved C2 0.67 mm to (131.8, 102.1)
- moved J1 0.65 mm to (127.6, 96.5)
- moved J2 0.65 mm to (127.6, 130.4)
- moved J3 0.64 mm to (143.3, 130.4)
- moved J4 0.64 mm to (143.3, 96.5)
- moved R2 0.63 mm to (137.3, 104.5)
- moved R3 0.62 mm to (136.1, 104.5)
- moved C1 0.60 mm to (134.4, 103.0)
- moved C3 0.26 mm to (131.4, 105.1)
Connections:
- net Net-(U1-LDO1V8) renamed /LDO1V8
- net Net-(U1-~{RESET}) renamed /~{RESET}
- C2 pad 1: Net-(U1-DVCC) -> /DVCC
- C3 pad 1: Net-(U1-DVCC) -> /DVCC
- R1 pad 1: unconnected-(R1-Pad1) -> /DVCC
- R2 pad 1: unconnected-(R2-Pad1) -> /DVCC
- R3 pad 1: unconnected-(R3-Pad1) -> /DVCC
- U1 pad 50: unconnected-(U1-~{SYNC}-Pad50) -> Net-(U1-~{SYNC})
- U1 pad 51: unconnected-(U1-SCLK-Pad51) -> Net-(U1-SCLK)
- U1 pad 52: unconnected-(U1-SDI-Pad52) -> Net-(U1-SDI)
- U1 pad 53: unconnected-(U1-SDO-Pad53) -> Net-(U1-SDO)
- U1 pad 62: Net-(U1-DVCC) -> /DVCC
Routing:
- net /~{RESET}: track 5.19 -> 25.3 mm
- net Net-(U1-SDO): track 0.00 -> 16.6 mm, vias 0 -> 1
- net Net-(U1-~{SYNC}): track 0.00 -> 16.5 mm, vias 0 -> 1
- net Net-(U1-SCLK): track 0.00 -> 16.3 mm, vias 0 -> 1
- net Net-(U1-SDI): track 0.00 -> 16.2 mm, vias 0 -> 1
- net Net-(U1-~{ALERT}): track 4.85 -> 18.2 mm
- net Net-(U1-~{ADC_RDY}): track 4.66 -> 17.7 mm
- net /GPIO_D: track 15.9 -> 24.4 mm
- net /GPIO_A: track 15.1 -> 22.7 mm
- net Net-(U1-DVCC): track 5.55 -> 0.00 mm
- net /GPIO_B: track 36.0 -> 38.9 mm
- net unconnected-(U1-SCLK-Pad51): track 2.70 -> 0.00 mm, vias 1 -> 0
- net unconnected-(U1-SDO-Pad53): track 2.69 -> 0.00 mm, vias 1 -> 0
- net /DVCC: track 0.00 -> 2.29 mm, vias 0 -> 5
- net unconnected-(U1-SDI-Pad52): track 2.15 -> 0.00 mm, vias 1 -> 0
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- added copper zone on F.Cu, net /DVCC
- added copper zone on In1.Cu, net /DVCC
Other:
- board size 53.4 x 38.1 mm -> 53.4 x 43.2 mm

Commit message: backup
Parts:
- added TP10: TestPoint, test_point_footprints:TestPoint_THTPad_Castelated, F.Cu at (131.0, 135.0)
- added TP11: TestPoint, test_point_footprints:TestPoint_THTPad_Castelated, F.Cu at (132.3, 135.0)
- added TP12: TestPoint, test_point_footprints:TestPoint_THTPad_Castelated, F.Cu at (136.1, 135.0)
- added TP13: TestPoint, test_point_footprints:TestPoint_THTPad_Castelated, F.Cu at (134.8, 135.0)
- added TP14: TestPoint, test_point_footprints:TestPoint_THTPad_Castelated, F.Cu at (139.9, 135.1)
- added TP15: TestPoint, test_point_footprints:TestPoint_THTPad_Castelated, F.Cu at (138.6, 135.1)
- added TP16: TestPoint, test_point_footprints:TestPoint_THTPad_Castelated, F.Cu at (141.2, 91.8)
- added TP17: TestPoint, test_point_footprints:TestPoint_THTPad_Castelated, F.Cu at (163.4, 112.8)
- added TP18: TestPoint, test_point_footprints:TestPoint_THTPad_Castelated, F.Cu at (163.4, 114.0)
- added TP19: TestPoint, test_point_footprints:TestPoint_THTPad_Castelated, F.Cu at (107.5, 112.8)
- added TP20: TestPoint, test_point_footprints:TestPoint_THTPad_Castelated, F.Cu at (107.5, 114.0)
- moved C15 0.86 mm to (123.2, 119.2)
- moved C16 0.86 mm to (147.8, 119.2)
- moved C14 0.81 mm to (123.2, 107.6)
- moved C17 0.81 mm to (147.8, 107.6)
- moved D17 0.76 mm to (125.2, 94.1)
- moved D18 0.76 mm to (125.2, 132.8)
- moved D19 0.76 mm to (145.8, 132.8)
- moved D20 0.76 mm to (145.8, 94.1)
- moved J1 0.76 mm to (126.9, 96.5)
- moved J2 0.76 mm to (126.9, 130.4)
- moved J3 0.76 mm to (144.1, 130.4)
- moved J4 0.76 mm to (144.1, 96.5)
- moved R48 0.76 mm to (127.3, 94.1)
- moved R49 0.76 mm to (127.3, 132.8)
- moved R50 0.76 mm to (143.6, 132.8)
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Connections:
- net Net-(U1-AVCC) renamed /AVCC
- net Net-(U1-AVDD_HI) renamed /AVDD_HI
- net Net-(U1-AVDD_LO) renamed /AVDD_LO
Routing:
- net GNDA: track 11.2 -> 1.02 mm, vias 32 -> 56
- net /VIOUT_A: track 11.0 -> 7.44 mm
- net /VIOUT_D: track 11.0 -> 7.48 mm
- net /VIOUT_B: track 11.0 -> 7.46 mm
- net /VIOUT_C: track 11.0 -> 7.50 mm
- net /SENSELF_B: track 11.2 -> 8.93 mm
- net Net-(Q12-G): track 5.10 -> 4.34 mm
- net Net-(Q10-G): track 5.23 -> 4.47 mm
- net /AVDD_LO: vias 0 -> 4
- net /AVDD_HI: vias 0 -> 4
- added copper zone on In1.Cu, net /AVCC
- added copper zone on In1.Cu, net /AVDD_HI
- added copper zone on In1.Cu, net /AVDD_LO
- added copper zone on In1.Cu, net /AVSS
Other:
- board size 53.4 x 43.2 mm -> 55.9 x 43.2 mm

Commit message: backup
Parts:
- added TP21: TestPoint, test_point_footprints:TestPoint_THTPad_Castelated, F.Cu at (106.2, 101.3)
- added TP22: TestPoint, test_point_footprints:TestPoint_THTPad_Castelated, F.Cu at (106.2, 103.9)
- added TP23: TestPoint, test_point_footprints:TestPoint_THTPad_Castelated, F.Cu at (106.2, 106.4)
- added TP24: TestPoint, test_point_footprints:TestPoint_THTPad_Castelated, F.Cu at (106.2, 109.0)
- added TP25: TestPoint, test_point_footprints:TestPoint_THTPad_Castelated, F.Cu at (106.2, 125.5)
- added TP26: TestPoint, test_point_footprints:TestPoint_THTPad_Castelated, F.Cu at (106.2, 122.9)
- added TP27: TestPoint, test_point_footprints:TestPoint_THTPad_Castelated, F.Cu at (106.2, 120.4)
- added TP28: TestPoint, test_point_footprints:TestPoint_THTPad_Castelated, F.Cu at (106.2, 117.9)
- added TP29: TestPoint, test_point_footprints:TestPoint_THTPad_Castelated, F.Cu at (164.7, 125.5)
- added TP30: TestPoint, test_point_footprints:TestPoint_THTPad_Castelated, F.Cu at (164.7, 122.9)
- added TP31: TestPoint, test_point_footprints:TestPoint_THTPad_Castelated, F.Cu at (164.7, 120.4)
- added TP32: TestPoint, test_point_footprints:TestPoint_THTPad_Castelated, F.Cu at (164.7, 117.9)
- added TP33: TestPoint, test_point_footprints:TestPoint_THTPad_Castelated, F.Cu at (164.7, 101.3)
- added TP34: TestPoint, test_point_footprints:TestPoint_THTPad_Castelated, F.Cu at (164.7, 103.9)
- added TP35: TestPoint, test_point_footprints:TestPoint_THTPad_Castelated, F.Cu at (164.7, 106.4)
- added TP36: TestPoint, test_point_footprints:TestPoint_THTPad_Castelated, F.Cu at (164.7, 109.0)
- moved J6 9.20 mm to (119.1, 120.8), turned to 180 degrees
- moved J5 9.20 mm to (119.1, 106.0), turned to 0 degrees
- moved J7 9.20 mm to (151.8, 120.8), turned to 180 degrees
- moved J8 9.20 mm to (151.8, 106.0), turned to 0 degrees
- moved R16 3.82 mm to (129.3, 105.5), turned to 90 degrees
- moved R19 3.82 mm to (141.7, 105.5), turned to 90 degrees
- moved R17 3.81 mm to (129.3, 121.3), turned to -90 degrees
- moved R18 3.81 mm to (141.7, 121.3), turned to -90 degrees
- moved R27 3.53 mm to (143.1, 104.5), turned to -90 degrees
- moved R24 3.53 mm to (127.8, 104.5), turned to -90 degrees
- moved R26 3.53 mm to (143.1, 122.3), turned to 90 degrees
- moved R25 3.53 mm to (127.8, 122.3), turned to 90 degrees
- moved C19 3.44 mm to (127.8, 119.5)
- moved C20 3.44 mm to (143.1, 119.5)
- moved C18 3.42 mm to (127.8, 107.3)
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Routing:
- net /ISP_A: track 3.15 -> 21.8 mm
- net /ISP_D: track 3.15 -> 21.8 mm
- net /ISP_C: track 3.15 -> 21.8 mm
- net /ISP_B: track 3.15 -> 21.8 mm
- net /ISN_D: track 14.9 -> 24.0 mm
- net /ISN_C: track 14.9 -> 23.8 mm
- net /ISN_A: track 15.6 -> 23.9 mm
- net /ISN_B: track 15.6 -> 23.9 mm
- net /VIOUT_C: track 7.50 -> 4.52 mm
- net /VIOUT_D: track 7.48 -> 4.52 mm
- net /VIOUT_B: track 7.46 -> 4.53 mm
- net /VIOUT_A: track 7.44 -> 4.53 mm
- net /LKG_COMP_C: track 13.6 -> 16.5 mm
- net /VSENSEP_D: track 3.81 -> 6.68 mm
- net /LKG_COMP_B: track 13.6 -> 16.5 mm
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Other:
- board size 55.9 x 43.2 mm -> 58.4 x 43.2 mm

Commit message: backup
Parts:
- added D21: 100.0 V, diode_footprints:SOD_523, F.Cu at (135.5, 97.6)
Routing:
- net /AVDD_LO: track 0.00 -> 5.08 mm, vias 4 -> 5
- net /AVDD_HI: track 0.00 -> 5.08 mm, vias 4 -> 5
- added copper zone on B.Cu, net /DO_VDD
- removed copper zone on In1.Cu, net /DO_VDD
