File: minimal_ad74416h/minimal_ad74416h.kicad_pcb (KiCad board)
At the start: 4 copper layers, 53.4 x 43.2 mm, 163 parts, among them J1 MTMM-101-04-L-D-196, J2 MTMM-101-04-L-D-196, J3 MTMM-101-04-L-D-196, J4 MTMM-101-04-L-D-196, J5 MTMM-101-04-L-D-196, J6 MTMM-101-04-L-D-196, J7 MTMM-101-04-L-D-196, J8 MTMM-101-04-L-D-196, Q1 50 V, Q10 -100.0 V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

Commit message: backup
Parts:
- moved R4 3.09 mm to (158.0, 93.6), turned to 0 degrees
- moved R3 3.09 mm to (112.9, 93.6), turned to 180 degrees
- moved R49 3.09 mm to (158.0, 133.3), turned to 0 degrees
- moved R48 3.09 mm to (112.9, 133.3), turned to 180 degrees
- moved J8 0.65 mm to (153.1, 131.0)
- moved Q12 0.65 mm to (157.1, 131.0)
- moved Q2 0.65 mm to (157.1, 96.0)
- moved D1 0.65 mm to (117.5, 92.8)
- moved D2 0.65 mm to (153.4, 92.8)
- moved D20 0.65 mm to (117.5, 134.0)
- moved D21 0.65 mm to (153.4, 134.0)
- moved J1 0.65 mm to (117.8, 96.0)
- moved J2 0.65 mm to (153.1, 96.0)
- moved J7 0.65 mm to (117.8, 131.0)
- moved Q1 0.65 mm to (113.8, 96.0)
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Routing:
- net /GPIO_B: track 45.7 -> 44.6 mm
- net /LKG_COMP_D: track 16.4 -> 15.4 mm
- net /LKG_COMP_C: track 16.5 -> 15.4 mm
- net /LKG_COMP_B: track 16.5 -> 15.4 mm
- net /LKG_COMP_A: track 16.4 -> 15.4 mm
- net /DO_SRC_GATE_A: track 27.9 -> 27.0 mm
- net /DO_SRC_SNS_A: track 22.9 -> 22.0 mm
- net unconnected-(U1-LVIN-Pad18): track 1.38 -> 2.24 mm
- net /GPIO_C: track 43.8 -> 43.0 mm
- net /DO_SRC_SNS_D: track 24.5 -> 23.8 mm
- net Net-(Q2-S): track 1.59 -> 2.19 mm
- net /DO_SRC_GATE_D: track 25.0 -> 24.4 mm
- net Net-(Q11-S): track 1.64 -> 2.22 mm
- net GNDA: vias 59 -> 83

Commit message: backup
Parts:
- added S2: 416131160802, dip_switches_footprints:416131160802, F.Cu at (130.6, 95.4)
- S3: renamed from J3; value MTMM-101-04-L-D-196 -> 416131160801; footprint connector_footprints:MTMM-101-04-L-D-196 -> dip_switches_footprints:416131160801
- S4: renamed from J4; value MTMM-101-04-L-D-196 -> 416131160801; footprint connector_footprints:MTMM-101-04-L-D-196 -> dip_switches_footprints:416131160801
- S5: renamed from J5; value MTMM-101-04-L-D-196 -> 416131160801; footprint connector_footprints:MTMM-101-04-L-D-196 -> dip_switches_footprints:416131160801
- S6: renamed from J6; value MTMM-101-04-L-D-196 -> 416131160801; footprint connector_footprints:MTMM-101-04-L-D-196 -> dip_switches_footprints:416131160801
- moved S5 3.91 mm to (122.3, 123.1), turned to 90 degrees
- moved S6 3.91 mm to (148.6, 123.1), turned to -90 degrees
- moved S3 3.81 mm to (122.3, 103.9), turned to 90 degrees
- moved S4 3.81 mm to (148.6, 103.9), turned to -90 degrees
- moved D5 2.64 mm to (138.1, 97.6)
- moved C32 1.27 mm to (122.8, 132.2)
- moved TP1 1.27 mm to (129.8, 90.6)
- moved TP10 1.27 mm to (141.2, 90.6)
- moved TP2 1.27 mm to (131.0, 90.6)
- moved TP3 1.27 mm to (132.3, 90.6)
- moved TP4 1.27 mm to (133.6, 90.6)
- moved TP5 1.27 mm to (134.8, 90.6)
- moved TP6 1.27 mm to (136.1, 90.6)
- moved TP7 1.27 mm to (137.4, 90.6)
- moved TP8 1.27 mm to (138.6, 90.6)
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Connections:
- S3 pad 1: /ISP_A -> /I/OP_A
- S3 pad 2: /I/OP_A -> /ISP_A
- S4 pad 1: /ISP_D -> /I/OP_D
- S4 pad 2: /I/OP_D -> /ISP_D
- S5 pad 1: /ISP_B -> /I/OP_B
- S5 pad 2: /I/OP_B -> /ISP_B
- S6 pad 1: /ISP_C -> /I/OP_C
- S6 pad 2: /I/OP_C -> /ISP_C
- U1 pad 63: unconnected-(U1-AD0-Pad63) -> /AD0
- U1 pad 64: unconnected-(U1-AD1-Pad64) -> /AD1
Routing:
- net /AD1: track 0.00 -> 16.5 mm, vias 0 -> 2
- net /AD0: track 0.00 -> 14.8 mm, vias 0 -> 2
- net /AVDD_HI: track 5.08 -> 8.33 mm
- net unconnected-(U1-AD1-Pad64): track 2.76 -> 0.00 mm, vias 1 -> 0
- net /AVDD_LO: track 5.08 -> 2.44 mm
- net unconnected-(U1-AD0-Pad63): track 2.64 -> 0.00 mm, vias 1 -> 0
- net /REFIO: track 18.7 -> 20.0 mm
- net Net-(U1-~{ALERT}): track 18.0 -> 19.3 mm
- net Net-(U1-~{ADC_RDY}): track 17.5 -> 18.8 mm
- net Net-(U1-SDO): track 16.4 -> 17.7 mm
- net Net-(U1-SDI): track 16.2 -> 17.5 mm
- net Net-(U1-SCLK): track 16.4 -> 17.7 mm
- net /~{RESET}: track 25.5 -> 26.8 mm
- net Net-(U1-~{SYNC}): track 16.7 -> 17.9 mm
- net /ISP_D: track 19.8 -> 21.0 mm, vias 0 -> 1
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Other:
- board size 53.4 x 43.2 mm -> 53.4 x 45.7 mm

Commit message: backup
Parts:
- removed J1, J2, J7, J8: MTMM-101-04-L-D-196, connector_footprints:MTMM-101-04-L-D-196
- added S10: 416131160801, dip_switches_footprints:416131160801, F.Cu at (153.3, 92.1)
- added S7: 416131160801, dip_switches_footprints:416131160801, F.Cu at (117.6, 92.1)
- added S8: 416131160801, dip_switches_footprints:416131160801, F.Cu at (117.6, 134.9)
- added S9: 416131160801, dip_switches_footprints:416131160801, F.Cu at (153.3, 134.9)
- moved D20 6.03 mm to (121.1, 130.1), turned to -90 degrees
- moved D21 6.03 mm to (149.8, 130.1), turned to -90 degrees
- moved D1 5.97 mm to (121.1, 96.8), turned to 90 degrees
- moved D2 5.97 mm to (149.8, 96.8), turned to 90 degrees
- moved R4 3.97 mm to (154.3, 94.2), turned to 180 degrees
- moved R49 3.97 mm to (154.3, 132.7), turned to 180 degrees
- moved R3 3.97 mm to (116.6, 94.2), turned to 0 degrees
- moved R48 3.97 mm to (116.6, 132.7), turned to 0 degrees
- moved R50 3.81 mm to (121.1, 132.2), turned to 90 degrees
- moved R51 3.81 mm to (149.8, 132.2), turned to 90 degrees
- moved R1 3.77 mm to (121.1, 94.6), turned to -90 degrees
- moved R2 3.77 mm to (149.8, 94.6), turned to -90 degrees
- moved D5 2.64 mm to (135.5, 97.6)
- moved C32 1.55 mm to (122.8, 130.7), turned to 90 degrees
- moved TP31 1.27 mm to (132.3, 137.5)
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Routing:
- net /AVDD_HI: track 8.33 -> 5.08 mm
- net /AVDD_LO: track 2.44 -> 5.08 mm
- net /REFIO: track 20.0 -> 21.7 mm
- net Net-(Q1-G): track 4.05 -> 5.59 mm
- net Net-(Q12-G): track 4.15 -> 5.59 mm
- net Net-(U1-~{ALERT}): track 19.3 -> 20.6 mm
- net Net-(U1-SCLK): track 17.7 -> 18.9 mm
- net Net-(U1-~{ADC_RDY}): track 18.8 -> 20.1 mm
- net Net-(U1-SDO): track 17.7 -> 18.9 mm
- net /~{RESET}: track 26.8 -> 28.1 mm
- net Net-(U1-SDI): track 17.5 -> 18.8 mm
- net Net-(U1-~{SYNC}): track 17.9 -> 19.2 mm
- net /GPIO_C: track 43.7 -> 42.5 mm, vias 1 -> 2
- net /GPIO_A: track 30.7 -> 29.6 mm, vias 1 -> 2
- net /GPIO_D: track 31.0 -> 30.0 mm, vias 1 -> 2
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Other:
- board size 53.4 x 45.7 mm -> 53.4 x 48.3 mm

Commit message: backup
Parts:
- added R52: 33 kΩ, resistor_footprints:R_0805_2012Metric, F.Cu at (125.7, 130.2)
- added RT1: 33 kΩ, resistor_footprints:RT_0805_RT_2012Metric, F.Cu at (122.8, 131.2)
- added TP37: TestPoint, test_point_footprints:TestPoint_THTPad_Castelated, F.Cu at (108.8, 97.5)
- added TP38: TestPoint, test_point_footprints:TestPoint_THTPad_Castelated, F.Cu at (108.7, 129.3)
- added TP39: TestPoint, test_point_footprints:TestPoint_THTPad_Castelated, F.Cu at (162.2, 129.3)
- added TP40: TestPoint, test_point_footprints:TestPoint_THTPad_Castelated, F.Cu at (162.2, 97.5)
- moved C32 6.30 mm to (129.1, 130.2), turned to 0 degrees
- moved U2 2.13 mm to (127.6, 134.2)
- moved C30 1.27 mm to (134.3, 133.4)
- moved C31 1.27 mm to (132.3, 133.4)
Connections:
- U1 pad 18: unconnected-(U1-LVIN-Pad18) -> /LVIN
Routing:
- net /LVIN: track 0.00 -> 21.5 mm, vias 0 -> 2
- net /GPIO_B: track 44.7 -> 63.1 mm
- net /GPIO_C: track 42.5 -> 59.0 mm
- net /GPIO_D: track 30.0 -> 46.4 mm
- net /GPIO_A: track 29.6 -> 45.9 mm
- net unconnected-(U1-LVIN-Pad18): track 2.24 -> 0.00 mm, vias 1 -> 0
- net /REFIO: track 21.7 -> 22.6 mm
