File: minimal_ad74416h/minimal_ad74416h.kicad_sch (KiCad schematic)
At the start: 1 part, among them U1 AD74416HBCPZ-RL7

Commit message: backup
Parts:
- added C1, C3, C5, C7, C9: 10 µF, capacitor_footprints:C_1206_3216Metric, symbol UNITED_CAPACITORS_DATA_BASE:C_CL31B106KBHNNN#
- added C10, C2, C4, C6, C8: 100 nF, capacitor_footprints:C_0402_1005Metric, symbol UNITED_CAPACITORS_DATA_BASE:C_GCM155R71H104KE02D
- added C11: 10 µF, capacitor_footprints:C_1210_250_3225Metric, symbol UNITED_CAPACITORS_DATA_BASE:C_GRM32EC72A106KE05L
- added C12: 2.2 µF, capacitor_footprints:C_0805_2012Metric, symbol UNITED_CAPACITORS_DATA_BASE:C_CGA4J1X7R1V225K125AC
- added C13: 39 nF, capacitor_footprints:C_0603_1608Metric, symbol UNITED_CAPACITORS_DATA_BASE:C_GCM188R71H393KA55D
- added R1, R12, R2: 10 kΩ, resistor_footprints:R_0402_1005Metric, symbol UNITED_RESISTORS_DATA_BASE:R_ERJ-2RKF1002X
Connections:
- net at U1.17 (REFIO1): now also C13.1
- net at U1.19 (AVCC): now also C5.1, C6.1
- net GNDA: now reaches U1.20 (AGND)
- net GNDA: now also U1.40 (AGND), U1.54 (DGND), U1.9 (AGND), C1.2, C10.2, C11.1, C12.1, C13.2, C2.2, C3.2, C4.2, C5.2, C6.2, C7.2, C8.2, C9.2
- net AVSS: now reaches U1.21 (AVSS)
- net AVSS: now also U1.PAD, C7.1, C8.1
- net at U1.26 (DO_VDD): now also C11.2
- net at U1.41 (AVDD_LO): now also C3.1, C4.1
- net at U1.49 (~{RESET}): now also R2.2
- net at U1.55 (~{ALERT}): now also R1.2
- net at U1.56 (~{ADC_RDY}): now also R12.2
- net at U1.61 (LDO1V8): now also C12.2
- net at U1.62 (DVCC): now also C10.1, C9.1
- net at U1.8 (AVDD_HI): now also C1.1, C2.1
Other:
- moved on the sheet: U1

Commit message: backup
Parts:
- renumbered C12 to C1, C7 to C10, C2 to C11, C8 to C12, C9 to C2, C10 to C3, C11 to C4, C3 to C5, C5 to C6, C4 to C7, C6 to C8, C1 to C9, R2 to R1, R1 to R2, R12 to R3
Connections:
- net VIOUT_A: now reaches U1.1 (VIOUT_A)
- net CCOMP_B: now reaches U1.10 (CCOMP_B)
- net SENSELF_B: now reaches U1.12 (SENSELF_B)
- net SENSEHF_B: now reaches U1.13 (SENSEHF_B)
- net VIOUT_B: now reaches U1.16 (VIOUT_B)
- net VIOUT_C: now reaches U1.33 (VIOUT_C)
- net SENSEHF_C: now reaches U1.36 (SENSEHF_C)
- net SENSELF_C: now reaches U1.37 (SENSELF_C)
- net CCOMP_C: now reaches U1.39 (CCOMP_C)
- net SENSEHF_A: now reaches U1.4 (SENSEHF_A)
- net CCOMP_D: now reaches U1.42 (CCOMP_D)
- net SENSELF_D: now reaches U1.44 (SENSELF_D)
- net SENSEHF_D: now reaches U1.45 (SENSEHF_D)
- net VIOUT_D: now reaches U1.48 (VIOUT_D)
- net SENSELF_A: now reaches U1.5 (SENSELF_A)
- net CCOMP_A: now reaches U1.7 (CCOMP_A)
Other:
- added sheet Front End Channel 1 (Front End Channel 1.kicad_sch)
- added sheet Front End Channel 2 (Front End Channel 1.kicad_sch)
- added sheet Front End Channel 3 (Front End Channel 1.kicad_sch)
- added sheet Front End Channel 4 (Front End Channel 1.kicad_sch)

Commit message: backup
Connections:
- net VSENSEN_B: now reaches U1.11 (VSENSEN_B)
- net VSENSEP_B: now reaches U1.14 (VSENSEP_B)
- net VSENSEP_A: now reaches U1.3 (VSENSEP_A)
- net VSENSEP_C: now reaches U1.35 (VSENSEP_C)
- net VSENSEN_C: now reaches U1.38 (VSENSEN_C)
- net VSENSEN_D: now reaches U1.43 (VSENSEN_D)
- net VSENSEP_D: now reaches U1.46 (VSENSEP_D)
- net VSENSEN_A: now reaches U1.6 (VSENSEN_A)
Other:
- sheet Front End Channel 1 ports: added I/OP, VSENSEN, VSENSEP; removed none
- sheet Front End Channel 2 ports: added I/OP, VSENSEN, VSENSEP; removed none
- sheet Front End Channel 3 ports: added I/OP, VSENSEN, VSENSEP; removed none
- sheet Front End Channel 4 ports: added I/OP, VSENSEN, VSENSEP; removed none

Commit message: backup
Connections:
- net LKG_COMP_B: now reaches U1.15 (LKG_COMP_B)
- net LKG_COMP_A: now reaches U1.2 (LKG_COMP_A)
- net LKG_COMP_C: now reaches U1.34 (LKG_COMP_C)
- net LKG_COMP_D: now reaches U1.47 (LKG_COMP_D)
Other:
- sheet Front End Channel 1 ports: added ISN, ISP, LKG_COMP; removed none
- sheet Front End Channel 2 ports: added ISN, ISP, LKG_COMP; removed none
- sheet Front End Channel 3 ports: added ISN, ISP, LKG_COMP; removed none
- sheet Front End Channel 4 ports: added ISN, ISP, LKG_COMP; removed none

Commit message: backup
Connections:
- net DO_SRC_GATE_A: now reaches U1.22 (DO_SRC_GATE_A)
- net DO_SRC_SNS_A: now reaches U1.23 (DO_SRC_SNS_A)
- net DO_SRC_GATE_B: now reaches U1.24 (DO_SRC_GATE_B)
- net DO_SRC_SNS_B: now reaches U1.25 (DO_SRC_SNS_B)
- net DO_SRC_SNS_C: now reaches U1.27 (DO_SRC_SNS_C)
- net DO_SRC_GATE_C: now reaches U1.28 (DO_SRC_GATE_C)
- net DO_SRC_SNS_D: now reaches U1.29 (DO_SRC_SNS_D)
- net DO_SRC_GATE_D: now reaches U1.30 (DO_SRC_GATE_D)
Other:
- sheet Front End Channel 1 ports: added DO_SRC_GATE, DO_SRC_SNS; removed none
- sheet Front End Channel 2 ports: added DO_SRC_GATE, DO_SRC_SNS; removed none
- sheet Front End Channel 3 ports: added DO_SRC_GATE, DO_SRC_SNS; removed none
- sheet Front End Channel 4 ports: added DO_SRC_GATE, DO_SRC_SNS; removed none

Commit message: backup
Parts:
- C13: footprint capacitor_footprints:C_0603_1608Metric -> capacitor_footprints:C_0402_1005Metric; symbol UNITED_CAPACITORS_DATA_BASE:C_GCM188R71H393KA55D -> UNITED_CAPACITORS_DATA_BASE:C_KGM05AR71C393KH; Case Code - in 0603 -> 0402; Case Code - mm 1608 -> 1005; MPN GCM188R71H393KA55D -> KGM05AR71C393KH; Manufacturer Murata Electronics -> KYOCERA AVX; Series GCM188R71H -> KGM05AR71C; Symbol Name C_GCM188R71H393KA55D -> C_KGM05AR71C393KH; Trustedparts Search https://www.trustedparts.com/en/search/GCM188R71H393KA55D -> https://www.trustedparts.com/en/search/KGM05AR71C393KH; Voltage Rating 50V -> 16V
Changed lines of the file:
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@@
 	)
 	(symbol
-		(lib_id "UNITED_CAPACITORS_DATA_BASE:C_GCM188R71H393KA55D")
+		(lib_id "UNITED_CAPACITORS_DATA_BASE:C_KGM05AR71C393KH")
 		(at 182.88 109.22 270)
 		(unit 1)
@@
 		(on_board yes)
 		(dnp no)
+		(fields_autoplaced yes)
 		(property "Reference" "C13"
 			(at 179.07 107.9499 90)
@@
 			)
 		)
-		(property "Footprint" "capacitor_footprints:C_0603_1608Metric"
+		(property "Footprint" "capacitor_footprints:C_0402_1005Metric"
 			(at 175.26 109.22 0)
 			(show_name yes)
@@
 			)
 		)
-		(property "Datasheet" "https://search.murata.co.jp/Ceramy/image/img/A01X/G101/ENG/GCM188R71H393KA55-01.pdf"
+		(property "Datasheet" "https://datasheets.kyocera-avx.com/KGM_X7R.pdfKGM05AR71C393KH"
 			(at 172.72 109.22 0)
 			(show_name yes)
@@
 			)
 		)
-		(property "Description" "CAP SMD 39 nF X7R 10% 0603 50V"
+		(property "Description" "CAP SMD 39 nF X7R 10% 0402 16V"
 			(at 170.18 109.22 0)
 			(show_name yes)
@@
 			)
 		)
-		(property "Case Code - in" "0603"
+		(property "Case Code - in" "0402"
 			(at 165.1 109.22 0)
 			(show_name yes)
@@
 			)
 		)
-		(property "Case Code - mm" "1608"
+		(property "Case Code - mm" "1005"
 			(at 162.56 109.22 0)
 			(show_name yes)
@@
 			)
 		)
-		(property "MPN" "GCM188R71H393KA55D"
+		(property "MPN" "KGM05AR71C393KH"
 			(at 157.48 109.22 0)
 			(show_name yes)
@@
 			)
 		)
-		(property "Manufacturer" "Murata Electronics"
+		(property "Manufacturer" "KYOCERA AVX"
 			(at 154.94 109.22 0)
 			(show_name yes)
@@
 			)
 		)
-		(property "Series" "GCM188R71H"
+		(property "Series" "KGM05AR71C"
 			(at 152.4 109.22 0)
 			(show_name yes)
@@
 			)
 		)
-		(property "Symbol Name" "C_GCM188R71H393KA55D"
+		(property "Symbol Name" "C_KGM05AR71C393KH"
 			(at 149.86 109.22 0)
 			(show_name yes)
@@
 			)
 		)
-		(property "Trustedparts Search" "https://www.trustedparts.com/en/search/GCM188R71H393KA55D"
+		(property "Trustedparts Search" "https://www.trustedparts.com/en/search/KGM05AR71C393KH"
 			(at 144.78 109.22 0)
 			(show_name yes)
@@
 			)
 		)
-		(property "Voltage Rating" "50V"
+		(property "Voltage Rating" "16V"
 			(at 142.24 109.22 0)
 			(show_name yes)

Commit message: backup
Connections:
- net DO_VDD: now reaches C4.2, U1.26 (DO_VDD)
Other:
- sheet Front End Channel 1 ports: added DO_VDD, I/ON; removed none
- sheet Front End Channel 2 ports: added DO_VDD, I/ON; removed none
- sheet Front End Channel 3 ports: added DO_VDD, I/ON; removed none
- sheet Front End Channel 4 ports: added DO_VDD, I/ON; removed none
- moved on the sheet: C1, C10, C11, C12, C2, C3, C4, C5, C6, C7, C8, C9

Commit message: backup
Connections:
- net GPIO_A: now reaches U1.57 (GPIO_A)
- net GPIO_B: now reaches U1.58 (GPIO_B)
- net GPIO_C: now reaches U1.59 (GPIO_C)
- net GPIO_D: now reaches U1.60 (GPIO_D)
Other:
- sheet Front End Channel 1 ports: added GPIO; removed none
- sheet Front End Channel 2 ports: added GPIO; removed none
- sheet Front End Channel 3 ports: added GPIO; removed none
- sheet Front End Channel 4 ports: added GPIO; removed none
Changed lines of the file:
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@@
 	(wire
 		(pts
+			(xy 182.88 162.56) (xy 185.42 162.56)
+		)
+		(stroke
+			(width 0)
+			(type default)
+		)
+	)
+	(wire
+		(pts
 			(xy 220.98 144.78) (xy 241.3 144.78)
 		)
@@
 	(wire
 		(pts
+			(xy 238.76 185.42) (xy 241.3 185.42)
+		)
+		(stroke
+			(width 0)
+			(type default)
+		)
+	)
+	(wire
+		(pts
 			(xy 208.28 223.52) (xy 208.28 224.79)
 		)
@@
 	(wire
 		(pts
-			(xy 238.76 154.94) (xy 241.3 154.94)
+			(xy 238.76 152.4) (xy 241.3 152.4)
 		)
 		(stroke
@@
 	(wire
 		(pts
+			(xy 182.88 165.1) (xy 185.42 165.1)
+		)
+		(stroke
+			(width 0)
+			(type default)
+		)
+	)
+	(wire
+		(pts
 			(xy 266.7 203.2) (xy 273.05 203.2)
 		)
@@
 	(wire
 		(pts
-			(xy 238.76 124.46) (xy 241.3 124.46)
+			(xy 238.76 121.92) (xy 241.3 121.92)
 		)
 		(stroke
@@
 	(wire
 		(pts
+			(xy 182.88 160.02) (xy 185.42 160.02)
+		)
+		(stroke
+			(width 0)
+			(type default)
+		)
+	)
+	(wire
+		(pts
 			(xy 205.74 27.94) (xy 205.74 33.02)
 		)
@@
 	(wire
 		(pts
+			(xy 182.88 167.64) (xy 185.42 167.64)
+		)
+		(stroke
+			(width 0)
+			(type default)
+		)
+	)
+	(wire
+		(pts
 			(xy 218.44 50.8) (xy 213.36 50.8)
 		)
@@
 	(wire
 		(pts
+			(xy 238.76 154.94) (xy 241.3 154.94)
+		)
+		(stroke
+			(width 0)
+			(type default)
+		)
+	)
+	(wire
+		(pts
 			(xy 220.98 193.04) (xy 241.3 193.04)
 		)
@@
 	(wire
 		(pts
-			(xy 238.76 185.42) (xy 241.3 185.42)
+			(xy 238.76 182.88) (xy 241.3 182.88)
 		)
 		(stroke
@@
 	(wire
 		(pts
+			(xy 238.76 91.44) (xy 241.3 91.44)
+		)
+		(stroke
+			(width 0)
+			(type default)
+		)
+	)
+	(wire
+		(pts
 			(xy 238.76 93.98) (xy 241.3 93.98)
 		)
@@
 	(wire
 		(pts
+			(xy 238.76 124.46) (xy 241.3 124.46)
+		)
+		(stroke
+			(width 0)
+			(type default)
+		)
+	)
+	(wire
+		(pts
 			(xy 190.5 78.74) (xy 187.96 78.74)
 		)
@@
 		)
 	)
+	(label "GPIO_A"
+		(at 238.76 93.98 180)
+		(effects
+			(font
+				(size 1.27 1.27)
+			)
+			(justify right bottom)
+		)
+	)
 	(label "AVSS"
 		(at 215.9 228.6 0)
@@
 		)
 	)
+	(label "GPIO_D"
+		(at 182.88 160.02 180)
+		(effects
+			(font
+				(size 1.27 1.27)
+			)
+			(justify right bottom)
+		)
+	)
 	(label "DO_SRC_GATE_B"
 		(at 222.25 129.54 0)
@@
 		)
 	)
+	(label "GPIO_D"
+		(at 238.76 185.42 180)
+		(effects
+			(font
+				(size 1.27 1.27)
+			)
+			(justify right bottom)
+		)
+	)
+	(label "GPIO_C"
+		(at 238.76 154.94 180)
+		(effects
+			(font
+				(size 1.27 1.27)
+			)
+			(justify right bottom)
+		)
+	)
 	(label "DO_SRC_GATE_A"
 		(at 222.25 99.06 0)
@@
 		)
 	)
+	(label "GPIO_B"
+		(at 238.76 124.46 180)
+		(effects
+			(font
+				(size 1.27 1.27)
+			)
+			(justify right bottom)
+		)
+	)
 	(label "SENSEHF_D"
 		(at 222.25 203.2 0)
@@
 	)
 	(label "DO_VDD"
-		(at 238.76 124.46 180)
+		(at 238.76 121.92 180)
+		(effects
+			(font
+				(size 1.27 1.27)
+			)
+			(justify right bottom)
+		)
+	)
+	(label "GPIO_B"
+		(at 182.88 165.1 180)
 		(effects
 			(font
@@
 		)
 	)
+	(label "GPIO_C"
+		(at 182.88 162.56 180)
+		(effects
+			(font
+				(size 1.27 1.27)
+			)
+			(justify right bottom)
+		)
+	)
+	(label "GPIO_A"
+		(at 182.88 167.64 180)
+		(effects
+			(font
+				(size 1.27 1.27)
+			)
+			(justify right bottom)
+		)
+	)
 	(label "SENSELF_A"
 		(at 222.25 114.3 0)
@@
 	)
 	(label "DO_VDD"
-		(at 238.76 154.94 180)
+		(at 238.76 152.4 180)
 		(effects
 			(font
@@
 	)
 	(label "DO_VDD"
-		(at 238.76 185.42 180)
+		(at 238.76 182.88 180)
 		(effects
 			(font
@@
 	)
 	(label "DO_VDD"
-		(at 238.76 93.98 180)
+		(at 238.76 91.44 180)
 		(effects
 			(font
@@
 	)
 	(sheet
-		(at 241.3 123.19)
-		(size 25.4 25.4)
+		(at 241.3 120.65)
+		(size 25.4 27.94)
 		(exclude_from_sim no)
 		(in_bom yes)
@@
 		)
 		(property "Sheetname" "Front End Channel 2"
-			(at 241.3 122.4784 0)
+			(at 241.3 119.9384 0)
 			(effects
 				(font
@@
 		)
 		(pin "DO_VDD" bidirectional
+			(at 241.3 121.92 180)
+			(effects
+				(font
+					(size 1.27 1.27)
+				)
+				(justify left)
+			)
+		)
+		(pin "GPIO" bidirectional
 			(at 241.3 124.46 180)
 			(effects
@@
 	)
 	(sheet
-		(at 241.3 92.71)
-		(size 25.4 25.4)
+		(at 241.3 90.17)
+		(size 25.4 27.94)
 		(exclude_from_sim no)
 		(in_bom yes)
@@
 		)
 		(property "Sheetname" "Front End Channel 1"
-			(at 241.3 91.9984 0)
+			(at 241.3 89.4584 0)
 			(effects
 				(font
@@
 		)
 		(pin "DO_VDD" bidirectional
+			(at 241.3 91.44 180)
+			(effects
+				(font
+					(size 1.27 1.27)
+				)
+				(justify left)
+			)
+		)
+		(pin "GPIO" bidirectional
 			(at 241.3 93.98 180)
 			(effects
@@
 	)
 	(sheet
-		(at 241.3 184.15)
-		(size 25.4 25.4)
+		(at 241.3 181.61)
+		(size 25.4 27.94)
 		(exclude_from_sim no)
 		(in_bom yes)
@@
 		)
 		(property "Sheetname" "Front End Channel 4"
-			(at 241.3 183.4384 0)
+			(at 241.3 180.8984 0)
 			(effects
 				(font
@@
 		)
 		(pin "DO_VDD" bidirectional
+			(at 241.3 182.88 180)
+			(effects
+				(font
+					(size 1.27 1.27)
+				)
+				(justify left)
+			)
+		)
+		(pin "GPIO" bidirectional
 			(at 241.3 185.42 180)
 			(effects
@@
 	)
 	(sheet
-		(at 241.3 153.67)
-		(size 25.4 25.4)
+		(at 241.3 151.13)
+		(size 25.4 27.94)
 		(exclude_from_sim no)
 		(in_bom yes)
@@
 		)
 		(property "Sheetname" "Front End Channel 3"
-			(at 241.3 152.9584 0)
+			(at 241.3 150.4184 0)
 			(effects
 				(font
@@
 		)
 		(pin "DO_VDD" bidirectional
+			(at 241.3 152.4 180)
+			(effects
+				(font
+					(size 1.27 1.27)
+				)
+				(justify left)
+			)
+		)
+		(pin "GPIO" bidirectional
 			(at 241.3 154.94 180)
 			(effects
