File: minimal_ad74416h/minimal_ad74416h.kicad_sch (KiCad schematic)
At the start: 61 parts, among them U2 AD74416HBCPZ-RL7, U3 ADR4525BRZ

Commit message: backup
Parts:
- removed TP14, TP15: TestPoint, test_point_footprints:TestPoint_THTPad_Castelated, symbol UNITED_TEST_POINTS:TestPoint_Castelated
Changed lines of the file:
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@@
 	(wire
 		(pts
-			(xy 228.6 50.8) (xy 228.6 49.53)
-		)
-		(stroke
-			(width 0)
-			(type default)
-		)
-	)
-	(wire
-		(pts
 			(xy 219.71 97.79) (xy 219.71 100.33)
 		)
@@
 	(wire
 		(pts
-			(xy 228.6 49.53) (xy 226.06 49.53)
-		)
-		(stroke
-			(width 0)
-			(type default)
-		)
-	)
-	(wire
-		(pts
 			(xy 292.1 78.74) (xy 289.56 78.74)
 		)
@@
 	)
 	(symbol
-		(lib_id "UNITED_TEST_POINTS:TestPoint_Castelated")
-		(at 226.06 46.99 90)
-		(unit 1)
-		(exclude_from_sim no)
-		(in_bom yes)
-		(on_board yes)
-		(dnp no)
-		(property "Reference" "TP14"
-			(at 220.98 46.9899 90)
-			(effects
-				(font
-					(size 1.27 1.27)
-				)
-				(justify left)
-			)
-		)
-		(property "Value" "TestPoint"
-			(at 223.52 44.45 0)
-			(effects
-				(font
-					(size 1.27 1.27)
-				)
-				(justify left)
-				(hide yes)
-			)
-		)
-		(property "Footprint" "test_point_footprints:TestPoint_THTPad_Castelated"
-			(at 231.14 44.45 0)
-			(effects
-				(font
-					(size 1.27 1.27)
-				)
-				(justify left)
-				(hide yes)
-			)
-		)
-		(property "Datasheet" "~"
-			(at 226.06 44.45 0)
-			(effects
-				(font
-					(size 1.27 1.27)
-				)
-				(justify left)
-				(hide yes)
-			)
-		)
-		(property "Description" "test point"
-			(at 228.6 44.45 0)
-			(effects
-				(font
-					(size 1.27 1.27)
-				)
-				(justify left)
-				(hide yes)
-			)
-		)
-		(pin "1"
-		)
-		(instances
-			(project "minimal_ad74416h"
-				(path "/996c4afa-af57-455f-b0b6-e0f996045a90"
-					(reference "TP14")
-					(unit 1)
-				)
-			)
-		)
-	)
-	(symbol
 		(lib_id "UNITED_NO_COMPONENTS_DATA_BASE:Fiducial")
 		(at 25.4 279.4 0)
@@
 	)
 	(symbol
-		(lib_id "power:GNDA")
-		(at 228.6 50.8 0)
-		(unit 1)
-		(exclude_from_sim no)
-		(in_bom yes)
-		(on_board yes)
-		(dnp no)
-		(property "Reference" "#PWR056"
-			(at 228.6 57.15 0)
-			(effects
-				(font
-					(size 1.27 1.27)
-				)
-				(hide yes)
-			)
-		)
-		(property "Value" "GNDA"
-			(at 226.06 52.0699 0)
-			(effects
-				(font
-					(size 1.27 1.27)
-				)
-				(justify right)
-			)
-		)
-		(property "Footprint" ""
-			(at 228.6 50.8 0)
-			(effects
-				(font
-					(size 1.27 1.27)
-				)
-				(hide yes)
-			)
-		)
-		(property "Datasheet" ""
-			(at 228.6 50.8 0)
-			(effects
-				(font
-					(size 1.27 1.27)
-				)
-				(hide yes)
-			)
-		)
-		(property "Description" "Power symbol creates a global label with name \"GNDA\" , analog ground"
-			(at 228.6 50.8 0)
-			(effects
-				(font
-					(size 1.27 1.27)
-				)
-				(hide yes)
-			)
-		)
-		(pin "1"
-		)
-		(instances
-			(project "minimal_ad74416h"
-				(path "/996c4afa-af57-455f-b0b6-e0f996045a90"
-					(reference "#PWR056")
-					(unit 1)
-				)
-			)
-		)
-	)
-	(symbol
 		(lib_id "UNITED_TEST_POINTS:TestPoint_Castelated")
 		(at 381 134.62 270)
@@
 					(unit 1)
 				)
-			)
-		)
-	)
-	(symbol
-		(lib_id "UNITED_TEST_POINTS:TestPoint_Castelated")
-		(at 226.06 49.53 90)
-		(unit 1)
-		(exclude_from_sim no)
-		(in_bom yes)
-		(on_board yes)
-		(dnp no)
-		(property "Reference" "TP15"
-			(at 220.98 49.5299 90)
-			(effects
-				(font
-					(size 1.27 1.27)
-				)
-				(justify left)
-			)
-		)
-		(property "Value" "TestPoint"
-			(at 223.52 46.99 0)
-			(effects
-				(font
-					(size 1.27 1.27)
-				)
-				(justify left)
-				(hide yes)
-			)
-		)
-		(property "Footprint" "test_point_footprints:TestPoint_THTPad_Castelated"
-			(at 231.14 46.99 0)
-			(effects
-				(font
-					(size 1.27 1.27)
-				)
-				(justify left)
-				(hide yes)
-			)
-		)
-		(property "Datasheet" "~"
-			(at 226.06 46.99 0)
-			(effects
-				(font
-					(size 1.27 1.27)
-				)
-				(justify left)
-				(hide yes)
-			)
-		)
-		(property "Description" "test point"
-			(at 228.6 46.99 0)
-			(effects
-				(font
-					(size 1.27 1.27)
-				)
-				(justify left)
-				(hide yes)
-			)
-		)
-		(pin "1"
-		)
-		(instances
-			(project "minimal_ad74416h"
-				(path "/996c4afa-af57-455f-b0b6-e0f996045a90"
-					(reference "TP15")
-					(unit 1)
-				)

Commit message: backup
Parts:
- renumbered FID2 to FID1, FID1 to FID2, TP6 to TP1, TP17 to TP10, TP18 to TP11, TP19 to TP12, TP20 to TP13, TP21 to TP14, TP22 to TP15, TP23 to TP16, TP24 to TP17, TP25 to TP18, TP7 to TP2, TP8 to TP3, TP9 to TP4, TP10 to TP5, TP11 to TP6, TP12 to TP7, TP13 to TP8, TP16 to TP9
Other:
- sheet Power Supply and Digital Interface ports: added ~{ADC_RDY}; removed none
Changed lines of the file:
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@@
 	(wire
 		(pts
+			(xy 152.4 106.68) (xy 160.02 106.68)
+		)
+		(stroke
+			(width 0)
+			(type default)
+		)
+	)
+	(wire
+		(pts
 			(xy 245.11 127) (xy 243.84 127)
 		)
@@
 		)
 	)
+	(label "~{ADC_RDY}"
+		(at 160.02 106.68 0)
+		(effects
+			(font
+				(size 1.27 1.27)
+			)
+			(justify left bottom)
+		)
+	)
 	(label "SCLK"
 		(at 160.02 96.52 0)
@@
 		(on_board yes)
 		(dnp no)
-		(property "Reference" "TP25"
+		(property "Reference" "TP18"
 			(at 220.98 38.0999 90)
 			(effects
@@
 			(project "minimal_ad74416h"
 				(path "/996c4afa-af57-455f-b0b6-e0f996045a90"
-					(reference "TP25")
+					(reference "TP18")
 					(unit 1)
 				)
@@
 		(on_board yes)
 		(dnp no)
-		(property "Reference" "TP11"
+		(property "Reference" "TP6"
 			(at 386.08 193.0399 90)
 			(effects
@@
 			(project "minimal_ad74416h"
 				(path "/996c4afa-af57-455f-b0b6-e0f996045a90"
-					(reference "TP11")
+					(reference "TP6")
 					(unit 1)
 				)
@@
 		(dnp no)
 		(fields_autoplaced yes)
-		(property "Reference" "FID1"
+		(property "Reference" "FID2"
 			(at 40.64 278.1299 0)
 			(effects
@@
 			(project "minimal_ad74416h"
 				(path "/996c4afa-af57-455f-b0b6-e0f996045a90"
-					(reference "FID1")
+					(reference "FID2")
 					(unit 1)
 				)
@@
 		(on_board yes)
 		(dnp no)
-		(property "Reference" "TP7"
+		(property "Reference" "TP2"
 			(at 386.08 195.5799 90)
 			(effects
@@
 			(project "minimal_ad74416h"
 				(path "/996c4afa-af57-455f-b0b6-e0f996045a90"
-					(reference "TP7")
+					(reference "TP2")
 					(unit 1)
 				)
@@
 		(on_board yes)
 		(dnp no)
-		(property "Reference" "TP21"
+		(property "Reference" "TP14"
 			(at 386.08 167.6399 90)
 			(effects
@@
 			(project "minimal_ad74416h"
 				(path "/996c4afa-af57-455f-b0b6-e0f996045a90"
-					(reference "TP21")
+					(reference "TP14")
 					(unit 1)
 				)
@@
 		(on_board yes)
 		(dnp no)
-		(property "Reference" "TP10"
+		(property "Reference" "TP5"
 			(at 386.08 101.5999 90)
 			(effects
@@
 			(project "minimal_ad74416h"
 				(path "/996c4afa-af57-455f-b0b6-e0f996045a90"
-					(reference "TP10")
+					(reference "TP5")
 					(unit 1)
 				)
@@
 		(on_board yes)
 		(dnp no)
-		(property "Reference" "TP20"
+		(property "Reference" "TP13"
 			(at 386.08 137.1599 90)
 			(effects
@@
 			(project "minimal_ad74416h"
 				(path "/996c4afa-af57-455f-b0b6-e0f996045a90"
-					(reference "TP20")
+					(reference "TP13")
 					(unit 1)
 				)
@@
 		(on_board yes)
 		(dnp no)
-		(property "Reference" "TP19"
+		(property "Reference" "TP12"
 			(at 386.08 162.5599 90)
 			(effects
@@
 			(project "minimal_ad74416h"
 				(path "/996c4afa-af57-455f-b0b6-e0f996045a90"
-					(reference "TP19")
+					(reference "TP12")
 					(unit 1)
 				)
@@
 		(on_board yes)
 		(dnp no)
-		(property "Reference" "TP9"
+		(property "Reference" "TP4"
 			(at 386.08 198.1199 90)
 			(effects
@@
 			(project "minimal_ad74416h"
 				(path "/996c4afa-af57-455f-b0b6-e0f996045a90"
-					(reference "TP9")
+					(reference "TP4")
 					(unit 1)
 				)
@@
 		(on_board yes)
 		(dnp no)
-		(property "Reference" "TP8"
+		(property "Reference" "TP3"
 			(at 386.08 106.6799 90)
 			(effects
@@
 			(project "minimal_ad74416h"
 				(path "/996c4afa-af57-455f-b0b6-e0f996045a90"
-					(reference "TP8")
+					(reference "TP3")
 					(unit 1)
 				)
@@
 		(dnp no)
 		(fields_autoplaced yes)
-		(property "Reference" "FID2"
+		(property "Reference" "FID1"
 			(at 53.34 278.1299 0)
 			(effects
@@
 			(project "minimal_ad74416h"
 				(path "/996c4afa-af57-455f-b0b6-e0f996045a90"
-					(reference "FID2")
+					(reference "FID1")
 					(unit 1)
 				)
@@
 		(on_board yes)
 		(dnp no)
-		(property "Reference" "TP17"
+		(property "Reference" "TP10"
 			(at 386.08 170.1799 90)
 			(effects
@@
 			(project "minimal_ad74416h"
 				(path "/996c4afa-af57-455f-b0b6-e0f996045a90"
-					(reference "TP17")
+					(reference "TP10")
 					(unit 1)
 				)
@@
 		(on_board yes)
 		(dnp no)
-		(property "Reference" "TP24"
+		(property "Reference" "TP17"
 			(at 220.98 35.5599 90)
 			(effects
@@
 			(project "minimal_ad74416h"
 				(path "/996c4afa-af57-455f-b0b6-e0f996045a90"
-					(reference "TP24")
+					(reference "TP17")
 					(unit 1)
 				)
@@
 		(on_board yes)
 		(dnp no)
-		(property "Reference" "TP18"
+		(property "Reference" "TP11"
 			(at 386.08 132.0799 90)
 			(effects
@@
 			(project "minimal_ad74416h"
 				(path "/996c4afa-af57-455f-b0b6-e0f996045a90"
-					(reference "TP18")
+					(reference "TP11")
 					(unit 1)
 				)
@@
 		(on_board yes)
 		(dnp no)
-		(property "Reference" "TP13"
+		(property "Reference" "TP8"
 			(at 386.08 200.6599 90)
 			(effects
@@
 			(project "minimal_ad74416h"
 				(path "/996c4afa-af57-455f-b0b6-e0f996045a90"
-					(reference "TP13")
+					(reference "TP8")
 					(unit 1)
 				)
@@
 		(on_board yes)
 		(dnp no)
-		(property "Reference" "TP22"
+		(property "Reference" "TP15"
 			(at 386.08 134.6199 90)
 			(effects
@@
 			(project "minimal_ad74416h"
 				(path "/996c4afa-af57-455f-b0b6-e0f996045a90"
-					(reference "TP22")
+					(reference "TP15")
 					(unit 1)
 				)
@@
 		(on_board yes)
 		(dnp no)
-		(property "Reference" "TP12"
+		(property "Reference" "TP7"
 			(at 386.08 109.2199 90)
 			(effects
@@
 			(project "minimal_ad74416h"
 				(path "/996c4afa-af57-455f-b0b6-e0f996045a90"
-					(reference "TP12")
+					(reference "TP7")
 					(unit 1)
 				)
@@
 		(on_board yes)
 		(dnp no)
-		(property "Reference" "TP23"
+		(property "Reference" "TP16"
 			(at 386.08 165.0999 90)
 			(effects
@@
 			(project "minimal_ad74416h"
 				(path "/996c4afa-af57-455f-b0b6-e0f996045a90"
-					(reference "TP23")
+					(reference "TP16")
 					(unit 1)
 				)
@@
 		(on_board yes)
 		(dnp no)
-		(property "Reference" "TP16"
+		(property "Reference" "TP9"
 			(at 386.08 139.6999 90)
 			(effects
@@
 			(project "minimal_ad74416h"
 				(path "/996c4afa-af57-455f-b0b6-e0f996045a90"
-					(reference "TP16")
+					(reference "TP9")
 					(unit 1)
 				)
@@
 		(on_board yes)
 		(dnp no)
-		(property "Reference" "TP6"
+		(property "Reference" "TP1"
 			(at 386.08 104.1399 90)
 			(effects
@@
 			(project "minimal_ad74416h"
 				(path "/996c4afa-af57-455f-b0b6-e0f996045a90"
-					(reference "TP6")
+					(reference "TP1")
 					(unit 1)
 				)
@@
 			(effects
 				(font
+					(size 1.27 1.27)
+				)
+				(justify right)
+			)
+		)
+		(pin "~{ADC_RDY}" input
+			(at 152.4 106.68 0)
+			(effects
+				(font

Commit message: backup
Other:
- sheet Power Supply and Digital Interface ports: added 14V5; removed MAX17570_VOUT
Changed lines of the file:
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@@
 			)
 		)
-		(pin "MAX17570_VOUT" output
-			(at 152.4 66.04 0)
+		(pin "~{ADC_RDY}" input
+			(at 152.4 106.68 0)
 			(effects
 				(font
@@
 			)
 		)
-		(pin "~{ADC_RDY}" input
-			(at 152.4 106.68 0)
+		(pin "14V5" output
+			(at 152.4 66.04 0)
 			(effects
 				(font

Commit message: backup
Parts:
- added TP19, TP20, TP21, TP22, TP23, TP24, TP26, TP27, TP29, TP30, TP32, TP33, TP35, TP36, TP38, TP39, TP41, TP42, TP44, TP45: TestPoint, test_point_footprints:TestPoint_THTPad_Castelated, symbol UNITED_TEST_POINTS:TestPoint_Castelated
Connections:
- net VDD_24V renamed 24V0
- new net GND: TP20.1
- new net GNDD: TP22.1
- new net GPIO_A_ISO: TP38.1
- new net GPIO_B_ISO: TP39.1
- new net GPIO_C_ISO: TP45.1
- new net GPIO_D_ISO: TP44.1
- new net GPIO_E_ISO: TP41.1
- new net GPIO_F_ISO: TP42.1
- new net MGPI1: TP24.1
- new net MVDD: TP21.1
- new net PWRGD: TP23.1
- new net SCLK_ISO: TP30.1
- new net SDI_ISO: TP29.1
- new net SDO_ISO: TP32.1
- new net VINP: TP19.1
- new net ~{ADC_RDY_ISO}: TP35.1
- new net ~{ALERT_ISO}: TP27.1
- new net ~{MAX17570_RESET_ISO}: TP36.1
- new net ~{RESET_ISO}: TP26.1
- new net ~{SYNC_ISO}: TP33.1
Other:
- sheet Power Supply and Digital Interface ports: added 24V0, GPIO_A_ISO, GPIO_B_ISO, GPIO_C_ISO, GPIO_D_ISO, GPIO_E_ISO, GPIO_F_ISO, MGPI1, MVDD, PWRGD, SCLK_ISO, SDI_ISO, SDO_ISO, VINP, ~{ADC_RDY_ISO}, ~{ALERT_ISO}, ~{MAX17570_RESET_ISO}, ~{RESET_ISO}, ~{SYNC_ISO}; removed VDD_24V

Commit message: backup
Other:
- sheet Power Supply and Digital Interface ports: added DO_VDD; removed none
Changed lines of the file:
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@@
 	(wire
 		(pts
-			(xy 160.02 124.46) (xy 167.64 124.46)
+			(xy 160.02 129.54) (xy 167.64 129.54)
 		)
 		(stroke
@@
 	(wire
 		(pts
-			(xy 160.02 116.84) (xy 167.64 116.84)
+			(xy 160.02 121.92) (xy 167.64 121.92)
 		)
 		(stroke
@@
 	(wire
 		(pts
-			(xy 160.02 121.92) (xy 167.64 121.92)
+			(xy 160.02 127) (xy 167.64 127)
 		)
 		(stroke
@@
 	(wire
 		(pts
-			(xy 160.02 119.38) (xy 167.64 119.38)
+			(xy 160.02 124.46) (xy 167.64 124.46)
 		)
 		(stroke
@@
 	(wire
 		(pts
+			(xy 160.02 119.38) (xy 167.64 119.38)
+		)
+		(stroke
+			(width 0)
+			(type default)
+		)
+	)
+	(wire
+		(pts
 			(xy 322.58 160.02) (xy 342.9 160.02)
 		)
@@
 	)
 	(label "5V0"
-		(at 167.64 121.92 0)
+		(at 167.64 127 0)
 		(effects
 			(font
@@
 	)
 	(label "-15V0"
-		(at 167.64 124.46 0)
+		(at 167.64 129.54 0)
 		(effects
 			(font
@@
 		)
 	)
+	(label "DO_VDD"
+		(at 167.64 119.38 0)
+		(effects
+			(font
+				(size 1.27 1.27)
+			)
+			(justify left bottom)
+		)
+	)
 	(label "VIOUT_A"
 		(at 323.85 109.22 0)
@@
 	)
 	(label "AVDD_LO"
-		(at 167.64 119.38 0)
+		(at 167.64 124.46 0)
 		(effects
 			(font
@@
 	)
 	(label "24V0"
-		(at 167.64 116.84 0)
+		(at 167.64 121.92 0)
 		(effects
 			(font
@@
 		)
 		(pin "-15V0" output
-			(at 160.02 124.46 0)
+			(at 160.02 129.54 0)
 			(effects
 				(font
@@
 		)
 		(pin "5V0" output
-			(at 160.02 121.92 0)
+			(at 160.02 127 0)
 			(effects
 				(font
@@
 		)
 		(pin "24V0" output
-			(at 160.02 116.84 0)
+			(at 160.02 121.92 0)
 			(effects
 				(font
@@
 		)
 		(pin "14V5" output
-			(at 160.02 119.38 0)
+			(at 160.02 124.46 0)
 			(effects
 				(font
@@
 			)
 		)
+		(pin "DO_VDD" output
+			(at 160.02 119.38 0)
+			(effects
+				(font
+					(size 1.27 1.27)
+				)
+				(justify right)
+			)
+		)

Commit message: backup
Parts:
- added R73, R74, R75: 100 kΩ, resistor_footprints:R_0402_1005Metric, symbol UNITED_RESISTORS_DATA_BASE:R_ERJ-2GEJ104X
Connections:
- net GNDA: now also R74.2, R75.2
- net SCLK: now also R73.2
- net SDI: now also R74.1
- net SDO: now also R75.1
- new net VOUT2: R73.1
Other:
- sheet Power Supply and Digital Interface ports: added {DIGITAL_INTERFACE}; removed GPIO_A, GPIO_B, GPIO_C, GPIO_D, GPIO_E, GPIO_F, SCLK, SDI, SDO, ~{ADC_RDY}, ~{ALERT}, ~{RESET}, ~{SYNC}
- moved on the sheet: D1, D2, D20, D21, D22, D23, R10, R20, R21, R22, R55, R56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

Commit message: backup
Parts:
- removed R73, R74, R75: 100 kΩ, resistor_footprints:R_0402_1005Metric, symbol UNITED_RESISTORS_DATA_BASE:R_ERJ-2GEJ104X
- added R61, R62: 10 kΩ, resistor_footprints:R_0402_1005Metric, symbol UNITED_RESISTORS_DATA_BASE:R_ERJ-2RKF1002X
Connections:
- net 5V0: now also R61.1, R62.1
- net AD0: now also R62.2
- net AD1: now also R61.2
- net AVDD_LO renamed 14V5
Other:
- sheet Power Supply and Digital Interface ports: added {POWER_BUS}; removed -15V0, 14V5, 24V0, 5V0, DO_VDD
- moved on the sheet: C18, C19, C20, C21, C24, C31, C32, C33, C34, C35, C36, C37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

Commit message: backup
Connections:
- net DO_VDD: now also C35.1; no longer C35.2
- net GNDA: now also C35.2, C8.2; no longer C35.1, C8.1
- net LDO1V8: now also C8.1; no longer C8.2
Other:
- sheet Power Supply and Digital Interface ports: added {DIGITAL_INTERFACE_INPUT}, {POWER_BUS_INPUT}; removed GPIO_A_ISO, GPIO_B_ISO, GPIO_C_ISO, GPIO_D_ISO, GPIO_E_ISO, GPIO_F_ISO, MGPI1, MVDD, PWRGD, SCLK_ISO, SDI_ISO, SDO_ISO, VINP, ~{ADC_RDY_ISO}, ~{ALERT_ISO}, ~{MAX17570_RESET_ISO}, ~{RESET_ISO}, ~{SYNC_ISO}
- moved on the sheet: C18, C19, C20, C21, C31, C32, C33, C34, C35, C7, C8, C9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
