File: minimal_ad74416h/minimal_ad74416h.kicad_sch (KiCad schematic)
At the start: 81 parts, among them U2 AD74416HBCPZ-RL7, U3 ADR4525BRZ

Commit message: backup
Parts:
- removed TP35, TP36, TP38, TP39, TP41, TP42, TP44, TP45: TestPoint, test_point_footprints:TestPoint_THTPad_Castelated, symbol UNITED_TEST_POINTS:TestPoint_Castelated
- renumbered C38 to C37, C37 to C38, D22 to D24, D23 to D25, R61 to R13, R62 to R14, R20 to R22, R21 to R23, R22 to R24, R54 to R56, R55 to R57, R56 to R58, R59 to R69, R60 to R73, TP5 to TP1, TP13 to TP11, TP14 to TP12, TP15 to TP13, TP16 to TP14, TP11 to TP15, TP12 to TP16, TP6 to TP2, TP1 to TP3, TP2 to TP4, TP3 to TP5, TP4 to TP6

Commit message: backup
Parts:
- added TP35, TP36: TestPoint, test_point_footprints:TestPoint_THTPad_Castelated, symbol UNITED_TEST_POINTS:TestPoint_Castelated
Connections:
- new net SCL_ISO: TP35.1
- new net SDA_ISO: TP36.1
Changed lines of the file:
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@@
 	)
 	(bus_entry
+		(at 88.9 187.96)
+		(size -2.54 2.54)
+		(stroke
+			(width 0)
+			(type default)
+		)
+	)
+	(bus_entry
 		(at 88.9 170.18)
 		(size -2.54 2.54)
@@
 	)
 	(bus_entry
+		(at 88.9 190.5)
+		(size -2.54 2.54)
+		(stroke
+			(width 0)
+			(type default)
+		)
+	)
+	(bus_entry
 		(at 271.78 187.96)
 		(size 2.54 -2.54)
@@
 		)
 	)
+	(bus
+		(pts
+			(xy 88.9 187.96) (xy 88.9 190.5)
+		)
+		(stroke
+			(width 0)
+			(type default)
+		)
+	)
 	(wire
 		(pts
@@
 	(wire
 		(pts
+			(xy 60.96 193.04) (xy 86.36 193.04)
+		)
+		(stroke
+			(width 0)
+			(type default)
+		)
+	)
+	(wire
+		(pts
 			(xy 274.32 182.88) (xy 287.02 182.88)
 		)
@@
 		)
 	)
+	(bus
+		(pts
+			(xy 88.9 185.42) (xy 88.9 187.96)
+		)
+		(stroke
+			(width 0)
+			(type default)
+		)
+	)
 	(wire
 		(pts
@@
 	(wire
 		(pts
+			(xy 60.96 190.5) (xy 86.36 190.5)
+		)
+		(stroke
+			(width 0)
+			(type default)
+		)
+	)
+	(wire
+		(pts
 			(xy 205.74 50.8) (xy 292.1 50.8)
 		)
@@
 		)
 	)
+	(label "SCL_ISO"
+		(at 83.82 190.5 180)
+		(effects
+			(font
+				(size 1.27 1.27)
+			)
+			(justify right bottom)
+		)
+	)
 	(label "VIOUT_B"
 		(at 328.93 149.86 0)
@@
 		)
 	)
+	(label "SDA_ISO"
+		(at 83.82 193.04 180)
+		(effects
+			(font
+				(size 1.27 1.27)
+			)
+			(justify right bottom)
+		)
+	)
 	(label "SENSELF_A"
 		(at 328.93 124.46 0)
@@
 	)
 	(symbol
+		(lib_id "UNITED_TEST_POINTS:TestPoint_Castelated")
+		(at 60.96 193.04 90)
+		(unit 1)
+		(exclude_from_sim no)
+		(in_bom yes)
+		(on_board yes)
+		(dnp no)
+		(property "Reference" "TP36"
+			(at 55.88 193.0399 90)
+			(effects
+				(font
+					(size 1.27 1.27)
+				)
+				(justify left)
+			)
+		)
+		(property "Value" "TestPoint"
+			(at 58.42 190.5 0)
+			(effects
+				(font
+					(size 1.27 1.27)
+				)
+				(justify left)
+				(hide yes)
+			)
+		)
+		(property "Footprint" "test_point_footprints:TestPoint_THTPad_Castelated"
+			(at 66.04 190.5 0)
+			(effects
+				(font
+					(size 1.27 1.27)
+				)
+				(justify left)
+				(hide yes)
+			)
+		)
+		(property "Datasheet" "~"
+			(at 60.96 190.5 0)
+			(effects
+				(font
+					(size 1.27 1.27)
+				)
+				(justify left)
+				(hide yes)
+			)
+		)
+		(property "Description" "test point"
+			(at 63.5 190.5 0)
+			(effects
+				(font
+					(size 1.27 1.27)
+				)
+				(justify left)
+				(hide yes)
+			)
+		)
+		(pin "1"
+		)
+		(instances
+			(project "minimal_ad74416h"
+				(path "/996c4afa-af57-455f-b0b6-e0f996045a90"
+					(reference "TP36")
+					(unit 1)
+				)
+			)
+		)
+	)
+	(symbol
 		(lib_id "power:GNDA")
 		(at 281.94 76.2 0)
@@
 					(unit 1)
 				)
+			)
+		)
+	)
+	(symbol
+		(lib_id "UNITED_TEST_POINTS:TestPoint_Castelated")
+		(at 60.96 190.5 90)
+		(unit 1)
+		(exclude_from_sim no)
+		(in_bom yes)
+		(on_board yes)
+		(dnp no)
+		(property "Reference" "TP35"
+			(at 55.88 190.4999 90)
+			(effects
+				(font
+					(size 1.27 1.27)
+				)
+				(justify left)
+			)
+		)
+		(property "Value" "TestPoint"
+			(at 58.42 187.96 0)
+			(effects
+				(font
+					(size 1.27 1.27)
+				)
+				(justify left)
+				(hide yes)
+			)
+		)
+		(property "Footprint" "test_point_footprints:TestPoint_THTPad_Castelated"
+			(at 66.04 187.96 0)
+			(effects
+				(font
+					(size 1.27 1.27)
+				)
+				(justify left)
+				(hide yes)
+			)
+		)
+		(property "Datasheet" "~"
+			(at 60.96 187.96 0)
+			(effects
+				(font
+					(size 1.27 1.27)
+				)
+				(justify left)
+				(hide yes)
+			)
+		)
+		(property "Description" "test point"
+			(at 63.5 187.96 0)
+			(effects
+				(font
+					(size 1.27 1.27)
+				)
+				(justify left)
+				(hide yes)
+			)
+		)
+		(pin "1"
+		)
+		(instances
+			(project "minimal_ad74416h"
+				(path "/996c4afa-af57-455f-b0b6-e0f996045a90"
+					(reference "TP35")
+					(unit 1)
+				)

Commit message: backup
Connections:
- net AD0: now also S3.4; no longer S3.3
- net AD1: now also S3.3; no longer S3.4
Changed lines of the file:
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@@
 	(bus_alias "DIGITAL_INTERFACE"
 		(members "GPIO_A" "GPIO_B" "GPIO_C" "GPIO_D" "GPIO_E" "GPIO_F" "~{ADC_RDY}"
-			"~{ALERT}" "~{RESET}" "SDO" "SDI" "SCLK" "~{SYNC}" "SGPO1" "~{MAX17570_RESET}"
+			"~{ALERT}" "~{RESET}" "SDO" "SDI" "SCLK" "~{SYNC}"
 		)
 	)
@@
 		)
 	)
-	(label "GPIO_A"
-		(at 375.92 109.22 0)
-		(effects
-			(font
-				(size 1.27 1.27)
-			)
-			(justify left bottom)
-		)
-	)
 	(label "-15V0"
 		(at 320.04 238.76 0)
@@
 		)
 	)
-	(label "GPIO_D"
-		(at 375.92 200.66 0)
-		(effects
-			(font
-				(size 1.27 1.27)
-			)
-			(justify left bottom)
-		)
-	)
 	(label "GPIO_F"
 		(at 284.48 205.74 180)
@@
 		)
 	)
-	(label "GPIO_C"
-		(at 375.92 170.18 0)
-		(effects
-			(font
-				(size 1.27 1.27)
-			)
-			(justify left bottom)
-		)
-	)
 	(label "DO_SRC_GATE_A"
 		(at 328.93 109.22 0)
@@
 		)
 	)
-	(label "GPIO_B"
-		(at 375.92 139.7 0)
-		(effects
-			(font
-				(size 1.27 1.27)
-			)
-			(justify left bottom)
-		)
-	)
 	(label "REFIO"
 		(at 256.54 106.68 0)
@@
 		(lib_id "UNITED_DIP_SWITCHES_DATA_BASE:S_416131160802")
 		(at 254 156.21 0)
+		(mirror x)
 		(unit 1)
 		(exclude_from_sim no)
@@
 		(fields_autoplaced yes)
 		(property "Reference" "S3"
-			(at 254 148.59 0)
+			(at 254 149.86 0)
 			(effects
 				(font
@@
 		)
 		(property "Value" "416131160802"
-			(at 254 151.13 0)
+			(at 254 152.4 0)
 			(effects
 				(font
@@
 		)
 		(property "Footprint" "dip_switches_footprints:416131160802"
-			(at 254 162.56 0)
+			(at 254 149.86 0)
 			(show_name yes)
 			(effects
@@
 		)
 		(property "Datasheet" "https://www.we-online.com/components/products/datasheet/416131160802.pdf"
-			(at 254 165.1 0)
+			(at 254 147.32 0)
 			(show_name yes)
 			(effects
@@
 		)
 		(property "Description" "Wurth Elektronik Vertical mounting,  Surface Mount,"
-			(at 254 167.64 0)
+			(at 254 144.78 0)
 			(show_name yes)
 			(effects
@@
 		)
 		(property "MPN" "416131160802"
-			(at 254 170.18 0)
+			(at 254 142.24 0)
 			(show_name yes)
 			(effects
@@
 		)
 		(property "Manufacturer" "Wurth Elektronik"
-			(at 254 172.72 0)
+			(at 254 139.7 0)
 			(show_name yes)
 			(effects
@@
 		)
 		(property "Mounting Angle" "Vertical"
-			(at 254 175.26 0)
+			(at 254 137.16 0)
 			(show_name yes)
 			(effects
@@
 		)
 		(property "Mounting Style" "Surface Mount"
-			(at 254 177.8 0)
+			(at 254 134.62 0)
 			(show_name yes)
 			(effects
@@
 		)
 		(property "Number of Rows" "2"
-			(at 254 180.34 0)
+			(at 254 132.08 0)
 			(show_name yes)
 			(effects
@@
 		)
 		(property "Pin Count" "2"
-			(at 254 182.88 0)
+			(at 254 129.54 0)
 			(show_name yes)
 			(effects
@@
 		)
 		(property "Series" "416131160802"
-			(at 254 185.42 0)
+			(at 254 127 0)
 			(show_name yes)
 			(effects
@@
 		)
 		(property "Symbol Name" "S_416131160802"
-			(at 254 187.96 0)
+			(at 254 124.46 0)
 			(show_name yes)
 			(effects
@@
 		)
 		(property "Trustedparts Search" "https://www.trustedparts.com/en/search/416131160802"
-			(at 254 190.5 0)
+			(at 254 121.92 0)
 			(show_name yes)
 			(effects

Commit message: backup
Parts:
- removed S4: TS21-34-035-BK-160-SMT-TR, tactile_switches_footprints:TS21, symbol UNITED_TACTILE_SWITCHES_DATA_BASE:S_TS21-34-035-BK-160-SMT-TR
- removed TP24, TP26, TP27: TestPoint, test_point_footprints:TestPoint_THTPad_Castelated, symbol UNITED_TEST_POINTS:TestPoint_Castelated
- added TP17, TP18, TP19, TP20, TP21, TP22, TP36, TP37, TP38, TP39, TP40, TP41: TestPoint, test_point_footprints:TestPoint_THTPad_Castelated, symbol UNITED_TEST_POINTS:TestPoint_Castelated_v2
- renumbered C7 to C1, C18 to C12, C19 to C13, C20 to C14, C21 to C15, C24 to C18, C8 to C2, C31 to C25, C32 to C26, C33 to C27, C34 to C28, C35 to C29, C9 to C3, C36 to C30, C37 to C31, C38 to C32, D20 to D2, D21 to D3, D2 to D4, D24 to D5, D25 to D6, D3 to D9, R13 to R11, R14 to R12, R22 to R15, R23 to R18, R24 to R21, R9 to R3, R57 to R4, R58 to R5, R10 to R6, R69 to R7, R73 to R8, S3 to S1, TP17 to TP23, TP18 to TP24, TP19 to TP25, TP20 to TP26, TP21 to TP27, TP22 to TP28, TP23 to TP29, TP29 to TP30, TP30 to TP31, TP35 to TP34, TP36 to TP35, U2 to U1, U3 to U2
Connections:
- net -15V0: now also TP40.1
- net 24V0: now also TP36.1
- net 5V0: now also TP38.1
- net GNDA: now also TP37.1, TP39.1, TP41.1
- net SCLK: now also TP20.1
- net SDI: now also TP19.1
- net SDO: now also TP18.1
- net ~{SYNC}: now also TP17.1
- new net SCL: TP21.1
- new net SDA: TP22.1
Other:
- moved on the sheet: D1, D2, D3, D4, D5, D6, R15, R18, R21, R3, R4, R5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

Commit message: backup
Parts:
- added TP42, TP43: TestPoint, test_point_footprints:TestPoint_THTPad_Castelated, symbol UNITED_TEST_POINTS:TestPoint_Castelated_v2
Connections:
- net 14V5: now also TP42.1
- net GNDA: now also TP43.1
Other:
- moved on the sheet: TP36, TP37, TP38, TP39, TP40, TP41

Commit message: backup
Parts:
- removed C1, C12, C15, C27, C28: 10 µF, capacitor_footprints:C_0805_125_2012Metric, symbol UNITED_CAPACITORS_DATA_BASE:C_GRM21BR61H106KE43L
- removed C13, C14, C25, C26, C3, C32: 100 nF, capacitor_footprints:C_0402_1005Metric, symbol UNITED_CAPACITORS_DATA_BASE:C_GCM155R71H104KE02D
- removed C18: 39 nF, capacitor_footprints:C_0402_1005Metric, symbol UNITED_CAPACITORS_DATA_BASE:C_KGM05AR71C393KH
- removed C2: 2.2 µF, capacitor_footprints:C_0805_2012Metric, symbol UNITED_CAPACITORS_DATA_BASE:C_CGA4J1X7R1V225K125AC
- removed C29: 10 µF, capacitor_footprints:C_1210_250_3225Metric, symbol UNITED_CAPACITORS_DATA_BASE:C_GRM32EC72A106KE05L
- removed C30: 2.2 µF, capacitor_footprints:C_0603_1608Metric, symbol UNITED_CAPACITORS_DATA_BASE:C_C1608X7S1A225K080AC
- removed C31: 1 µF, capacitor_footprints:C_0805_2012Metric, symbol UNITED_CAPACITORS_DATA_BASE:C_GRJ21BC72A105KE11L
- removed D1, D2, D3, D4, D5, D6: 1.8 V, diode_footprints:LED_GREEN_0402_1005Metric, symbol UNITED_DIODES_DATA_BASE:D_APHHS1005CGCK
- removed D9: 100.0 V, diode_footprints:SOD_523, symbol UNITED_DIODES_DATA_BASE:D_BAT41KFILM
- removed R11, R12, R15, R18, R21, R3, R4, R5, R6, R7, R8: 10 kΩ, resistor_footprints:R_0402_1005Metric, symbol UNITED_RESISTORS_DATA_BASE:R_ERJ-2RKF1002X
- removed R56: 33 kΩ, resistor_footprints:R_0805_2012Metric, symbol UNITED_RESISTORS_DATA_BASE:R_ERJ-6ENF3302V
- removed RT1: 33 kΩ, resistor_footprints:RT_0805_RT_2012Metric, symbol UNITED_RESISTORS_DATA_BASE:RT_NTCS0805E3333JHT
- removed S1: 416131160802, dip_switches_footprints:416131160802, symbol UNITED_DIP_SWITCHES_DATA_BASE:S_416131160802
- removed U1: AD74416HBCPZ-RL7, analog_devices_footprints:CP-64-15_ADI, symbol UNITED_IC_ADI:U_AD74416HBCPZ-RL7
- removed U2: ADR4525BRZ, analog_devices_footprints:R_8_ADI, symbol UNITED_IC_ADI:U_ADR4525BRZ
Other:
- added sheet AD74416H (AD74416H.kicad_sch)
- moved on the sheet: TP1, TP10, TP11, TP12, TP13, TP14, TP15, TP16, TP17, TP18, TP19, TP2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

Commit message: backup
Parts:
- added TP44, TP45, TP46, TP47, TP48, TP49, TP50, TP51: TestPoint, test_point_footprints:TestPoint_THTPad_Castelated, symbol UNITED_TEST_POINTS:TestPoint_Castelated_v2
Connections:
- net 5V0 renamed 3V3
- new net 1B1: TP44.1
- new net 1B2: TP45.1
- new net 1B3: TP46.1
- new net 1B4: TP47.1
- new net 2B1: TP48.1
- new net 2B2: TP49.1
- new net 2B3: TP50.1
- new net 2B4: TP51.1

Commit message: backup
Other:
- sheet Front End Channel 1 ports: added EN_10K; removed none
- sheet Front End Channel 2 ports: added EN_10K; removed none
- sheet Front End Channel 3 ports: added EN_10K; removed none
- sheet Front End Channel 4 ports: added EN_10K; removed none
Changed lines of the file:
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@@
 	)
 	(bus_entry
-		(at 330.2 172.72)
+		(at 330.2 170.18)
 		(size -2.54 -2.54)
 		(stroke
@@
 	)
 	(bus_entry
-		(at 330.2 142.24)
+		(at 330.2 139.7)
+		(size -2.54 -2.54)
+		(stroke
+			(width 0)
+			(type default)
+		)
+	)
+	(bus_entry
+		(at 330.2 167.64)
 		(size -2.54 -2.54)
 		(stroke
@@
 	)
 	(bus_entry
+		(at 330.2 137.16)
+		(size -2.54 -2.54)
+		(stroke
+			(width 0)
+			(type default)
+		)
+	)
+	(bus_entry
 		(at 68.58 180.34)
 		(size -2.54 2.54)
@@
 	)
 	(bus_entry
-		(at 330.2 111.76)
+		(at 330.2 109.22)
 		(size -2.54 -2.54)
 		(stroke
@@
 	)
 	(bus_entry
+		(at 330.2 198.12)
+		(size -2.54 -2.54)
+		(stroke
+			(width 0)
+			(type default)
+		)
+	)
+	(bus_entry
 		(at 68.58 172.72)
 		(size -2.54 2.54)
@@
 	)
 	(bus_entry
+		(at 330.2 106.68)
+		(size -2.54 -2.54)
+		(stroke
+			(width 0)
+			(type default)
+		)
+	)
+	(bus_entry
 		(at 157.48 190.5)
 		(size -2.54 -2.54)
@@
 	)
 	(bus_entry
-		(at 330.2 203.2)
+		(at 330.2 200.66)
 		(size -2.54 -2.54)
 		(stroke
@@
 	(wire
 		(pts
-			(xy 304.8 200.66) (xy 327.66 200.66)
+			(xy 304.8 198.12) (xy 327.66 198.12)
 		)
 		(stroke
@@
 	(bus
 		(pts
-			(xy 330.2 111.76) (xy 330.2 142.24)
+			(xy 330.2 109.22) (xy 330.2 137.16)
 		)
 		(stroke
@@
 	(bus
 		(pts
-			(xy 330.2 142.24) (xy 330.2 172.72)
+			(xy 330.2 198.12) (xy 330.2 200.66)
+		)
+		(stroke
+			(width 0)
+			(type default)
+		)
+	)
+	(bus
+		(pts
+			(xy 330.2 139.7) (xy 330.2 167.64)
 		)
 		(stroke
@@
 	(wire
 		(pts
+			(xy 304.8 195.58) (xy 327.66 195.58)
+		)
+		(stroke
+			(width 0)
+			(type default)
+		)
+	)
+	(wire
+		(pts
 			(xy 304.8 210.82) (xy 317.5 210.82)
 		)
@@
 	(bus
 		(pts
-			(xy 330.2 203.2) (xy 330.2 241.3)
+			(xy 330.2 200.66) (xy 330.2 241.3)
 		)
 		(stroke
@@
 		)
 	)
+	(wire
+		(pts
+			(xy 304.8 104.14) (xy 327.66 104.14)
+		)
+		(stroke
+			(width 0)
+			(type default)
+		)
+	)
+	(bus
+		(pts
+			(xy 330.2 167.64) (xy 330.2 170.18)
+		)
+		(stroke
+			(width 0)
+			(type default)
+		)
+	)
 	(bus
 		(pts
@@
 	(bus
 		(pts
+			(xy 330.2 137.16) (xy 330.2 139.7)
+		)
+		(stroke
+			(width 0)
+			(type default)
+		)
+	)
+	(bus
+		(pts
 			(xy 157.48 195.58) (xy 157.48 200.66)
 		)
@@
 	(wire
 		(pts
+			(xy 304.8 165.1) (xy 327.66 165.1)
+		)
+		(stroke
+			(width 0)
+			(type default)
+		)
+	)
+	(wire
+		(pts
 			(xy 142.24 193.04) (xy 154.94 193.04)
 		)
@@
 	(wire
 		(pts
+			(xy 304.8 134.62) (xy 327.66 134.62)
+		)
+		(stroke
+			(width 0)
+			(type default)
+		)
+	)
+	(wire
+		(pts
 			(xy 40.64 172.72) (xy 66.04 172.72)
 		)
@@
 	(wire
 		(pts
-			(xy 304.8 170.18) (xy 327.66 170.18)
+			(xy 304.8 167.64) (xy 327.66 167.64)
 		)
 		(stroke
@@
 	(wire
 		(pts
-			(xy 304.8 109.22) (xy 327.66 109.22)
+			(xy 304.8 106.68) (xy 327.66 106.68)
 		)
 		(stroke
@@
 	(bus
 		(pts
-			(xy 330.2 172.72) (xy 330.2 203.2)
+			(xy 330.2 170.18) (xy 330.2 198.12)
+		)
+		(stroke
+			(width 0)
+			(type default)
+		)
+	)
+	(bus
+		(pts
+			(xy 330.2 106.68) (xy 330.2 109.22)
 		)
 		(stroke
@@
 	(wire
 		(pts
-			(xy 304.8 139.7) (xy 327.66 139.7)
+			(xy 304.8 137.16) (xy 327.66 137.16)
 		)
 		(stroke
@@
 	)
 	(label "P1_1"
-		(at 307.34 139.7 0)
+		(at 307.34 106.68 0)
 		(effects
 			(font
@@
 		)
 	)
+	(label "P1_6"
+		(at 307.34 198.12 0)
+		(effects
+			(font
+				(size 1.27 1.27)
+			)
+			(justify left bottom)
+		)
+	)
 	(label "LKG_COMP_B"
 		(at 276.86 142.24 180)
@@
 		)
 	)
+	(label "P1_7"
+		(at 307.34 195.58 0)
+		(effects
+			(font
+				(size 1.27 1.27)
+			)
+			(justify left bottom)
+		)
+	)
+	(label "P1_4"
+		(at 307.34 165.1 0)
+		(effects
+			(font
+				(size 1.27 1.27)
+			)
+			(justify left bottom)
+		)
+	)
 	(label "SDO_ISO"
 		(at 63.5 177.8 180)
@@
 		)
 	)
+	(label "P1_5"
+		(at 307.34 167.64 0)
+		(effects
+			(font
+				(size 1.27 1.27)
+			)
+			(justify left bottom)
+		)
+	)
 	(label "SDA_ISO"
 		(at 63.5 185.42 180)
@@
 	)
 	(label "P1_0"
-		(at 307.34 109.22 0)
+		(at 307.34 104.14 0)
 		(effects
 			(font
@@
 	)
 	(label "P1_2"
-		(at 307.34 170.18 0)
+		(at 307.34 134.62 0)
 		(effects
 			(font
@@
 	)
 	(label "P1_3"
-		(at 307.34 200.66 0)
+		(at 307.34 137.16 0)
 		(effects
 			(font
@@
 		)
 		(pin "GPIO" bidirectional
-			(at 304.8 139.7 0)
+			(at 304.8 137.16 0)
+			(effects
+				(font
+					(size 1.27 1.27)
+				)
+				(justify right)
+			)
+		)
+		(pin "EN_10K" bidirectional
+			(at 304.8 134.62 0)
 			(effects
 				(font
@@
 		)
 		(pin "GPIO" bidirectional
-			(at 304.8 109.22 0)
+			(at 304.8 106.68 0)
+			(effects
+				(font
+					(size 1.27 1.27)
+				)
+				(justify right)
+			)
+		)
+		(pin "EN_10K" bidirectional
+			(at 304.8 104.14 0)
 			(effects
 				(font
@@
 		)
 		(pin "GPIO" bidirectional
-			(at 304.8 200.66 0)
+			(at 304.8 198.12 0)
+			(effects
+				(font
+					(size 1.27 1.27)
+				)
+				(justify right)
+			)
+		)
+		(pin "EN_10K" bidirectional
+			(at 304.8 195.58 0)
 			(effects
 				(font
@@
 		)
 		(pin "GPIO" bidirectional
-			(at 304.8 170.18 0)
+			(at 304.8 167.64 0)
+			(effects
+				(font
+					(size 1.27 1.27)
+				)
+				(justify right)
+			)
+		)
+		(pin "EN_10K" bidirectional
+			(at 304.8 165.1 0)
 			(effects
 				(font
