File: minimal_ad74416h/Front End Channel 1.kicad_sch (KiCad schematic)
At the start: 5 parts

Commit message: backup
Parts:
- added C26: 4.7 nF, capacitor_footprints:C_0603_1608Metric, symbol UNITED_CAPACITORS_DATA_BASE:C_VJ0603Y472KXBAC
- added D1, D5: 36 V, diode_footprints:DO-214AA, symbol UNITED_DIODES_DATA_BASE:D_SMBJ36CA
- added R12: 2 kΩ, resistor_footprints:R_0603_1608Metric, symbol UNITED_RESISTORS_DATA_BASE:R_RNCF0603TKY2K00
- added R16: 2 kΩ, resistor_footprints:R_0402_1005Metric, symbol UNITED_RESISTORS_DATA_BASE:R_ERJ-2RKF2001X
Connections:
- net GNDA: now also C26.2, D1.1, D5.1
- net SENSEHF: now also R12.1
- net VIOUT: now also R12.2
- net I/OP: now reaches R4.2, R5.2
- net I/OP: now also C26.1, D1.2
- new net VSENSEN: D5.2
- new net VSENSEP: R16.1

Commit message: backup
Parts:
- added Q1, Q5: -100.0 V, transistor_footprints:PowerPAK 1212-8, symbol UNITED_TRANSISTORS_DATA_BASE:Q_SI7113ADN-T1-GE3
- added R20: 100 kΩ, resistor_footprints:R_0402_1005Metric, symbol UNITED_RESISTORS_DATA_BASE:R_RMCF0402JT100K
Connections:
- net GNDA: now also R20.2
- net I/OP: now also Q1.1 (S), Q1.2 (S), Q1.3 (S)
- net ISP: now reaches R16.2
- net VSENSEN renamed ISN
- net ISN: now also R20.1
- new net LKG_COMP: Q1.5 (D), Q5.5 (D)
Other:
- moved on the sheet: C14, C18, C22, C26, D1, D5, R12, R16, R4, R5

Commit message: backup
Parts:
- added J5: MTMM-101-04-L-D-196, connector_footprints:MTMM-101-04-L-D-196, symbol UNITED_CONNECTORS_DATA_BASE:J_MTMM-101-04-L-D-196
- added R24: 10 kΩ, resistor_footprints:R_0402_1005Metric, symbol UNITED_RESISTORS_DATA_BASE:R_ERJ-2RKF1002X
- added R28: 0 Ω, resistor_footprints:R_0402_1005Metric, symbol UNITED_RESISTORS_DATA_BASE:R_ERJ-2GE0R00X
- added R32: 0.15 Ω, resistor_footprints:R_1206_3216Metric, symbol UNITED_RESISTORS_DATA_BASE:R_CRM1206-FX-R150ELF
Connections:
- net ISP: now also J5.1, R24.2
- net I/OP: now also J5.2, R24.1
- net DO_SRC_SNS: now reaches Q5.1 (S)
- net DO_SRC_SNS: now also Q5.2 (S), Q5.3 (S), R32.2
- net at Q5.4 (G): now also R28.2
- new net DO_SRC_GATE: R28.1

Commit message: backup
Parts:
- added R36: 10 kΩ, resistor_footprints:R_0402_1005Metric, symbol UNITED_RESISTORS_DATA_BASE:R_ERJ-2RKF1002X
Connections:
- net I/OP: now also R36.2
- net at Q1.4 (G): now also R36.1
- net DO_VDD: now reaches R32.1
Other:
- moved on the sheet: Q1, Q5, R28, R32

Commit message: backup
Parts:
- added D13: 100.0 V, diode_footprints:DO-219AD, symbol UNITED_DIODES_DATA_BASE:D_MSE1PB-M3-89A
- added D9: 5.0 V, diode_footprints:SOD323, symbol UNITED_DIODES_DATA_BASE:D_ESD9M5.0ST5G
- added Q9: 50 V, transistor_footprints:SOT23-3, symbol UNITED_TRANSISTORS_DATA_BASE:Q_BSS138-7-F
- added R40: 100 kΩ, resistor_footprints:R_0402_1005Metric, symbol UNITED_RESISTORS_DATA_BASE:R_RMCF0402JT100K
- added R44: 3.9 kΩ, resistor_footprints:R_0402_1005Metric, symbol UNITED_RESISTORS_DATA_BASE:R_ERJ-2RKF3901X
Connections:
- net GNDA: now also R40.2, R44.2
- net I/OP: now also D9.1
- net at Q1.4 (G), R36.1: now also D13.2, D9.2
- new net: Q9.1 (G), R40.1
- new net: Q9.2 (S), R44.1
- new net: D13.1, Q9.3 (D)
Other:
- moved on the sheet: C14, C18, C22, C26, D1, D5, J5, R12, R16, R20, R24, R36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

Commit message: backup
Parts:
- added J1: MTMM-101-04-L-D-196, connector_footprints:MTMM-101-04-L-D-196, symbol UNITED_CONNECTORS_DATA_BASE:J_MTMM-101-04-L-D-196
Connections:
- net at Q9.1 (G), R40.1: now also J1.2
- new net GPIO: J1.1
Other:
- moved on the sheet: D13, Q9, R40, R44

Commit message: backup
Parts:
- renumbered C22 to C10, C26 to C4, C14 to C6, C18 to C7, D5 to D10, D13 to D3, D9 to D6, D1 to D8, J5 to J3, Q9 to Q1, Q1 to Q3, Q5 to Q4, R32 to R10, R36 to R11, R24 to R13, R16 to R18, R5 to R20, R12 to R22, R4 to R24, R20 to R26, R44 to R3, R40 to R5, R28 to R7

Commit message: backup
Parts:
- S3: renamed from J3; value MTMM-101-04-L-D-196 -> 416131160801; footprint connector_footprints:MTMM-101-04-L-D-196 -> dip_switches_footprints:416131160801; symbol UNITED_CONNECTORS_DATA_BASE:J_MTMM-101-04-L-D-196 -> UNITED_DIP_SWITCHES_DATA_BASE:S_416131160801; MPN MTMM-101-04-L-D-196 -> 416131160801; Manufacturer Samtec -> Wurth Elektronik; Mounting Style Through Hole -> Surface Mount; Series MTMM-1xx-04-L-D-196 -> 416131160801; Symbol Name J_MTMM-101-04-L-D-196 -> S_416131160801; Trustedparts Search https://www.trustedparts.com/en/search/MTMM-101-04-L-D-196 -> https://www.trustedparts.com/en/search/416131160801
Connections:
- net ISP: now also S3.2; no longer S3.1
- net I/OP: now also S3.1; no longer S3.2
Changed lines of the file:
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@@
 	)
 	(symbol
-		(lib_id "UNITED_CONNECTORS_DATA_BASE:J_MTMM-101-04-L-D-196")
+		(lib_id "UNITED_DIP_SWITCHES_DATA_BASE:S_416131160801")
 		(at 209.55 190.5 90)
+		(mirror x)
 		(unit 1)
 		(exclude_from_sim no)
@@
 		(on_board yes)
 		(dnp no)
-		(property "Reference" "J3"
-			(at 214.63 189.2299 90)
+		(fields_autoplaced yes)
+		(property "Reference" "S3"
+			(at 210.82 189.2299 90)
 			(effects
 				(font
@@
 			)
 		)
-		(property "Value" "MTMM-101-04-L-D-196"
-			(at 214.63 191.7699 90)
+		(property "Value" "416131160801"
+			(at 210.82 191.7699 90)
 			(effects
 				(font
@@
 			)
 		)
-		(property "Footprint" "connector_footprints:MTMM-101-04-L-D-196"
-			(at 215.9 185.42 0)
-			(show_name yes)
-			(effects
-				(font
-					(size 1.27 1.27)
-				)
-				(justify left)
-				(hide yes)
-			)
-		)
-		(property "Datasheet" "https://suddendocs.samtec.com/catalog_english/mtmm_th.pdf?_gl=1*10xs2wh*_gcl_au*OTQ3NjE2MTIwLjE3NTQ5MDMyODE.*_ga*NzIxODQzNjU3LjE3NTQ5MDMyODI.*_ga_3KFNZC07WW*czE3NTQ5MDMyODEkbzEkZzEkdDE3NTQ5MDYwODAkajYwJGwwJGgw"
-			(at 218.44 185.42 0)
-			(show_name yes)
-			(effects
-				(font
-					(size 1.27 1.27)
-				)
-				(justify left)
-				(hide yes)
-			)
-		)
-		(property "Description" "Samtec MTMM-1xx-04-L-D-196 series,  1 positions connector,  2.0 mm pitch,  Black,  Vertical mounting,  5.2 A,  300 V,  Through Hole,  Tin plated"
-			(at 220.98 185.42 0)
+		(property "Footprint" "dip_switches_footprints:416131160801"
+			(at 214.63 190.5 0)
+			(show_name yes)
+			(effects
+				(font
+					(size 1.27 1.27)
+				)
+				(justify left)
+				(hide yes)
+			)
+		)
+		(property "Datasheet" "https://www.we-online.com/components/products/datasheet/416131160801.pdf"
+			(at 217.17 190.5 0)
+			(show_name yes)
+			(effects
+				(font
+					(size 1.27 1.27)
+				)
+				(justify left)
+				(hide yes)
+			)
+		)
+		(property "Description" "Wurth Elektronik Vertical mounting,  Surface Mount,"
+			(at 219.71 190.5 0)
 			(show_name yes)
 			(effects
@@
 		)
 		(property "Color" "Black"
-			(at 223.52 185.42 0)
+			(at 223.52 195.58 0)
 			(show_name yes)
 			(effects
@@
 		)
 		(property "Contact Plating" "Tin"
-			(at 226.06 185.42 0)
+			(at 226.06 195.58 0)
 			(show_name yes)
 			(effects
@@
 		)
 		(property "Current Rating (A)" "5.2"
-			(at 228.6 185.42 0)
-			(show_name yes)
-			(effects
-				(font
-					(size 1.27 1.27)
-				)
-				(justify left)
-				(hide yes)
-			)
-		)
-		(property "MPN" "MTMM-101-04-L-D-196"
-			(at 231.14 185.42 0)
-			(show_name yes)
-			(effects
-				(font
-					(size 1.27 1.27)
-				)
-				(justify left)
-				(hide yes)
-			)
-		)
-		(property "Manufacturer" "Samtec"
-			(at 233.68 185.42 0)
+			(at 228.6 195.58 0)
+			(show_name yes)
+			(effects
+				(font
+					(size 1.27 1.27)
+				)
+				(justify left)
+				(hide yes)
+			)
+		)
+		(property "MPN" "416131160801"
+			(at 222.25 190.5 0)
+			(show_name yes)
+			(effects
+				(font
+					(size 1.27 1.27)
+				)
+				(justify left)
+				(hide yes)
+			)
+		)
+		(property "Manufacturer" "Wurth Elektronik"
+			(at 224.79 190.5 0)
 			(show_name yes)
 			(effects
@@
 		)
 		(property "Mounting Angle" "Vertical"
-			(at 236.22 185.42 0)
-			(show_name yes)
-			(effects
-				(font
-					(size 1.27 1.27)
-				)
-				(justify left)
-				(hide yes)
-			)
-		)
-		(property "Mounting Style" "Through Hole"
-			(at 238.76 185.42 0)
+			(at 227.33 190.5 0)
+			(show_name yes)
+			(effects
+				(font
+					(size 1.27 1.27)
+				)
+				(justify left)
+				(hide yes)
+			)
+		)
+		(property "Mounting Style" "Surface Mount"
+			(at 229.87 190.5 0)
 			(show_name yes)
 			(effects
@@
 		)
 		(property "Number of Rows" "2"
-			(at 241.3 185.42 0)
+			(at 232.41 190.5 0)
 			(show_name yes)
 			(effects
@@
 		)
 		(property "Pin Count" "1"
-			(at 243.84 185.42 0)
+			(at 234.95 190.5 0)
 			(show_name yes)
 			(effects
@@
 		)
 		(property "Pitch (mm)" "2.0"
-			(at 246.38 185.42 0)
-			(show_name yes)
-			(effects
-				(font
-					(size 1.27 1.27)
-				)
-				(justify left)
-				(hide yes)
-			)
-		)
-		(property "Series" "MTMM-1xx-04-L-D-196"
-			(at 248.92 185.42 0)
-			(show_name yes)
-			(effects
-				(font
-					(size 1.27 1.27)
-				)
-				(justify left)
-				(hide yes)
-			)
-		)
-		(property "Symbol Name" "J_MTMM-101-04-L-D-196"
-			(at 251.46 185.42 0)
-			(show_name yes)
-			(effects
-				(font
-					(size 1.27 1.27)
-				)
-				(justify left)
-				(hide yes)
-			)
-		)
-		(property "Trustedparts Search" "https://www.trustedparts.com/en/search/MTMM-101-04-L-D-196"
-			(at 254 185.42 0)
+			(at 246.38 195.58 0)
+			(show_name yes)
+			(effects
+				(font
+					(size 1.27 1.27)
+				)
+				(justify left)
+				(hide yes)
+			)
+		)
+		(property "Series" "416131160801"
+			(at 237.49 190.5 0)
+			(show_name yes)
+			(effects
+				(font
+					(size 1.27 1.27)
+				)
+				(justify left)
+				(hide yes)
+			)
+		)
+		(property "Symbol Name" "S_416131160801"
+			(at 240.03 190.5 0)
+			(show_name yes)
+			(effects
+				(font
+					(size 1.27 1.27)
+				)
+				(justify left)
+				(hide yes)
+			)
+		)
+		(property "Trustedparts Search" "https://www.trustedparts.com/en/search/416131160801"
+			(at 242.57 190.5 0)
 			(show_name yes)
 			(effects
@@
 		)
 		(property "Voltage Rating (V)" "300"
-			(at 256.54 185.42 0)
+			(at 256.54 195.58 0)
 			(show_name yes)
 			(effects
@@
 			(project ""
 				(path "/996c4afa-af57-455f-b0b6-e0f996045a90/010e8139-4c72-4154-a66e-8d0ded735c08"
-					(reference "J5")
+					(reference "S5")
 					(unit 1)
 				)
 				(path "/996c4afa-af57-455f-b0b6-e0f996045a90/0786ce20-9b4f-45a9-9d62-20c78d282fdc"
-					(reference "J3")
+					(reference "S3")
 					(unit 1)
 				)
 				(path "/996c4afa-af57-455f-b0b6-e0f996045a90/0d35b6da-5370-4b8d-bdb2-6a6466fd726d"
-					(reference "J4")
+					(reference "S4")
 					(unit 1)
 				)
 				(path "/996c4afa-af57-455f-b0b6-e0f996045a90/56f471d9-4771-4bab-9fc0-7f2502be0d29"
-					(reference "J6")
-					(unit 1)
-				)
+					(reference "S6")
+					(unit 1)
+				)
