File: minimal_ad74416h/Front End Channel 1.kicad_sch (KiCad schematic)
At the start: 24 parts, among them J1 MTMM-101-04-L-D-196, Q1 50 V, Q3 -100.0 V, Q4 -100.0 V

Commit message: backup
Parts:
- removed J1: MTMM-101-04-L-D-196, connector_footprints:MTMM-101-04-L-D-196, symbol UNITED_CONNECTORS_DATA_BASE:J_MTMM-101-04-L-D-196
- added S7: 416131160801, dip_switches_footprints:416131160801, symbol UNITED_DIP_SWITCHES_DATA_BASE:S_416131160801
Connections:
- net GPIO: now also S7.1
- net at Q1.1 (G), R5.1: now also S7.2
Changed lines of the file:
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@@
+	)
+	(symbol
+		(lib_id "UNITED_DIP_SWITCHES_DATA_BASE:S_416131160801")
+		(at 146.05 101.6 0)
+		(unit 1)
+		(exclude_from_sim no)
+		(in_bom yes)
+		(on_board yes)
+		(dnp no)
+		(fields_autoplaced yes)
+		(property "Reference" "S7"
+			(at 146.05 95.25 0)
+			(effects
+				(font
+					(size 1.27 1.27)
+				)
+			)
+		)
+		(property "Value" "416131160801"
+			(at 146.05 97.79 0)
+			(effects
+				(font
+					(size 1.27 1.27)
+				)
+			)
+		)
+		(property "Footprint" "dip_switches_footprints:416131160801"
+			(at 146.05 106.68 0)
+			(show_name yes)
+			(effects
+				(font
+					(size 1.27 1.27)
+				)
+				(justify left)
+				(hide yes)
+			)
+		)
+		(property "Datasheet" "https://www.we-online.com/components/products/datasheet/416131160801.pdf"
+			(at 146.05 109.22 0)
+			(show_name yes)
+			(effects
+				(font
+					(size 1.27 1.27)
+				)
+				(justify left)
+				(hide yes)
+			)
+		)
+		(property "Description" "Wurth Elektronik Vertical mounting,  Surface Mount,"
+			(at 146.05 111.76 0)
+			(show_name yes)
+			(effects
+				(font
+					(size 1.27 1.27)
+				)
+				(justify left)
+				(hide yes)
+			)
+		)
+		(property "Color" "Black"
+			(at 151.13 115.57 0)
+			(show_name yes)
+			(effects
+				(font
+					(size 1.27 1.27)
+				)
+				(justify left)
+				(hide yes)
+			)
+		)
+		(property "Contact Plating" "Tin"
+			(at 151.13 118.11 0)
+			(show_name yes)
+			(effects
+				(font
+					(size 1.27 1.27)
+				)
+				(justify left)
+				(hide yes)
+			)
+		)
+		(property "Current Rating (A)" "5.2"
+			(at 151.13 120.65 0)
+			(show_name yes)
+			(effects
+				(font
+					(size 1.27 1.27)
+				)
+				(justify left)
+				(hide yes)
+			)
+		)
+		(property "MPN" "416131160801"
+			(at 146.05 114.3 0)
+			(show_name yes)
+			(effects
+				(font
+					(size 1.27 1.27)
+				)
+				(justify left)
+				(hide yes)
+			)
+		)
+		(property "Manufacturer" "Wurth Elektronik"
+			(at 146.05 116.84 0)
+			(show_name yes)
+			(effects
+				(font
+					(size 1.27 1.27)
+				)
+				(justify left)
+				(hide yes)
+			)
+		)
+		(property "Mounting Angle" "Vertical"
+			(at 146.05 119.38 0)
+			(show_name yes)
+			(effects
+				(font
+					(size 1.27 1.27)
+				)
+				(justify left)
+				(hide yes)
+			)
+		)
+		(property "Mounting Style" "Surface Mount"
+			(at 146.05 121.92 0)
+			(show_name yes)
+			(effects
+				(font
+					(size 1.27 1.27)
+				)
+				(justify left)
+				(hide yes)
+			)
+		)
+		(property "Number of Rows" "2"
+			(at 146.05 124.46 0)
+			(show_name yes)
+			(effects
+				(font
+					(size 1.27 1.27)
+				)
+				(justify left)
+				(hide yes)
+			)
+		)
+		(property "Pin Count" "1"
+			(at 146.05 127 0)
+			(show_name yes)
+			(effects
+				(font
+					(size 1.27 1.27)
+				)
+				(justify left)
+				(hide yes)
+			)
+		)
+		(property "Pitch (mm)" "2.0"
+			(at 151.13 138.43 0)
+			(show_name yes)
+			(effects
+				(font
+					(size 1.27 1.27)
+				)
+				(justify left)
+				(hide yes)
+			)
+		)
+		(property "Series" "416131160801"
+			(at 146.05 129.54 0)
+			(show_name yes)
+			(effects
+				(font
+					(size 1.27 1.27)
+				)
+				(justify left)
+				(hide yes)
+			)
+		)
+		(property "Symbol Name" "S_416131160801"
+			(at 146.05 132.08 0)
+			(show_name yes)
+			(effects
+				(font
+					(size 1.27 1.27)
+				)
+				(justify left)
+				(hide yes)
+			)
+		)
+		(property "Trustedparts Search" "https://www.trustedparts.com/en/search/416131160801"
+			(at 146.05 134.62 0)
+			(show_name yes)
+			(effects
+				(font
+					(size 1.27 1.27)
+				)
+				(justify left)
+				(hide yes)
+			)
+		)
+		(property "Voltage Rating (V)" "300"
+			(at 151.13 148.59 0)
+			(show_name yes)
+			(effects
+				(font
+					(size 1.27 1.27)
+				)
+				(justify left)
+				(hide yes)
+			)
+		)
+		(pin "1"
+		)
+		(pin "2"
+		)
+		(instances
+			(project "minimal_ad74416h"
+				(path "/996c4afa-af57-455f-b0b6-e0f996045a90/010e8139-4c72-4154-a66e-8d0ded735c08"
+					(reference "S8")
+					(unit 1)
+				)
+				(path "/996c4afa-af57-455f-b0b6-e0f996045a90/0786ce20-9b4f-45a9-9d62-20c78d282fdc"
+					(reference "S7")
+					(unit 1)
+				)
+				(path "/996c4afa-af57-455f-b0b6-e0f996045a90/0d35b6da-5370-4b8d-bdb2-6a6466fd726d"
+					(reference "S10")
+					(unit 1)
+				)
+				(path "/996c4afa-af57-455f-b0b6-e0f996045a90/56f471d9-4771-4bab-9fc0-7f2502be0d29"
+					(reference "S9")
+					(unit 1)
+				)
+			)
+		)
 	)
 	(symbol
@@
 					(unit 1)
 				)
-			)
-		)
-	)
-	(symbol
-		(lib_id "UNITED_CONNECTORS_DATA_BASE:J_MTMM-101-04-L-D-196")
-		(at 146.05 101.6 0)
-		(mirror x)
-		(unit 1)
-		(exclude_from_sim no)
-		(in_bom yes)
-		(on_board yes)
-		(dnp no)
-		(property "Reference" "J1"
-			(at 146.05 92.71 0)
-			(effects
-				(font
-					(size 1.27 1.27)
-				)
-			)
-		)
-		(property "Value" "MTMM-101-04-L-D-196"
-			(at 146.05 95.25 0)
-			(effects
-				(font
-					(size 1.27 1.27)
-				)
-			)
-		)
-		(property "Footprint" "connector_footprints:MTMM-101-04-L-D-196"
-			(at 151.13 95.25 0)
-			(show_name yes)
-			(effects
-				(font
-					(size 1.27 1.27)
-				)
-				(justify left)
-				(hide yes)
-			)
-		)
-		(property "Datasheet" "https://suddendocs.samtec.com/catalog_english/mtmm_th.pdf?_gl=1*10xs2wh*_gcl_au*OTQ3NjE2MTIwLjE3NTQ5MDMyODE.*_ga*NzIxODQzNjU3LjE3NTQ5MDMyODI.*_ga_3KFNZC07WW*czE3NTQ5MDMyODEkbzEkZzEkdDE3NTQ5MDYwODAkajYwJGwwJGgw"
-			(at 151.13 92.71 0)
-			(show_name yes)
-			(effects
-				(font
-					(size 1.27 1.27)
-				)
-				(justify left)
-				(hide yes)
-			)
-		)
-		(property "Description" "Samtec MTMM-1xx-04-L-D-196 series,  1 positions connector,  2.0 mm pitch,  Black,  Vertical mounting,  5.2 A,  300 V,  Through Hole,  Tin plated"
-			(at 151.13 90.17 0)
-			(show_name yes)
-			(effects
-				(font
-					(size 1.27 1.27)
-				)
-				(justify left)
-				(hide yes)
-			)
-		)
-		(property "Color" "Black"
-			(at 151.13 87.63 0)
-			(show_name yes)
-			(effects
-				(font
-					(size 1.27 1.27)
-				)
-				(justify left)
-				(hide yes)
-			)
-		)
-		(property "Contact Plating" "Tin"
-			(at 151.13 85.09 0)
-			(show_name yes)
-			(effects
-				(font
-					(size 1.27 1.27)
-				)
-				(justify left)
-				(hide yes)
-			)
-		)
-		(property "Current Rating (A)" "5.2"
-			(at 151.13 82.55 0)
-			(show_name yes)
-			(effects
-				(font
-					(size 1.27 1.27)
-				)
-				(justify left)
-				(hide yes)
-			)
-		)
-		(property "MPN" "MTMM-101-04-L-D-196"
-			(at 151.13 80.01 0)
-			(show_name yes)
-			(effects
-				(font
-					(size 1.27 1.27)
-				)
-				(justify left)
-				(hide yes)
-			)
-		)
-		(property "Manufacturer" "Samtec"
-			(at 151.13 77.47 0)
-			(show_name yes)
-			(effects
-				(font
-					(size 1.27 1.27)
-				)
-				(justify left)
-				(hide yes)
-			)
-		)
-		(property "Mounting Angle" "Vertical"
-			(at 151.13 74.93 0)
-			(show_name yes)
-			(effects
-				(font
-					(size 1.27 1.27)
-				)
-				(justify left)
-				(hide yes)
-			)
-		)
-		(property "Mounting Style" "Through Hole"
-			(at 151.13 72.39 0)
-			(show_name yes)
-			(effects
-				(font
-					(size 1.27 1.27)
-				)
-				(justify left)
-				(hide yes)
-			)
-		)
-		(property "Number of Rows" "2"
-			(at 151.13 69.85 0)
-			(show_name yes)
-			(effects
-				(font
-					(size 1.27 1.27)
-				)
-				(justify left)
-				(hide yes)
-			)
-		)
-		(property "Pin Count" "1"
-			(at 151.13 67.31 0)
-			(show_name yes)
-			(effects
-				(font
-					(size 1.27 1.27)
-				)
-				(justify left)
-				(hide yes)
-			)
-		)
-		(property "Pitch (mm)" "2.0"
-			(at 151.13 64.77 0)
-			(show_name yes)
-			(effects
-				(font
-					(size 1.27 1.27)
-				)
-				(justify left)
-				(hide yes)
-			)
-		)
-		(property "Series" "MTMM-1xx-04-L-D-196"
-			(at 151.13 62.23 0)
-			(show_name yes)
-			(effects
-				(font
-					(size 1.27 1.27)
-				)
-				(justify left)
-				(hide yes)
-			)
-		)
-		(property "Symbol Name" "J_MTMM-101-04-L-D-196"
-			(at 151.13 59.69 0)
-			(show_name yes)
-			(effects
-				(font
-					(size 1.27 1.27)
-				)
-				(justify left)
-				(hide yes)
-			)
-		)
-		(property "Trustedparts Search" "https://www.trustedparts.com/en/search/MTMM-101-04-L-D-196"
-			(at 151.13 57.15 0)
-			(show_name yes)
-			(effects
-				(font
-					(size 1.27 1.27)
-				)
-				(justify left)
-				(hide yes)
-			)
-		)
-		(property "Voltage Rating (V)" "300"
-			(at 151.13 54.61 0)
-			(show_name yes)
-			(effects
-				(font
-					(size 1.27 1.27)
-				)
-				(justify left)
-				(hide yes)
-			)
-		)
-		(pin "1"
-		)
-		(pin "2"
-		)
-		(instances
-			(project "minimal_ad74416h"
-				(path "/996c4afa-af57-455f-b0b6-e0f996045a90/010e8139-4c72-4154-a66e-8d0ded735c08"
-					(reference "J7")
-					(unit 1)
-				)
-				(path "/996c4afa-af57-455f-b0b6-e0f996045a90/0786ce20-9b4f-45a9-9d62-20c78d282fdc"
-					(reference "J1")
-					(unit 1)
-				)
-				(path "/996c4afa-af57-455f-b0b6-e0f996045a90/0d35b6da-5370-4b8d-bdb2-6a6466fd726d"
-					(reference "J2")
-					(unit 1)
-				)
-				(path "/996c4afa-af57-455f-b0b6-e0f996045a90/56f471d9-4771-4bab-9fc0-7f2502be0d29"
-					(reference "J8")
-					(unit 1)
-				)

Commit message: backup
Parts:
- renumbered D3 to D4, R3 to R1, S7 to S1, S3 to S5
Changed lines of the file:
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@@
 		(dnp no)
 		(fields_autoplaced yes)
-		(property "Reference" "S7"
+		(property "Reference" "S1"
 			(at 146.05 95.25 0)
 			(effects
@@
 			(project "minimal_ad74416h"
 				(path "/996c4afa-af57-455f-b0b6-e0f996045a90/010e8139-4c72-4154-a66e-8d0ded735c08"
-					(reference "S8")
+					(reference "S9")
 					(unit 1)
 				)
 				(path "/996c4afa-af57-455f-b0b6-e0f996045a90/0786ce20-9b4f-45a9-9d62-20c78d282fdc"
-					(reference "S7")
+					(reference "S1")
 					(unit 1)
 				)
 				(path "/996c4afa-af57-455f-b0b6-e0f996045a90/0d35b6da-5370-4b8d-bdb2-6a6466fd726d"
-					(reference "S10")
+					(reference "S2")
 					(unit 1)
 				)
 				(path "/996c4afa-af57-455f-b0b6-e0f996045a90/56f471d9-4771-4bab-9fc0-7f2502be0d29"
-					(reference "S9")
+					(reference "S10")
 					(unit 1)
 				)
@@
 		(dnp no)
 		(fields_autoplaced yes)
-		(property "Reference" "S3"
+		(property "Reference" "S5"
 			(at 210.82 189.2299 90)
 			(effects
@@
 			(project ""
 				(path "/996c4afa-af57-455f-b0b6-e0f996045a90/010e8139-4c72-4154-a66e-8d0ded735c08"
-					(reference "S5")
+					(reference "S7")
 					(unit 1)
 				)
 				(path "/996c4afa-af57-455f-b0b6-e0f996045a90/0786ce20-9b4f-45a9-9d62-20c78d282fdc"
-					(reference "S3")
+					(reference "S5")
 					(unit 1)
 				)
 				(path "/996c4afa-af57-455f-b0b6-e0f996045a90/0d35b6da-5370-4b8d-bdb2-6a6466fd726d"
-					(reference "S4")
+					(reference "S6")
 					(unit 1)
 				)
 				(path "/996c4afa-af57-455f-b0b6-e0f996045a90/56f471d9-4771-4bab-9fc0-7f2502be0d29"
-					(reference "S6")
+					(reference "S8")
 					(unit 1)
 				)
@@
 		(dnp no)
 		(fields_autoplaced yes)
-		(property "Reference" "D3"
+		(property "Reference" "D4"
 			(at 175.26 82.55 0)
 			(effects
@@
 				)
 				(path "/996c4afa-af57-455f-b0b6-e0f996045a90/0786ce20-9b4f-45a9-9d62-20c78d282fdc"
-					(reference "D3")
+					(reference "D4")
 					(unit 1)
 				)
 				(path "/996c4afa-af57-455f-b0b6-e0f996045a90/0d35b6da-5370-4b8d-bdb2-6a6466fd726d"
-					(reference "D4")
+					(reference "D5")
 					(unit 1)
 				)
@@
 		(on_board yes)
 		(dnp no)
-		(property "Reference" "R3"
+		(property "Reference" "R1"
 			(at 162.56 110.4899 90)
 			(effects
@@
 				)
 				(path "/996c4afa-af57-455f-b0b6-e0f996045a90/0786ce20-9b4f-45a9-9d62-20c78d282fdc"
-					(reference "R3")
+					(reference "R1")
 					(unit 1)
 				)
@@
 				)
 				(path "/996c4afa-af57-455f-b0b6-e0f996045a90/56f471d9-4771-4bab-9fc0-7f2502be0d29"
-					(reference "R49")
+					(reference "R54")
 					(unit 1)
 				)
@@
 			(project "minimal_ad74416h"
 				(path "/996c4afa-af57-455f-b0b6-e0f996045a90/010e8139-4c72-4154-a66e-8d0ded735c08"
-					(reference "R48")
+					(reference "R53")
 					(unit 1)
 				)
@@
 				)
 				(path "/996c4afa-af57-455f-b0b6-e0f996045a90/0d35b6da-5370-4b8d-bdb2-6a6466fd726d"
-					(reference "R4")
+					(reference "R2")
 					(unit 1)
 				)

Commit message: backup
Parts:
- renumbered C4 to C10, C6 to C12, C7 to C13, C10 to C16, R5 to R11, R7 to R13, R10 to R16, R11 to R17, R13 to R19, R18 to R24, R20 to R26, R22 to R28, R24 to R30, R26 to R32, R1 to R7

Commit message: backup
Parts:
- renumbered R7 to R3
Changed lines of the file:
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@@
 		(on_board yes)
 		(dnp no)
-		(property "Reference" "R7"
+		(property "Reference" "R3"
 			(at 162.56 110.4899 90)
 			(effects
@@
 				)
 				(path "/996c4afa-af57-455f-b0b6-e0f996045a90/0786ce20-9b4f-45a9-9d62-20c78d282fdc"
-					(reference "R7")
+					(reference "R3")
 					(unit 1)
 				)
@@
 				)
 				(path "/996c4afa-af57-455f-b0b6-e0f996045a90/0d35b6da-5370-4b8d-bdb2-6a6466fd726d"
-					(reference "R8")
-					(unit 1)
-				)
+					(reference "R4")
+					(unit 1)
+				)

Commit message: backup
Parts:
- renumbered R13 to R15, R16 to R18, R17 to R19, R19 to R21, R24 to R26, R26 to R28, R28 to R30, R30 to R32, R32 to R34
Changed lines of the file:
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@@
 		(dnp no)
 		(fields_autoplaced yes)
-		(property "Reference" "R30"
+		(property "Reference" "R32"
 			(at 196.85 133.35 0)
 			(effects
@@
 			(project "minimal_ad74416h"
 				(path "/996c4afa-af57-455f-b0b6-e0f996045a90/010e8139-4c72-4154-a66e-8d0ded735c08"
-					(reference "R36")
+					(reference "R38")
 					(unit 1)
 				)
 				(path "/996c4afa-af57-455f-b0b6-e0f996045a90/0786ce20-9b4f-45a9-9d62-20c78d282fdc"
-					(reference "R30")
+					(reference "R32")
 					(unit 1)
 				)
 				(path "/996c4afa-af57-455f-b0b6-e0f996045a90/0d35b6da-5370-4b8d-bdb2-6a6466fd726d"
-					(reference "R31")
+					(reference "R33")
 					(unit 1)
 				)
 				(path "/996c4afa-af57-455f-b0b6-e0f996045a90/56f471d9-4771-4bab-9fc0-7f2502be0d29"
-					(reference "R37")
+					(reference "R39")
 					(unit 1)
 				)
@@
 		(dnp no)
 		(fields_autoplaced yes)
-		(property "Reference" "R13"
+		(property "Reference" "R15"
 			(at 184.15 57.15 0)
 			(effects
@@
 			(project ""
 				(path "/996c4afa-af57-455f-b0b6-e0f996045a90/010e8139-4c72-4154-a66e-8d0ded735c08"
-					(reference "R46")
+					(reference "R48")
 					(unit 1)
 				)
 				(path "/996c4afa-af57-455f-b0b6-e0f996045a90/0786ce20-9b4f-45a9-9d62-20c78d282fdc"
-					(reference "R13")
+					(reference "R15")
 					(unit 1)
 				)
 				(path "/996c4afa-af57-455f-b0b6-e0f996045a90/0d35b6da-5370-4b8d-bdb2-6a6466fd726d"
-					(reference "R18")
+					(reference "R20")
 					(unit 1)
 				)
 				(path "/996c4afa-af57-455f-b0b6-e0f996045a90/56f471d9-4771-4bab-9fc0-7f2502be0d29"
-					(reference "R51")
+					(reference "R53")
 					(unit 1)
 				)
@@
 		(dnp no)
 		(fields_autoplaced yes)
-		(property "Reference" "R24"
+		(property "Reference" "R26"
 			(at 184.15 196.85 0)
 			(effects
@@
 			(project "minimal_ad74416h"
 				(path "/996c4afa-af57-455f-b0b6-e0f996045a90/010e8139-4c72-4154-a66e-8d0ded735c08"
-					(reference "R42")
+					(reference "R44")
 					(unit 1)
 				)
 				(path "/996c4afa-af57-455f-b0b6-e0f996045a90/0786ce20-9b4f-45a9-9d62-20c78d282fdc"
-					(reference "R24")
+					(reference "R26")
 					(unit 1)
 				)
 				(path "/996c4afa-af57-455f-b0b6-e0f996045a90/0d35b6da-5370-4b8d-bdb2-6a6466fd726d"
-					(reference "R25")
+					(reference "R27")
 					(unit 1)
 				)
 				(path "/996c4afa-af57-455f-b0b6-e0f996045a90/56f471d9-4771-4bab-9fc0-7f2502be0d29"
-					(reference "R43")
+					(reference "R45")
 					(unit 1)
 				)
@@
 		(on_board yes)
 		(dnp no)
-		(property "Reference" "R17"
+		(property "Reference" "R19"
 			(at 194.31 93.9799 90)
 			(effects
@@
 			(project "minimal_ad74416h"
 				(path "/996c4afa-af57-455f-b0b6-e0f996045a90/010e8139-4c72-4154-a66e-8d0ded735c08"
-					(reference "R50")
+					(reference "R52")
 					(unit 1)
 				)
 				(path "/996c4afa-af57-455f-b0b6-e0f996045a90/0786ce20-9b4f-45a9-9d62-20c78d282fdc"
-					(reference "R17")
+					(reference "R19")
 					(unit 1)
 				)
 				(path "/996c4afa-af57-455f-b0b6-e0f996045a90/0d35b6da-5370-4b8d-bdb2-6a6466fd726d"
-					(reference "R14")
+					(reference "R16")
 					(unit 1)
 				)
 				(path "/996c4afa-af57-455f-b0b6-e0f996045a90/56f471d9-4771-4bab-9fc0-7f2502be0d29"
-					(reference "R47")
+					(reference "R49")
 					(unit 1)
 				)
@@
 		(on_board yes)
 		(dnp no)
-		(property "Reference" "R16"
+		(property "Reference" "R18"
 			(at 200.66 43.1799 90)
 			(effects
@@
 			(project ""
 				(path "/996c4afa-af57-455f-b0b6-e0f996045a90/010e8139-4c72-4154-a66e-8d0ded735c08"
-					(reference "R49")
+					(reference "R51")
 					(unit 1)
 				)
 				(path "/996c4afa-af57-455f-b0b6-e0f996045a90/0786ce20-9b4f-45a9-9d62-20c78d282fdc"
-					(reference "R16")
+					(reference "R18")
 					(unit 1)
 				)
 				(path "/996c4afa-af57-455f-b0b6-e0f996045a90/0d35b6da-5370-4b8d-bdb2-6a6466fd726d"
-					(reference "R15")
+					(reference "R17")
 					(unit 1)
 				)
 				(path "/996c4afa-af57-455f-b0b6-e0f996045a90/56f471d9-4771-4bab-9fc0-7f2502be0d29"
-					(reference "R48")
+					(reference "R50")
 					(unit 1)
 				)
@@
 		(on_board yes)
 		(dnp no)
-		(property "Reference" "R32"
+		(property "Reference" "R34"
 			(at 175.26 220.9799 90)
 			(effects
@@
 			(project ""
 				(path "/996c4afa-af57-455f-b0b6-e0f996045a90/010e8139-4c72-4154-a66e-8d0ded735c08"
-					(reference "R34")
+					(reference "R36")
 					(unit 1)
 				)
 				(path "/996c4afa-af57-455f-b0b6-e0f996045a90/0786ce20-9b4f-45a9-9d62-20c78d282fdc"
-					(reference "R32")
+					(reference "R34")
 					(unit 1)
 				)
 				(path "/996c4afa-af57-455f-b0b6-e0f996045a90/0d35b6da-5370-4b8d-bdb2-6a6466fd726d"
-					(reference "R33")
+					(reference "R35")
 					(unit 1)
 				)
 				(path "/996c4afa-af57-455f-b0b6-e0f996045a90/56f471d9-4771-4bab-9fc0-7f2502be0d29"
-					(reference "R35")
+					(reference "R37")
 					(unit 1)
 				)
@@
 		(dnp no)
 		(fields_autoplaced yes)
-		(property "Reference" "R28"
+		(property "Reference" "R30"
 			(at 184.15 146.05 0)
 			(effects
@@
 			(project ""
 				(path "/996c4afa-af57-455f-b0b6-e0f996045a90/010e8139-4c72-4154-a66e-8d0ded735c08"
-					(reference "R38")
+					(reference "R40")
 					(unit 1)
 				)
 				(path "/996c4afa-af57-455f-b0b6-e0f996045a90/0786ce20-9b4f-45a9-9d62-20c78d282fdc"
-					(reference "R28")
+					(reference "R30")
 					(unit 1)
 				)
 				(path "/996c4afa-af57-455f-b0b6-e0f996045a90/0d35b6da-5370-4b8d-bdb2-6a6466fd726d"
-					(reference "R29")
+					(reference "R31")
 					(unit 1)
 				)
 				(path "/996c4afa-af57-455f-b0b6-e0f996045a90/56f471d9-4771-4bab-9fc0-7f2502be0d29"
-					(reference "R39")
+					(reference "R41")
 					(unit 1)
 				)
@@
 			(project ""
 				(path "/996c4afa-af57-455f-b0b6-e0f996045a90/010e8139-4c72-4154-a66e-8d0ded735c08"
-					(reference "R52")
+					(reference "R54")
 					(unit 1)
 				)
@@
 				)
 				(path "/996c4afa-af57-455f-b0b6-e0f996045a90/56f471d9-4771-4bab-9fc0-7f2502be0d29"
-					(reference "R58")
+					(reference "R60")
 					(unit 1)
 				)
@@
 		(on_board yes)
 		(dnp no)
-		(property "Reference" "R19"
+		(property "Reference" "R21"
 			(at 200.66 189.2299 90)
 			(effects
@@
 			(project "minimal_ad74416h"
 				(path "/996c4afa-af57-455f-b0b6-e0f996045a90/010e8139-4c72-4154-a66e-8d0ded735c08"
-					(reference "R44")
+					(reference "R46")
 					(unit 1)
 				)
 				(path "/996c4afa-af57-455f-b0b6-e0f996045a90/0786ce20-9b4f-45a9-9d62-20c78d282fdc"
-					(reference "R19")
+					(reference "R21")
 					(unit 1)
 				)
 				(path "/996c4afa-af57-455f-b0b6-e0f996045a90/0d35b6da-5370-4b8d-bdb2-6a6466fd726d"
-					(reference "R23")
+					(reference "R25")
 					(unit 1)
 				)
 				(path "/996c4afa-af57-455f-b0b6-e0f996045a90/56f471d9-4771-4bab-9fc0-7f2502be0d29"
-					(reference "R45")
+					(reference "R47")
 					(unit 1)
 				)
@@
 		(dnp no)
 		(fields_autoplaced yes)
-		(property "Reference" "R26"
+		(property "Reference" "R28"
 			(at 184.15 171.45 0)
 			(effects
@@
 			(project ""
 				(path "/996c4afa-af57-455f-b0b6-e0f996045a90/010e8139-4c72-4154-a66e-8d0ded735c08"
-					(reference "R40")
+					(reference "R42")
 					(unit 1)
 				)
 				(path "/996c4afa-af57-455f-b0b6-e0f996045a90/0786ce20-9b4f-45a9-9d62-20c78d282fdc"
-					(reference "R26")
+					(reference "R28")
 					(unit 1)
 				)
 				(path "/996c4afa-af57-455f-b0b6-e0f996045a90/0d35b6da-5370-4b8d-bdb2-6a6466fd726d"
-					(reference "R27")
+					(reference "R29")
 					(unit 1)
 				)
 				(path "/996c4afa-af57-455f-b0b6-e0f996045a90/56f471d9-4771-4bab-9fc0-7f2502be0d29"
-					(reference "R41")
+					(reference "R43")
 					(unit 1)
 				)
@@
 			(project "minimal_ad74416h"
 				(path "/996c4afa-af57-455f-b0b6-e0f996045a90/010e8139-4c72-4154-a66e-8d0ded735c08"
-					(reference "R57")
+					(reference "R59")
 					(unit 1)
 				)
@@
 				)
 				(path "/996c4afa-af57-455f-b0b6-e0f996045a90/56f471d9-4771-4bab-9fc0-7f2502be0d29"
-					(reference "R53")
+					(reference "R55")
 					(unit 1)
 				)

Commit message: backup
Parts:
- removed S1, S5: 416131160801, dip_switches_footprints:416131160801, symbol UNITED_DIP_SWITCHES_DATA_BASE:S_416131160801
- added Q7: 50 V, transistor_footprints:SOT23-3, symbol UNITED_TRANSISTORS_DATA_BASE:Q_BSS138-7-F
- renumbered C16 to C10, C10 to C4, C12 to C6, C13 to C7, D6 to D10, D8 to D12, D10 to D14, D4 to D7, R3 to R1, R15 to R13, R18 to R17, R21 to R22, R26 to R24, R28 to R26, R30 to R28, R32 to R30, R34 to R32, R11 to R9
Connections:
- net GPIO: now also Q1.1 (G), R9.1
- net ISP: now also Q7.2 (S)
- net I/OP: now also Q7.3 (D)
Other:
- moved on the sheet: D14, R22, R24, R32

Commit message: backup
Connections:
- net EN_10K: now reaches Q7.1 (G)
Changed lines of the file:
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@@
+	(wire
+		(pts
+			(xy 127 203.2) (xy 182.88 203.2)
+		)
+		(stroke
+			(width 0)
+			(type default)
+		)
+	)
 	(wire
 		(pts
@@
 	)
 	(label "SENSEHF"
-		(at 166.37 152.4 0)
+		(at 165.1 152.4 0)
 		(effects
 			(font
@@
 	)
 	(label "CCOMP"
-		(at 166.37 127 0)
+		(at 165.1 127 0)
+		(effects
+			(font
+				(size 1.27 1.27)
+			)
+			(justify left bottom)
+		)
+	)
+	(label "EN_10K"
+		(at 165.1 203.2 0)
 		(effects
 			(font
@@
 	)
 	(label "VIOUT"
-		(at 166.37 139.7 0)
+		(at 165.1 139.7 0)
 		(effects
 			(font
@@
 	)
 	(label "SENSELF"
-		(at 166.37 177.8 0)
+		(at 165.1 177.8 0)
 		(effects
 			(font
@@
 	)
 	(label "VSENSEN"
-		(at 166.37 241.3 0)
+		(at 165.1 241.3 0)
 		(effects
 			(font
@@
 		(effects
 			(font
+				(size 1.27 1.27)
+			)
+			(justify right)
+		)
+	)
+	(hierarchical_label "EN_10K"
+		(shape bidirectional)
+		(at 127 203.2 180)
+		(effects
+			(font
