File: minimal_ad74416h/Front End Channel 1.kicad_sch (KiCad schematic)
At the start: 23 parts, among them Q1 50 V, Q3 -100.0 V, Q4 -100.0 V, Q7 50 V

Commit message: backup
Parts:
- renumbered R13 to R11
Changed lines of the file:
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@@
 		(dnp no)
 		(fields_autoplaced yes)
-		(property "Reference" "R13"
+		(property "Reference" "R11"
 			(at 184.15 57.15 0)
 			(effects
@@
 				)
 				(path "/996c4afa-af57-455f-b0b6-e0f996045a90/0786ce20-9b4f-45a9-9d62-20c78d282fdc"
-					(reference "R13")
+					(reference "R11")
 					(unit 1)
 				)
@@
 				)
 				(path "/996c4afa-af57-455f-b0b6-e0f996045a90/0d35b6da-5370-4b8d-bdb2-6a6466fd726d"
-					(reference "R14")
-					(unit 1)
-				)
+					(reference "R12")
+					(unit 1)
+				)

Commit message: backup
Parts:
- added J6: FW-02-01-G-D-160-160, connector_footprints:FW-02-01-G-D-160-160, symbol CONNECTORS_FW-xx-01-G-D-160-160_DATA_BASE:J_FW-02-01-G-D-160-160
Connections:
- net GNDA: now also J6.2, J6.4
- net I/OP: now also J6.1, J6.3
