File: minimal_ad74416h/Power Supply and Digital Interface.kicad_sch (KiCad schematic)
At the start: 75 parts, among them T1 ZA9644-AED, U3 ADP1031ACPZ-2-R7, U4 ADUM1252AUA+, U5 ADUM1252AUA+, U6 ADUM1252AUA+

Commit message: backup
Parts:
- renumbered C52 to C38, C44 to C39, C48 to C40, C51 to C41, C43 to C42, C47 to C43, C38 to C44, C50 to C45, C42 to C46, C46 to C47, C49 to C48, C41 to C49, C45 to C50, C39 to C51, C40 to C52, R60 to R55, R61 to R56, R62 to R57, R55 to R58, R56 to R59, R57 to R60, R58 to R61, R59 to R62, R105 to R63, R67 to R64, R73 to R65, R63 to R66, R64 to R67, R65 to R68, R78 to R69, R68 to R70, R74 to R71, R75 to R72, R70 to R73, R71 to R74, R76 to R75, R69 to R76, R72 to R77, R66 to R78, TP7 to TP21, TP8 to TP22, TP51 to TP23, TP52 to TP24, TP43 to TP25, TP44 to TP26, TP45 to TP27, TP47 to TP28, TP46 to TP29, TP48 to TP30, TP49 to TP31, TP2 to TP32, TP1 to TP33, TP4 to TP34, TP3 to TP35, TP6 to TP36, TP5 to TP37, U6 to U4, U4 to U5, U5 to U6

Commit message: backup
Parts:
- removed R63: 1 kΩ, resistor_footprints:R_0402_1005Metric, symbol UNITED_RESISTORS_DATA_BASE:R_ERJ-2RKF1001X
- added C1: 1 µF, capacitor_footprints:C_0805_2012Metric, symbol CAPACITORS_GRJ21BC72A_DATA_BASE:C_GRJ21BC72A105KE11L
- added C2, C4: 100 nF, capacitor_footprints:C_0603_1608Metric, symbol CAPACITORS_C1608X7S2A_DATA_BASE:C_C1608X7S2A104K080AB
- added C3: 220 pF, capacitor_footprints:C_0402_1005Metric, symbol CAPACITORS_CGA2B2NP02A_DATA_BASE:C_CGA2B2NP02A221J050BA
- added C5: 1 µF, capacitor_footprints:C_0402_1005Metric, symbol CAPACITORS_C1005X6S1C_DATA_BASE:C_C1005X6S1C105K050BC
- added C6: 10 µF, capacitor_footprints:C_1206_3216Metric, symbol CAPACITORS_CL31B_DATA_BASE:C_CL31B106KBHNNN#
- added L1: 100.0 µH, inductor_footprints:74404054, symbol INDUCTORS_74404054_DATA_BASE:L_74404054101
- added R1: 294 kΩ, resistor_footprints:R_0402_1005Metric, symbol RESISTORS_ERJ-2RKF_DATA_BASE:R_ERJ-2RKF2943X
- added R2: 3.32 MΩ, resistor_footprints:R_0402_1005Metric, symbol RESISTORS_RC0402FR-07_DATA_BASE:R_RC0402FR-073M32L
- added R3: 40.2 kΩ, resistor_footprints:R_0402_1005Metric, symbol RESISTORS_ERJ-2RKF_DATA_BASE:R_ERJ-2RKF4022X
- added R4: 499 kΩ, resistor_footprints:R_0402_1005Metric, symbol RESISTORS_ERJ-2RKF_DATA_BASE:R_ERJ-2RKF4993X
- added R5: 9.76 kΩ, resistor_footprints:R_0402_1005Metric, symbol RESISTORS_ERJ-2RKF_DATA_BASE:R_ERJ-2RKF9761X
- added R6, R69: 1 kΩ, resistor_footprints:R_0402_1005Metric, symbol UNITED_RESISTORS_DATA_BASE:R_ERJ-2RKF1001X
- added U1: MAX17570FATA+, analog_devices_footprints:21-100514_T822C&plus_6C_ADI, symbol UNITED_IC_ADI:U_MAX17570FATA+
- renumbered C33 to C39, C34 to C40, C35 to C41, C36 to C42, C37 to C43, C38 to C44, C39 to C45, C40 to C46, C41 to C47, C42 to C48, C43 to C49, C44 to C50, C45 to C51, C46 to C52, C47 to C53, C48 to C54, C49 to C55, C50 to C56, C51 to C57, C52 to C58, L1 to L2, L2 to L3, R55 to R61, R56 to R62, R57 to R63, R58 to R64, R59 to R65, R60 to R66, R61 to R67, R62 to R68, R64 to R70, R65 to R71, R66 to R72, R67 to R73, R68 to R74, R69 to R75, R70 to R76, R71 to R77, R72 to R78, R73 to R79, R74 to R80, R75 to R81, R76 to R82, R77 to R83, R78 to R84, TP21 to TP26, TP22 to TP27, TP23 to TP28, TP24 to TP29, TP25 to TP30, TP26 to TP31, TP27 to TP32, TP28 to TP33, TP29 to TP34, TP30 to TP35, TP31 to TP36, TP32 to TP37, TP33 to TP38, TP34 to TP39, TP35 to TP40, TP36 to TP41, TP37 to TP42, U3 to U4, U4 to U5, U5 to U6, U6 to U7
Connections:
- net GNDA: now also C1.2, C2.2, C3.2, C4.2, C5.2, C6.2, R1.2, R3.2, R5.2, U1.7 (GND)
- net GPIO_B: now also R69.2
- net VDD_24V: now also C1.1, C2.1, C3.1, R2.1, U1.1 (VIN)
- net VOUT2: now also R69.1
- new net: R5.1, U1.5 (RT/SYNC)
- new net EN: R1.1, R2.2, U1.2 (EN/UVLO)
- new net FB: R3.1, R4.2, U1.4 (VOUT/FB)
- new net LX: L1.1, U1.8 (LX)
- new net MAX17570_VOUT: C4.1, C6.1, L1.2, R4.1
- new net VCC: C5.1, R6.1, U1.3 (VCC)
- new net ~{MAX17570_RESET}: R6.2, U1.6 (~{RESET})

Commit message: backup
Parts:
- L1: footprint inductor_footprints:74404054 -> inductor_footprints:74404032; symbol INDUCTORS_74404054_DATA_BASE:L_74404054101 -> INDUCTORS_74404032_DATA_BASE:L_74404032101; MPN 74404054101 -> 74404032101; Maximum DC Current (A) 0.7 -> 0.3; Maximum DC Resistance (Ω) 0.560 -> 1.900; Series 74404054 -> 74404032; Symbol Name L_74404054101 -> L_74404032101; Trustedparts Search https://www.trustedparts.com/en/search/74404054101 -> https://www.trustedparts.com/en/search/74404032101
- R4: value 499 kΩ -> 604 kΩ; symbol RESISTORS_ERJ-2RKF_DATA_BASE:R_ERJ-2RKF4993X -> RESISTORS_ERJ-2RKF_DATA_BASE:R_ERJ-2RKF6043X; MPN ERJ-2RKF4993X -> ERJ-2RKF6043X; Symbol Name R_ERJ-2RKF4993X -> R_ERJ-2RKF6043X; Trustedparts Search https://www.trustedparts.com/en/search/ERJ-2RKF4993X -> https://www.trustedparts.com/en/search/ERJ-2RKF6043X
Other:
- moved on the sheet: C1, C2, C3, C4, C5, C6, L1, R1, R2, R3, R4, R5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

Commit message: backup
Parts:
- added C44, C57: 100 nF, capacitor_footprints:C_0402_1005Metric, symbol UNITED_CAPACITORS_DATA_BASE:C_GCM155R71H104KE02D
- added C48, C53: 1 nF, capacitor_footprints:C_0402_1005Metric, symbol UNITED_CAPACITORS_DATA_BASE:C_GCM155R71H102KA37D
- added R69, R76, R80, R84: 1 kΩ, resistor_footprints:R_0402_1005Metric, symbol UNITED_RESISTORS_DATA_BASE:R_ERJ-2RKF1001X
- added TP23, TP31, TP32: TestPoint, test_point_footprints:TestPoint_THTPad_Castelated, symbol UNITED_TEST_POINTS:TestPoint_Castelated
- added U5: ADUM1252AUA+, analog_devices_footprints:21-0036_ADI, symbol UNITED_IC_ADI:U_ADUM1252AUA+
- renumbered C2 to C1, C1 to C2, C44 to C45, C45 to C46, C46 to C47, C47 to C49, C48 to C50, C49 to C51, C50 to C52, C51 to C54, C52 to C55, C53 to C56, C54 to C58, C55 to C59, C56 to C60, C57 to C61, C58 to C62, R3 to R5, R4 to R6, R5 to R7, R69 to R70, R70 to R71, R71 to R72, R72 to R73, R73 to R74, R74 to R75, R75 to R77, R76 to R78, R77 to R79, R6 to R8, R78 to R81, R79 to R82, R80 to R83, R81 to R85, R82 to R86, R83 to R87, R84 to R88, TP26 to TP19, TP27 to TP20, TP28 to TP21, TP29 to TP22, TP30 to TP24, TP31 to TP25, TP32 to TP26, TP33 to TP27, TP34 to TP28, TP35 to TP29, TP36 to TP30, TP37 to TP33, TP38 to TP34, TP39 to TP35, TP40 to TP36, TP41 to TP37, TP42 to TP38, U5 to U6, U6 to U7, U7 to U8
Connections:
- net GNDA: now also C44.2, C48.2, U5.5 (GND2)
- net GNDD: now also C53.2, C57.2, U5.4 (GND1)
- net MVDD: now also C53.1, C57.1, R80.1, R84.1, U5.1 (VDD1)
- net PWRGD: now also TP23.1
- net VOUT2: now also C44.1, C48.1, R69.1, R76.1, U5.8 (VDD2)
- net ~{MAX17570_RESET}: now also R69.2, U5.7 (SDA2)
- new net: R84.2, TP32.1, U5.2 (SDA1)
- new net: R80.2, TP31.1, U5.3 (SCL1)
- new net ~{ADC_RDY}: R76.2, U5.6 (SCL2)
Other:
- moved on the sheet: C1, C2, C3, C39, C4, C40, C41, C42, C43, C45, C46, C47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

Commit message: backup
Parts:
- added JP1, JP2: SolderJumper_2_Bridged, solder_jumper_footprints:SolderJumper-2_P1.3mm_Bridged_RoundedPad1.0x1.5mm, symbol UNITED_SOLDER_JUMPERS:SolderJumper_2_Bridged
- added TP25, TP28, TP31, TP34, TP37, TP40, TP43, TP46: TestPoint, test_point_footprints:TestPoint_THTPad_Castelated, symbol UNITED_TEST_POINTS:TestPoint_Castelated
- renumbered JP1 to JP3, JP2 to JP4, JP3 to JP5, JP4 to JP6, R2 to R1, R1 to R2, TP25 to TP26, TP26 to TP27, TP27 to TP29, TP28 to TP30, TP29 to TP32, TP30 to TP33, TP31 to TP35, TP32 to TP36, TP33 to TP38, TP34 to TP39, TP35 to TP41, TP36 to TP42, TP37 to TP44, TP38 to TP45
Connections:
- net GNDD: now also TP25.1, TP28.1, TP31.1, TP34.1, TP37.1, TP40.1, TP43.1, TP46.1
- net MAX17570_VOUT: now also JP1.1
- net VDD_24V: now also JP2.1; no longer C1.1, C2.1, C3.1, R1.1, U1.1 (VIN)
- net ~{MAX17570_RESET_ISO}: now reaches R84.2, TP36.1, U5.2 (SDA1)
- net ~{ADC_RDY_ISO}: now reaches R80.2, TP35.1, U5.3 (SCL1)
- new net 14V5: JP1.2
- new net MAX17570_VIN: C1.1, C2.1, C3.1, JP2.2, R1.1, U1.1 (VIN)

Commit message: backup
Parts:
- removed TP19, TP20, TP21, TP22, TP23, TP24, TP26, TP27, TP29, TP30, TP32, TP33, TP35, TP36, TP38, TP39, TP41, TP42, TP44, TP45: TestPoint, test_point_footprints:TestPoint_THTPad_Castelated, symbol UNITED_TEST_POINTS:TestPoint_Castelated
Connections:
- net MCK renamed SCLK_ISO
- net MGPI2 renamed ~{RESET_ISO}
- net MGPO3 renamed ~{ALERT_ISO}
- net MI renamed SDO_ISO
- net MO renamed SDI_ISO
- net VDD_24V renamed 24V0
- net ~{MSS} renamed ~{SYNC_ISO}
Other:
- moved on the sheet: JP2, R5, R61, R62, R63, R73, R74, R75, TP31, TP34, TP37, TP40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

Commit message: backup
Parts:
- added C63: 220 nF, capacitor_footprints:C_0402_1005Metric, symbol CAPACITORS_KGM05AR71C_DATA_BASE:C_KGM05AR71C224KH
- added R89: 470 kΩ, resistor_footprints:R_0402_1005Metric, symbol RESISTORS_RC0402FR-07_DATA_BASE:R_RC0402FR-07470KL
- added R90: 18.2 kΩ, resistor_footprints:R_0402_1005Metric, symbol RESISTORS_RC0402FR-07_DATA_BASE:R_RC0402FR-0718K2L
- added R91: 2.2 MΩ, resistor_footprints:R_0402_1005Metric, symbol RESISTORS_RC0402FR-07_DATA_BASE:R_RC0402FR-072M2L
- added R92: 1.1 MΩ, resistor_footprints:R_0402_1005Metric, symbol RESISTORS_RC0402FR-7W_DATA_BASE:R_RC0402FR-7W1M1L
- added R93: 1.5 kΩ, resistor_footprints:R_0402_1005Metric, symbol RESISTORS_ERJ-2GEJ_DATA_BASE:R_ERJ-2GEJ152X
- added R94: 150 kΩ, resistor_footprints:R_0402_1005Metric, symbol RESISTORS_ERJ-2GEJ_DATA_BASE:R_ERJ-2GEJ154X
- added R95, R96: 10 kΩ, resistor_footprints:R_0402_1005Metric, symbol UNITED_RESISTORS_DATA_BASE:R_ERJ-2RKF1002X
- added U9: MAX17614ATP+, analog_devices_footprints:21-100172_T2044&plus_4C_MXM_ADI, symbol UNITED_IC_ADI:U_MAX17614ATP+
Connections:
- net 24V0: now also R89.1, R91.1, U9.1 (IN), U9.2 (IN), U9.3 (IN)
- net GNDA: now also C63.2, R90.2, R92.2, R93.2, R94.2, U9.21 (GND), U9.8 (GND)
- net SGPO1: now also U9.9 (EN)
- net VOUT2: now also R95.1, R96.1
- new net: R96.2, U9.11 (~{FLAG})
- new net: R93.1, U9.7 (SETI)
- new net: R94.1, U9.6 (CLMODE)
- new net: C63.1, U9.12 (TSTART)
- new net: R89.2, R90.1, U9.5 (OVLO)
- new net: R95.2, U9.10 (UVOV)
- new net: R91.2, R92.1, U9.4 (UVLO)
- new net DO_VDD: U9.13 (OUT), U9.14 (OUT), U9.15 (OUT)
Other:
- moved on the sheet: C1, C2, C3, C4, C5, C6, JP1, JP2, L1, R1, R2, R5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

Commit message: backup
Parts:
- removed R61, R62, R63, R73, R74, R75: 100 kΩ, resistor_footprints:R_0402_1005Metric, symbol UNITED_RESISTORS_DATA_BASE:R_ERJ-2GEJ104X
