File: minimal_ad74416h/Power Supply and Digital Interface.kicad_sch (KiCad schematic)
At the start: 95 parts, among them T1 ZA9644-AED, U1 MAX17570FATA+, U4 ADP1031ACPZ-2-R7, U5 ADUM1252AUA+, U6 ADUM1252AUA+, U7 ADUM1252AUA+, U8 ADUM1252AUA+, U9 MAX17614ATP+

Commit message: backup
Other:
- moved on the sheet: C1, C2, C3, C4, C5, C6, C63, JP1, JP2, JP4, JP5, L1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

Commit message: backup
Connections:
- net VOUT2: no longer U4.26 (DNC)
Other:
- moved on the sheet: C42, C43, C44, C45, C46, C47, C48, C49, C50, C51, C53, C54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

Commit message: backup
Parts:
- removed R95, R96: 10 kΩ, resistor_footprints:R_0402_1005Metric, symbol UNITED_RESISTORS_DATA_BASE:R_ERJ-2RKF1002X
- added D27, D28: 1.8 V, diode_footprints:LED_RED_0402_1005Metric, symbol DIODES_APHHS1005LSECK-J3-PF_DATA_BASE:D_APHHS1005LSECK-J3-PF
- added R63, R73: 3.3 kΩ, resistor_footprints:R_0402_1005Metric, symbol RESISTORS_ERJ-2RKF_DATA_BASE:R_ERJ-2RKF3301X
- R90: value 18.2 kΩ -> 30 kΩ; symbol RESISTORS_RC0402FR-07_DATA_BASE:R_RC0402FR-0718K2L -> RESISTORS_ERJ-2RKF_DATA_BASE:R_ERJ-2RKF3002X; MPN RC0402FR-0718K2L -> ERJ-2RKF3002X; Manufacturer Yageo -> Panasonic; Series RC0402FR-07 -> ERJ-2RKF; Symbol Name R_RC0402FR-0718K2L -> R_ERJ-2RKF3002X; Temperature Coefficient 200 ppm/°C -> 100 ppm/°C; Trustedparts Search https://www.trustedparts.com/en/search/RC0402FR-0718K2L -> https://www.trustedparts.com/en/search/ERJ-2RKF3002X
- R92: value 1.1 MΩ -> 150 kΩ; symbol RESISTORS_RC0402FR-7W_DATA_BASE:R_RC0402FR-7W1M1L -> RESISTORS_ERJ-2RKF_DATA_BASE:R_ERJ-2RKF1503X; MPN RC0402FR-7W1M1L -> ERJ-2RKF1503X; Manufacturer Yageo -> Panasonic; Series RC0402FR-7W -> ERJ-2RKF; Symbol Name R_RC0402FR-7W1M1L -> R_ERJ-2RKF1503X; Temperature Coefficient 200 ppm/°C -> 100 ppm/°C; Trustedparts Search https://www.trustedparts.com/en/search/RC0402FR-7W1M1L -> https://www.trustedparts.com/en/search/ERJ-2RKF1503X
- R93: value 1.5 kΩ -> 15 kΩ; symbol RESISTORS_ERJ-2GEJ_DATA_BASE:R_ERJ-2GEJ152X -> RESISTORS_ERJ-2RKF_DATA_BASE:R_ERJ-2RKF1502X; MPN ERJ-2GEJ152X -> ERJ-2RKF1502X; Series ERJ-2GEJ -> ERJ-2RKF; Symbol Name R_ERJ-2GEJ152X -> R_ERJ-2RKF1502X; Temperature Coefficient 200 ppm/°C -> 100 ppm/°C; Tolerance 5% -> 1%; Trustedparts Search https://www.trustedparts.com/en/search/ERJ-2GEJ152X -> https://www.trustedparts.com/en/search/ERJ-2RKF1502X
Connections:
- net VOUT2: now also D27.2, D28.2
- net ~{FLAG}: now reaches U9.11 (~{FLAG})
- net ~{FLAG}: now also R63.2
- net SETI: now reaches R93.1, U9.7 (SETI)
- net CLMODE: now reaches R94.1, U9.6 (CLMODE)
- net TSTART: now reaches C63.1, U9.12 (TSTART)
- net RT/SYNC: now reaches R7.1, U1.5 (RT/SYNC)
- net OVLO: now reaches R89.2, R90.1, U9.5 (OVLO)
- net UVOV: now reaches U9.10 (UVOV)
- net UVOV: now also R73.2
- net UVLO: now reaches R91.2, R92.1, U9.4 (UVLO)
- new net: D27.1, R63.1
- new net: D28.1, R73.1
Other:
- moved on the sheet: C1, C2, C3, C39, C4, C40, C41, C42, C43, C44, C45, C46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

Commit message: backup
Parts:
- removed C45, C46, C47, C58, C59, C60: 100 nF, capacitor_footprints:C_0402_1005Metric, symbol UNITED_CAPACITORS_DATA_BASE:C_GCM155R71H104KE02D
- removed C49, C50, C51, C54, C55, C56: 1 nF, capacitor_footprints:C_0402_1005Metric, symbol UNITED_CAPACITORS_DATA_BASE:C_GCM155R71H102KA37D
- removed R70, R71, R72, R77, R78, R79, R81, R82, R83, R85, R86, R87: 1 kΩ, resistor_footprints:R_0402_1005Metric, symbol UNITED_RESISTORS_DATA_BASE:R_ERJ-2RKF1001X
- removed TP37, TP40, TP43, TP46: TestPoint, test_point_footprints:TestPoint_THTPad_Castelated, symbol UNITED_TEST_POINTS:TestPoint_Castelated
- removed U6, U7, U8: ADUM1252AUA+, analog_devices_footprints:21-0036_ADI, symbol UNITED_IC_ADI:U_ADUM1252AUA+
- added C43: 1 nF, capacitor_footprints:C_0402_1005Metric, symbol UNITED_CAPACITORS_DATA_BASE:C_GCM155R71H102KA37D
- added U5: PCA9538ABSHP, nxp_footprints:HVQFN16_SOT758-1_NXP, symbol UNITED_IC_NXP:PCA9538ABSHP
- renumbered C63 to C39, C39 to C40, C40 to C41, C41 to C42, C42 to C44, C43 to C45, C44 to C46, C48 to C47, C52 to C48, C53 to C49, C57 to C50, C61 to C51, C62 to C52, D27 to D22, D28 to D23, D24 to D26, D25 to D27, D26 to D28, R91 to R61, R92 to R62, R90 to R63, R63 to R64, R64 to R65, R89 to R66, R94 to R67, R73 to R68, R65 to R70, R66 to R71, R93 to R72, R67 to R74, R68 to R75, R69 to R76, R76 to R77, R80 to R78, R84 to R79, R88 to R80, U9 to U4, U4 to U6, U5 to U7
Connections:
- net GNDA: now also C43.2, U5.17 (VSS), U5.6 (VSS)
- net GPIO_A: now also U5.9 (P6)
- net GPIO_B: now also U5.10 (P7)
- net GPIO_C: now also U5.2 (P0)
- net GPIO_D: now also U5.7 (P4)
- net GPIO_E: now also U5.5 (P3)
- net GPIO_F: now also U5.4 (P2)
- net VOUT2: now also C43.1, U5.14 (VDD)
- net ~{ADC_RDY}: now also U5.8 (P5); no longer R77.2, U7.6 (SCL2)
- net ~{MAX17570_RESET}: now also U5.3 (P1); no longer R76.2, U7.7 (SDA2)
- net ~{ADC_RDY_ISO} renamed SCL_ISO
- net ~{MAX17570_RESET_ISO} renamed SDA_ISO
- new net A0: U5.15 (A0)
- new net A1: U5.16 (A1)
- new net SCL: R77.2, U5.12 (SCL), U7.6 (SCL2)
- new net SDA: R76.2, U5.13 (SDA), U7.7 (SDA2)
Other:
- moved on the sheet: C46, C47, C49, C50, R76, R77, R78, R79, U7

Commit message: backup
Connections:
- net 5V0: now also C43.1, C46.1, C47.1, D22.2, D23.2, R76.1, R77.1, U5.14 (VDD), U7.8 (VDD2)
- net VOUT2: no longer C43.1, C46.1, C47.1, D22.2, D23.2, R76.1, R77.1, U5.14 (VDD), U7.8 (VDD2)
Changed lines of the file:
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@@
 	)
 	(bus_entry
-		(at 254 200.66)
-		(size -2.54 2.54)
+		(at 254 203.2)
+		(size -2.54 -2.54)
 		(stroke
 			(width 0)
@@
 	)
 	(bus_entry
-		(at 254 203.2)
-		(size -2.54 2.54)
+		(at 254 200.66)
+		(size -2.54 -2.54)
 		(stroke
 			(width 0)
@@
 	)
 	(bus_entry
-		(at 254 208.28)
-		(size -2.54 2.54)
+		(at 254 195.58)
+		(size -2.54 -2.54)
 		(stroke
 			(width 0)
@@
 	)
 	(bus_entry
-		(at 254 193.04)
-		(size -2.54 2.54)
+		(at 254 210.82)
+		(size -2.54 -2.54)
 		(stroke
 			(width 0)
@@
 	)
 	(bus_entry
-		(at 63.5 190.5)
-		(size 2.54 2.54)
+		(at 63.5 198.12)
+		(size 2.54 -2.54)
 		(stroke
 			(width 0)
@@
 	)
 	(bus_entry
-		(at 63.5 193.04)
-		(size 2.54 2.54)
+		(at 63.5 195.58)
+		(size 2.54 -2.54)
 		(stroke
 			(width 0)
@@
 	)
 	(bus_entry
-		(at 254 195.58)
-		(size -2.54 2.54)
+		(at 254 208.28)
+		(size -2.54 -2.54)
 		(stroke
 			(width 0)
@@
 	)
 	(bus_entry
-		(at 254 190.5)
-		(size -2.54 2.54)
+		(at 254 213.36)
+		(size -2.54 -2.54)
 		(stroke
 			(width 0)
@@
 	)
 	(bus_entry
-		(at 254 205.74)
-		(size -2.54 2.54)
+		(at 254 198.12)
+		(size -2.54 -2.54)
 		(stroke
 			(width 0)
@@
 	)
 	(bus_entry
-		(at 254 198.12)
-		(size -2.54 2.54)
+		(at 254 205.74)
+		(size -2.54 -2.54)
 		(stroke
 			(width 0)
@@
 	(bus
 		(pts
-			(xy 63.5 190.5) (xy 63.5 193.04)
-		)
-		(stroke
-			(width 0)
-			(type default)
-		)
-	)
-	(bus
-		(pts
 			(xy 203.2 20.32) (xy 203.2 27.94)
 		)
@@
 		)
 	)
-	(bus
-		(pts
-			(xy 254 172.72) (xy 254 190.5)
-		)
-		(stroke
-			(width 0)
-			(type default)
-		)
-	)
 	(wire
 		(pts
@@
 	(bus
 		(pts
-			(xy 63.5 203.2) (xy 63.5 193.04)
+			(xy 63.5 228.6) (xy 63.5 198.12)
 		)
 		(stroke
@@
 	(bus
 		(pts
+			(xy 254 210.82) (xy 254 213.36)
+		)
+		(stroke
+			(width 0)
+			(type default)
+		)
+	)
+	(bus
+		(pts
 			(xy 160.02 157.48) (xy 160.02 172.72)
 		)
@@
 		)
 	)
+	(bus
+		(pts
+			(xy 254 208.28) (xy 254 210.82)
+		)
+		(stroke
+			(width 0)
+			(type default)
+		)
+	)
 	(wire
 		(pts
@@
 		)
 	)
+	(bus
+		(pts
+			(xy 254 213.36) (xy 254 228.6)
+		)
+		(stroke
+			(width 0)
+			(type default)
+		)
+	)
 	(wire
 		(pts
@@
 	(bus
 		(pts
-			(xy 254 193.04) (xy 254 195.58)
+			(xy 254 172.72) (xy 254 195.58)
 		)
 		(stroke
@@
 		)
 	)
-	(bus
-		(pts
-			(xy 254 190.5) (xy 254 193.04)
-		)
-		(stroke
-			(width 0)
-			(type default)
-		)
-	)
 	(wire
 		(pts
@@
 	(bus
 		(pts
-			(xy 63.5 172.72) (xy 63.5 190.5)
+			(xy 63.5 172.72) (xy 63.5 195.58)
 		)
 		(stroke
@@
 	(bus
 		(pts
-			(xy 254 208.28) (xy 381 208.28)
+			(xy 254 228.6) (xy 381 228.6)
 		)
 		(stroke
@@
 		)
 	)
+	(bus
+		(pts
+			(xy 63.5 198.12) (xy 63.5 195.58)
+		)
+		(stroke
+			(width 0)
+			(type default)
+		)
+	)
 	(wire
 		(pts
@@
 	(bus
 		(pts
-			(xy 50.8 203.2) (xy 63.5 203.2)
+			(xy 50.8 228.6) (xy 63.5 228.6)
 		)
 		(stroke
@@
 		)
 	)
+	(label "5V0"
+		(at 137.16 180.34 180)
+		(effects
+			(font
+				(size 1.27 1.27)
+			)
+			(justify right bottom)
+		)
+	)
 	(label "MAX17570_VOUT"
 		(at 330.2 53.34 0)
@@
 		)
 	)
+	(label "5V0"
+		(at 337.82 96.52 0)
+		(effects
+			(font
+				(size 1.27 1.27)
+			)
+			(justify left bottom)
+		)
+	)
+	(label "5V0"
+		(at 363.22 96.52 0)
+		(effects
+			(font
+				(size 1.27 1.27)
+			)
+			(justify left bottom)
+		)
+	)
 	(label "SDI"
 		(at 142.24 149.86 0)
@@
 		)
 	)
-	(label "VOUT2"
-		(at 337.82 96.52 0)
-		(effects
-			(font
-				(size 1.27 1.27)
-			)
-			(justify left bottom)
-		)
-	)
 	(label "SGPO1"
 		(at 281.94 119.38 180)
@@
 		)
 	)
-	(label "VOUT2"
-		(at 137.16 180.34 180)
-		(effects
-			(font
-				(size 1.27 1.27)
-			)
-			(justify right bottom)
-		)
-	)
 	(label "PWRGD"
 		(at 111.76 137.16 180)
@@
 		)
 	)
-	(label "VOUT2"
-		(at 215.9 182.88 0)
-		(effects
-			(font
-				(size 1.27 1.27)
-			)
-			(justify left bottom)
-		)
-	)
 	(label "~{ALERT}"
 		(at 142.24 144.78 0)
@@
 		)
 	)
-	(label "VOUT2"
-		(at 363.22 96.52 0)
+	(label "~{MAX17570_RESET}"
+		(at 228.6 195.58 0)
 		(effects
 			(font
@@
 		)
 	)
-	(label "~{MAX17570_RESET}"
-		(at 228.6 195.58 0)
+	(label "VOUT3"
+		(at 167.64 91.44 0)
 		(effects
 			(font
@@
 		)
 	)
-	(label "VOUT3"
-		(at 167.64 91.44 0)
+	(label "VOUT2"
+		(at 142.24 124.46 0)
 		(effects
 			(font
@@
 		)
 	)
-	(label "VOUT2"
-		(at 142.24 124.46 0)
+	(label "5V0"
+		(at 215.9 182.88 0)
 		(effects
 			(font
@@
 	(hierarchical_label "{DIGITAL_INTERFACE_INPUT}"
 		(shape bidirectional)
-		(at 50.8 203.2 180)
+		(at 50.8 228.6 180)
 		(effects
 			(font
@@
 	(hierarchical_label "{DIGITAL_INTERFACE}"
 		(shape bidirectional)
-		(at 381 208.28 0)
+		(at 381 228.6 0)
 		(effects
 			(font

Commit message: backup
Parts:
- removed C43: 1 nF, capacitor_footprints:C_0402_1005Metric, symbol UNITED_CAPACITORS_DATA_BASE:C_GCM155R71H102KA37D
- removed U5: PCA9538ABSHP, nxp_footprints:HVQFN16_SOT758-1_NXP, symbol UNITED_IC_NXP:PCA9538ABSHP
- added C53: 1 nF, capacitor_footprints:C_0402_1005Metric, symbol UNITED_CAPACITORS_DATA_BASE:C_GCM155R71H102KA37D
- added U8: PCAL9555AHF_128, nxp_footprints:HWQFN24_SOT994-1_NXP, symbol UNITED_IC_NXP:U_PCAL9555AHF_128
Connections:
- net 5V0: now also C53.1, U8.21 (VDD)
- net A0: now also U8.18 (A0)
- net A1: now also U8.23 (A1)
- net GNDA: now also C53.2, U8.25 (VSS), U8.9 (VSS)
- net GPIO_A: now also U8.12 (P1_2)
- net GPIO_B: now also U8.11 (P1_1)
- net GPIO_C: now also U8.16 (P1_6)
- net GPIO_D: now also U8.17 (P1_7)
- net GPIO_E: now also U8.5 (P0_4)
- net GPIO_F: now also U8.6 (P0_5)
- net SCL: now also U8.19 (SCL)
- net SDA: now also U8.20 (SDA)
- net ~{ADC_RDY}: now also U8.7 (P0_6)
- net MGPI1: no longer names the net of U6.36 (MGPI1)
- net SGPO1: no longer names the net of U4.9 (EN)
- net SGPO1: no longer U6.23 (SGPO1)
- net ~{ALERT_ISO}: no longer names the net of U6.38 (MGPO3)
- net ~{ALERT}: no longer names the net of U6.21 (SGPI3)
- net ~{MAX17570_RESET}: no longer names the net of R8.2, U1.6 (~{RESET})
- net ~{RESET_ISO}: no longer names the net of U6.37 (MGPI2)
- net ~{RESET}: no longer names the net of U6.22 (SGPO2)
- new net A2: U8.24 (A2)
- no-connect marks 0 -> 7

Commit message: backup
Parts:
- removed TP25, TP28, TP31, TP34: TestPoint, test_point_footprints:TestPoint_THTPad_Castelated, symbol UNITED_TEST_POINTS:TestPoint_Castelated
- renumbered C53 to C33, C1 to C34, C2 to C35, C3 to C36, C40 to C37, C41 to C38, C4 to C39, C5 to C40, C42 to C41, C6 to C42, C44 to C43, C45 to C44, C48 to C45, C39 to C46, C46 to C48, C51 to C49, C52 to C50, C49 to C51, C50 to C52, D26 to D24, D22 to D25, D23 to D26, JP3 to JP1, JP4 to JP2, JP5 to JP3, JP1 to JP4, JP2 to JP5, R65 to R57, R1 to R58, R70 to R59, R71 to R60, R2 to R61, R74 to R62, R75 to R63, R5 to R64, R6 to R65, R7 to R66, R8 to R67, R61 to R68, R62 to R69, R63 to R70, R64 to R71, R76 to R72, R66 to R73, R67 to R74, R68 to R75, R77 to R76, R72 to R77, R80 to R78, R78 to R79, R79 to R80, U8 to U3, U1 to U4, U4 to U5
Connections:
- net GPIO_A: now also U3.1 (P0_0); no longer U3.12 (P1_2)
- net GPIO_B: now also U3.2 (P0_1); no longer U3.11 (P1_1)
- net GPIO_C: now also U3.3 (P0_2); no longer U3.16 (P1_6)
- net GPIO_D: now also U3.4 (P0_3); no longer U3.17 (P1_7)
- net GPIO_E: now also U3.6 (P0_5); no longer U3.5 (P0_4)
- net GPIO_F: now also U3.5 (P0_4); no longer U3.6 (P0_5)
- net ~{ADC_RDY}: now also U3.8 (P0_7); no longer U3.7 (P0_6)
- new net ~{ALERT}: U3.7 (P0_6)
- no-connect marks 7 -> 8
Other:
- moved on the sheet: C33, U3

Commit message: backup
Connections:
- net P1_0: now reaches U3.10 (P1_0)
- net P1_1: now reaches U3.11 (P1_1)
- net P1_2: now reaches U3.12 (P1_2)
- net P1_3: now reaches U3.13 (P1_3)
- net P1_4: now reaches U3.14 (P1_4)
- net P1_5: now reaches U3.15 (P1_5)
- net P1_6: now reaches U3.16 (P1_6)
- net P1_7: now reaches U3.17 (P1_7)
