File: minimal_ad74416h/Power Supply and Digital Interface.kicad_sch (KiCad schematic)
At the start: 64 parts, among them T1 ZA9644-AED, U3 PCAL9555AHF_128, U4 MAX17570FATA+, U5 MAX17614ATP+, U6 ADP1031ACPZ-2-R7, U7 ADUM1252AUA+

Commit message: backup
Parts:
- removed C33: 1 nF, capacitor_footprints:C_0402_1005Metric, symbol UNITED_CAPACITORS_DATA_BASE:C_GCM155R71H102KA37D
- removed U3: PCAL9555AHF_128, nxp_footprints:HWQFN24_SOT994-1_NXP, symbol UNITED_IC_NXP:U_PCAL9555AHF_128
Connections:
- no-connect marks 8 -> 7

Commit message: backup
Parts:
- U6: value ADP1031ACPZ-2-R7 -> ADP1031ACPZ-3-R7; symbol UNITED_IC_ADI:U_ADP1031ACPZ-2-R7 -> UNITED_IC_ADI:U_ADP1031ACPZ-3-R7; MPN ADP1031ACPZ-2-R7 -> ADP1031ACPZ-3-R7
Connections:
- net 5V0 renamed 3V3
Changed lines of the file:
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@@
 	)
 	(bus_alias "POWER_BUS"
-		(members "24V0" "5V0" "14V5" "-15V0" "DO_VDD")
+		(members "24V0" "3V3" "14V5" "-15V0" "DO_VDD" "5V0")
 	)
 	(junction
@@
 	)
 	(bus_entry
-		(at 187.96 152.4)
+		(at 160.02 152.4)
 		(size -2.54 -2.54)
 		(stroke
@@
 	)
 	(bus_entry
-		(at 187.96 149.86)
+		(at 160.02 149.86)
 		(size -2.54 -2.54)
 		(stroke
@@
 	)
 	(bus_entry
-		(at 187.96 154.94)
+		(at 160.02 154.94)
 		(size -2.54 -2.54)
 		(stroke
@@
 	)
 	(bus_entry
-		(at 187.96 190.5)
-		(size -2.54 2.54)
+		(at 187.96 198.12)
+		(size -2.54 -2.54)
 		(stroke
 			(width 0)
@@
 	)
 	(bus_entry
-		(at 187.96 157.48)
+		(at 160.02 157.48)
 		(size -2.54 -2.54)
 		(stroke
@@
 	)
 	(bus_entry
-		(at 187.96 193.04)
-		(size -2.54 2.54)
+		(at 187.96 195.58)
+		(size -2.54 -2.54)
 		(stroke
 			(width 0)
@@
 	(bus
 		(pts
-			(xy 187.96 142.24) (xy 187.96 149.86)
+			(xy 187.96 203.2) (xy 187.96 198.12)
 		)
 		(stroke
@@
 	(bus
 		(pts
-			(xy 187.96 149.86) (xy 187.96 152.4)
+			(xy 160.02 149.86) (xy 160.02 152.4)
 		)
 		(stroke
@@
 	(bus
 		(pts
-			(xy 243.84 142.24) (xy 243.84 203.2)
+			(xy 160.02 157.48) (xy 160.02 154.94)
 		)
 		(stroke
@@
 		)
 	)
+	(bus
+		(pts
+			(xy 187.96 172.72) (xy 187.96 195.58)
+		)
+		(stroke
+			(width 0)
+			(type default)
+		)
+	)
 	(wire
 		(pts
@@
 	(wire
 		(pts
-			(xy 139.7 152.4) (xy 185.42 152.4)
+			(xy 139.7 152.4) (xy 157.48 152.4)
 		)
 		(stroke
@@
 	(bus
 		(pts
-			(xy 243.84 142.24) (xy 187.96 142.24)
+			(xy 187.96 203.2) (xy 381 203.2)
 		)
 		(stroke
@@
 	(wire
 		(pts
-			(xy 139.7 149.86) (xy 185.42 149.86)
+			(xy 139.7 149.86) (xy 157.48 149.86)
 		)
 		(stroke
@@
 	(wire
 		(pts
-			(xy 139.7 147.32) (xy 185.42 147.32)
+			(xy 139.7 147.32) (xy 157.48 147.32)
 		)
 		(stroke
@@
 		)
 	)
+	(bus
+		(pts
+			(xy 187.96 172.72) (xy 160.02 172.72)
+		)
+		(stroke
+			(width 0)
+			(type default)
+		)
+	)
 	(wire
 		(pts
@@
 	(bus
 		(pts
-			(xy 187.96 152.4) (xy 187.96 154.94)
+			(xy 160.02 152.4) (xy 160.02 154.94)
 		)
 		(stroke
@@
 	(wire
 		(pts
-			(xy 139.7 154.94) (xy 185.42 154.94)
+			(xy 139.7 154.94) (xy 157.48 154.94)
 		)
 		(stroke
@@
 		)
 	)
-	(bus
-		(pts
-			(xy 187.96 154.94) (xy 187.96 157.48)
-		)
-		(stroke
-			(width 0)
-			(type default)
-		)
-	)
 	(wire
 		(pts
@@
 		)
 	)
-	(bus
-		(pts
-			(xy 187.96 193.04) (xy 187.96 190.5)
-		)
-		(stroke
-			(width 0)
-			(type default)
-		)
-	)
 	(wire
 		(pts
@@
 	(bus
 		(pts
-			(xy 187.96 157.48) (xy 187.96 190.5)
+			(xy 160.02 157.48) (xy 160.02 172.72)
 		)
 		(stroke
@@
 		)
 	)
-	(bus
-		(pts
-			(xy 243.84 203.2) (xy 381 203.2)
-		)
-		(stroke
-			(width 0)
-			(type default)
-		)
-	)
 	(wire
 		(pts
@@
 		)
 	)
+	(bus
+		(pts
+			(xy 187.96 198.12) (xy 187.96 195.58)
+		)
+		(stroke
+			(width 0)
+			(type default)
+		)
+	)
 	(wire
 		(pts
@@
 		)
 	)
-	(label "5V0"
+	(label "3V3"
 		(at 137.16 180.34 180)
 		(effects
@@
 		)
 	)
-	(label "5V0"
+	(label "3V3"
 		(at 337.82 96.52 0)
 		(effects
@@
 		)
 	)
-	(label "5V0"
+	(label "3V3"
 		(at 363.22 96.52 0)
 		(effects
@@
 		)
 	)
-	(label "5V0"
+	(label "3V3"
 		(at 193.04 66.04 0)
 		(effects
@@
 	)
 	(label "{DIGITAL_INTERFACE}"
-		(at 190.5 142.24 0)
+		(at 185.42 172.72 180)
 		(effects
 			(font
 				(size 1.27 1.27)
 			)
-			(justify left bottom)
+			(justify right bottom)
 		)
 	)
@@
 	)
 	(symbol
-		(lib_id "UNITED_IC_ADI:U_ADP1031ACPZ-2-R7")
+		(lib_id "UNITED_IC_ADI:U_ADP1031ACPZ-3-R7")
 		(at 127 111.76 0)
 		(unit 1)
@@
 			)
 		)
-		(property "Value" "ADP1031ACPZ-2-R7"
+		(property "Value" "ADP1031ACPZ-3-R7"
 			(at 127 48.26 0)
 			(effects
@@
 		)
 		(property "Footprint" "analog_devices_footprints:CP-41-1_ADI"
-			(at 137.16 187.96 0)
+			(at 137.16 180.34 0)
 			(effects
 				(font
@@
 		)
 		(property "Datasheet" "https://www.analog.com/media/en/technical-documentation/data-sheets/ADP1031.pdf"
-			(at 137.16 182.88 0)
+			(at 137.16 175.26 0)
 			(effects
 				(font
@@
 			)
 		)
-		(property "Description" "Three-Channel, Isolated Micropower Management Unit with Seven Digital Isolators (VOUT1=Adjustable, VOUT2=5 V, VOUT3=Adjustable)"
-			(at 137.16 185.42 0)
+		(property "Description" "Three-Channel, Isolated Micropower Management Unit with Seven Digital Isolators (VOUT1=Adjustable, VOUT2=3.3 V, VOUT3=Adjustable)"
+			(at 137.16 177.8 0)
 			(effects
 				(font
@@
 			)
 		)
-		(property "MPN" "ADP1031ACPZ-2-R7"
-			(at 137.16 190.5 0)
+		(property "MPN" "ADP1031ACPZ-3-R7"
+			(at 137.16 182.88 0)
 			(effects
 				(font

Commit message: backup
Parts:
- added C54, C55: 10 µF, capacitor_footprints:C_0603_1608Metric, symbol CAPACITORS_C1608X5R1C_DATA_BASE:C_C1608X5R1C106M080AB
- added JP7, JP8: SolderJumper_2_Bridged, solder_jumper_footprints:SolderJumper-2_P1.3mm_Bridged_RoundedPad1.0x1.5mm, symbol UNITED_SOLDER_JUMPERS:SolderJumper_2_Bridged
- added L4: 2.2 µH, inductor_footprints:74479276, symbol UNITED_INDUCTORS_DATA_BASE:L_74479276222
- added R81: 10 kΩ, resistor_footprints:R_0402_1005Metric, symbol UNITED_RESISTORS_DATA_BASE:R_ERJ-2RKF1002X
- added U9: MAX17227JATA+, analog_devices_footprints:21-0168_T822&plus_3C_ADI, symbol UNITED_IC_ADI:U_MAX17227JATA+
Connections:
- net 3V3: now also JP7.1
- net GNDA: now also C54.2, C55.2, R81.2, U9.4 (GND), U9.5 (AGND), U9.9 (GND)
- new net: R81.1, U9.6 (RSEL)
- new net: L4.2, U9.3 (LX)
- new net 5V0: JP8.2
- new net MAX17227_VIN: C55.1, JP7.2, L4.1, U9.7 (IN), U9.8 (EN)
- new net MAX17227_VOUT: C54.1, JP8.1, U9.1 (OUT), U9.2 (OUT)
Other:
- moved on the sheet: C46, D25, D26, R68, R69, R70, R71, R73, R74, R75, R77, U5

Commit message: backup
Parts:
- removed JP1, JP2, JP3, JP4, JP8: SolderJumper_2_Bridged, solder_jumper_footprints:SolderJumper-2_P1.3mm_Bridged_RoundedPad1.0x1.5mm, symbol UNITED_SOLDER_JUMPERS:SolderJumper_2_Bridged
- added C50, C51, C56, C57: 100 nF, capacitor_footprints:C_0402_1005Metric, symbol UNITED_CAPACITORS_DATA_BASE:C_GCM155R71H104KE02D
- added TP50, TP51, TP52, TP53, TP54, TP55, TP56, TP57, TP58, TP59, TP60, TP61, TP62, TP63, TP64, TP65, TP66, TP67, TP68, TP69, TP70, TP71, TP72, TP74, TP75, TP77, TP78, TP79, TP80, TP81, TP82: TestPoint, test_point_footprints:TestPoint_THTPad_Castelated, symbol UNITED_TEST_POINTS:TestPoint_Castelated_v2
- added TP73, TP76: TestPoint, test_point_footprints:TestPoint_THTPad_Castelated, symbol UNITED_TEST_POINTS:TestPoint_Castelated
- added U10, U9: ADUM340E0BRQZ, analog_devices_footprints:RQ-16_ADI, symbol UNITED_IC_ADI:U_ADUM340E0BRQZ
- renumbered C46 to C35, C42 to C36, C39 to C37, C37 to C38, C54 to C39, C38 to C40, C34 to C41, C36 to C42, C41 to C43, C55 to C44, C43 to C45, C44 to C46, C40 to C47, C35 to C48, C45 to C49, C47 to C52, C48 to C53, C49 to C54, C50 to C55, C51 to C58, C52 to C59, D25 to D24, D26 to D25, D24 to D26, JP7 to JP1, JP5 to JP2, JP6 to JP3, L4 to L1, L1 to L2, L2 to L3, L3 to L4, R71 to R59, R75 to R60, R57 to R61, R67 to R62, R66 to R63, R59 to R64, R60 to R65, R74 to R66, R77 to R67, R62 to R68, R81 to R69, R63 to R70, R65 to R71, R68 to R72, R69 to R73, R70 to R74, R73 to R75, R64 to R76, R58 to R77, R61 to R78, R72 to R79, R76 to R80, R78 to R81, R79 to R82, R80 to R83, U7 to U11, U9 to U5, U5 to U6, U4 to U7, U6 to U8
Connections:
- net MAX17227_VOUT is gone; now on net 5V0: C39.1, U5.1 (OUT), U5.2 (OUT)
- net MAX17570_VOUT is gone; now on net 14V5: C36.1, C37.1, L2.2, R71.1
- net VOUT1 is gone; now on net 24V0: C40.1, C49.1, D26.1, R68.1, U8.18 (VOUT1)
- net VOUT2 is gone; now on net 3V3: C43.1, C45.1, C46.1, L3.2, U8.10 (SVDD1), U8.15 (VOUT2), U8.20 (SVDD2)
- net VOUT3 is gone; now on net -15V0: C38.1, R64.1, U8.12 (VOUT3)
- net -15V0: now also TP72.1
- net 14V5: now also TP81.1
- net 24V0: now also TP51.1
- net 3V3: now also C50.1, C51.1, TP66.1, U10.16 (VDD2), U9.16 (VDD2)
- net 5V0: now also TP69.1
- net DO_VDD: now also TP78.1
- net GNDA: now also C50.2, C51.2, TP50.1, TP52.1, TP65.1, TP67.1, TP68.1, TP70.1, TP71.1, TP73.1, TP76.1, TP77.1, TP79.1, TP80.1, TP82.1, U10.15 (GND2), U10.9 (GND2), U9.15 (GND2), U9.9 (GND2)
- net GNDD: now also C56.2, C57.2, U10.2 (GND1), U10.8 (GND1), U9.2 (GND1), U9.8 (GND1)
- net MVDD: now also C56.1, C57.1, U10.1 (VDD1), U9.1 (VDD1)
- net SCL: now also TP74.1
- net SCLK: now also TP56.1
- net SDA: now also TP75.1
- net SDI: now also TP55.1
- net SDO: now also TP54.1
- net ~{SYNC}: now also TP53.1
- new net 1B1: TP64.1, U10.11 (VOD)
- new net 1B1_ISO: U10.6 (VID)
- new net 1B2: TP63.1, U10.12 (VOC)
- new net 1B2_ISO: U10.5 (VIC)
- new net 1B3: TP62.1, U10.13 (VOB)
- new net 1B3_ISO: U10.4 (VIB)
- new net 1B4: TP61.1, U10.14 (VOA)
- new net 1B4_ISO: U10.3 (VIA)
- new net 2B1: TP60.1, U9.11 (VOD)
- new net 2B1_ISO: U9.6 (VID)
- new net 2B2: TP59.1, U9.12 (VOC)
- new net 2B2_ISO: U9.5 (VIC)
- new net 2B3: TP58.1, U9.13 (VOB)
- new net 2B3_ISO: U9.4 (VIB)
- new net 2B4: TP57.1, U9.14 (VOA)
- new net 2B4_ISO: U9.3 (VIA)
- no-connect marks 7 -> 9

Commit message: backup
Parts:
- added J7: FW-33-03-G-D-085-155, connector_footprints:FW-33-03-G-D-085-155, symbol CONNECTORS_FW-xx-03-G-D-085-155_DATA_BASE:J_FW-33-03-G-D-085-155
- added TP100, TP101, TP83, TP84, TP85, TP86, TP87, TP88, TP89, TP90, TP91, TP92, TP93, TP94, TP95, TP96, TP97, TP98, TP99: TestPoint, test_point_footprints:TestPoint_THTPad_Castelated, symbol UNITED_TEST_POINTS:TestPoint_Castelated_v2
Connections:
- net -15V0: now also J7.45, J7.46
- net 14V5: now also J7.63, J7.64
- net 1B1: now also J7.29, J7.30
- net 1B1_ISO: now also TP99.1
- net 1B2: now also J7.27, J7.28
- net 1B2_ISO: now also TP98.1
- net 1B3: now also J7.25, J7.26
- net 1B3_ISO: now also TP97.1
- net 1B4: now also J7.23, J7.24
- net 1B4_ISO: now also TP96.1
- net 24V0: now also J7.3, J7.4
- net 2B1: now also J7.21, J7.22
- net 2B1_ISO: now also TP95.1
- net 2B2: now also J7.19, J7.20
- net 2B2_ISO: now also TP94.1
- net 2B3: now also J7.17, J7.18
- net 2B3_ISO: now also TP93.1
- net 2B4: now also J7.15, J7.16
- net 2B4_ISO: now also TP92.1
- net 3V3: now also J7.33, J7.34
- net 5V0: now also J7.39, J7.40
- net DO_VDD: now also J7.57, J7.58
- net GND: now also TP84.1
- net GNDA: now also J7.1, J7.2, J7.31, J7.32, J7.35, J7.36, J7.37, J7.38, J7.41, J7.42, J7.43, J7.44, J7.47, J7.48, J7.5, J7.53, J7.54, J7.55, J7.56, J7.59, J7.6, J7.60, J7.61, J7.62, J7.65, J7.66
- net GNDD: now also TP86.1
- net MVDD: now also TP85.1
- net PWRGD: now also TP87.1
- net SCL: now also J7.49, J7.50
- net SCLK: now also J7.13, J7.14
- net SCLK_ISO: now also TP89.1
- net SCL_ISO: now also TP100.1
- net SDA: now also J7.51, J7.52
- net SDA_ISO: now also TP101.1
- net SDI: now also J7.11, J7.12
- net SDI_ISO: now also TP88.1
- net SDO: now also J7.10, J7.9
- net SDO_ISO: now also TP90.1
- net VINP: now also TP83.1
- net ~{SYNC_ISO}: now also TP91.1
- net ~{SYNC}: now also J7.7, J7.8
Other:
- moved on the sheet: TP53, TP54, TP55, TP56, TP57, TP58, TP59, TP60, TP61, TP62, TP63, TP64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
