File: minimal_ad74416h/AD74416H.kicad_sch (KiCad schematic)
At the start: 43 parts, among them U1 AD74416HBCPZ-RL7, U2 ADR4525BRZ, U3 PCAL9555AHF_128, U8 U_74CBTLV3253BQ_115

Commit message: backup
Connections:
- net 3V3: now also C1.1, C3.1, C31.1, C32.1, C33.1, R11.1, R12.1, R15.1, R18.1, R21.1, U1.62 (DVCC), U2.2 (VIN), U3.21 (VDD)
- net 5V0: no longer C1.1, C3.1, C31.1, C32.1, C33.1, R11.1, R12.1, R15.1, R18.1, R21.1, U1.62 (DVCC), U2.2 (VIN), U3.21 (VDD)
- net 2B1: now reaches U8.10 (2B1)
- net 2B2: now reaches U8.11 (2B2)
- net 2B3: now reaches U8.12 (2B3)
- net 2B4: now reaches U8.13 (2B4)
- net 1B4: now reaches U8.3 (1B4)
- net 1B3: now reaches U8.4 (1B3)
- net 1B2: now reaches U8.5 (1B2)
- net 1B1: now reaches U8.6 (1B1)

Commit message: backup
Parts:
- added R82, R83: 0 Ω, resistor_footprints:R_0402_1005Metric, symbol UNITED_RESISTORS_DATA_BASE:R_ERJ-2GE0R00X
- R56: footprint resistor_footprints:R_0805_2012Metric -> resistor_footprints:R_0402_1005Metric; symbol UNITED_RESISTORS_DATA_BASE:R_ERJ-6ENF3302V -> RESISTORS_ERJ-2RKF_DATA_BASE:R_ERJ-2RKF3302X; Case Code - in 0805 -> 0402; Case Code - mm 2012 -> 1005; MPN ERJ-6ENF3302V -> ERJ-2RKF3302X; Series ERJ-6ENF -> ERJ-2RKF; Symbol Name R_ERJ-6ENF3302V -> R_ERJ-2RKF3302X; Trustedparts Search https://www.trustedparts.com/en/search/ERJ-6ENF3302V -> https://www.trustedparts.com/en/search/ERJ-2RKF3302X; Voltage Rating 150V -> 50V
Connections:
- net A0 is gone; now on net 3V3: U3.18 (A0)
- net A1 is gone; now on net AD0: U3.23 (A1)
- net A2 is gone; now on net AD1: U3.24 (A2)
- net AD0: now also U8.14 (S0)
- net AD1: now also U8.2 (S1)
- net GNDA: now also R82.2, R83.2
- net at U8.1 (1~{OE}): now also R82.1
- net at U8.15 (2~{OE}): now also R83.1
- no-connect marks 1 -> 3
Other:
- moved on the sheet: C33, C53, S1, U3, U8

Commit message: backup
Parts:
- renumbered C31 to C30, C32 to C31, C30 to C32, C53 to C34, R56 to R54, R83 to R57, R82 to R58, U8 to U3, U3 to U4
Changed lines of the file:
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@@
 		(dnp no)
 		(fields_autoplaced yes)
-		(property "Reference" "R83"
+		(property "Reference" "R57"
 			(at 104.14 222.2499 90)
 			(effects
@@
 			(project "minimal_ad74416h"
 				(path "/996c4afa-af57-455f-b0b6-e0f996045a90/31f46f6a-0bfc-4ecd-bee8-e46e4c2e5b44"
-					(reference "R83")
+					(reference "R57")
 					(unit 1)
 				)
@@
 		(dnp no)
 		(fields_autoplaced yes)
-		(property "Reference" "U3"
+		(property "Reference" "U4"
 			(at 88.5033 124.46 0)
 			(effects
@@
 			(project "minimal_ad74416h"
 				(path "/996c4afa-af57-455f-b0b6-e0f996045a90/31f46f6a-0bfc-4ecd-bee8-e46e4c2e5b44"
-					(reference "U3")
+					(reference "U4")
 					(unit 1)
 				)
@@
 		(dnp no)
 		(fields_autoplaced yes)
-		(property "Reference" "C53"
+		(property "Reference" "C34"
 			(at 80.01 180.34 0)
 			(effects
@@
 			(project "minimal_ad74416h"
 				(path "/996c4afa-af57-455f-b0b6-e0f996045a90/31f46f6a-0bfc-4ecd-bee8-e46e4c2e5b44"
-					(reference "C53")
+					(reference "C34")
 					(unit 1)
 				)
@@
 		(dnp no)
 		(fields_autoplaced yes)
-		(property "Reference" "C30"
+		(property "Reference" "C32"
 			(at 179.07 100.3299 90)
 			(effects
@@
 			(project "minimal_ad74416h"
 				(path "/996c4afa-af57-455f-b0b6-e0f996045a90/31f46f6a-0bfc-4ecd-bee8-e46e4c2e5b44"
-					(reference "C30")
+					(reference "C32")
 					(unit 1)
 				)
@@
 		(on_board yes)
 		(dnp no)
-		(property "Reference" "C32"
+		(property "Reference" "C31"
 			(at 146.05 100.3299 90)
 			(effects
@@
 			(project "minimal_ad74416h"
 				(path "/996c4afa-af57-455f-b0b6-e0f996045a90/31f46f6a-0bfc-4ecd-bee8-e46e4c2e5b44"
-					(reference "C32")
+					(reference "C31")
 					(unit 1)
 				)
@@
 		(dnp no)
 		(fields_autoplaced yes)
-		(property "Reference" "R82"
+		(property "Reference" "R58"
 			(at 104.14 201.9299 90)
 			(effects
@@
 			(project ""
 				(path "/996c4afa-af57-455f-b0b6-e0f996045a90/31f46f6a-0bfc-4ecd-bee8-e46e4c2e5b44"
-					(reference "R82")
+					(reference "R58")
 					(unit 1)
 				)
@@
 		(on_board yes)
 		(dnp no)
-		(property "Reference" "C31"
+		(property "Reference" "C30"
 			(at 130.81 100.3299 90)
 			(effects
@@
 			(project "minimal_ad74416h"
 				(path "/996c4afa-af57-455f-b0b6-e0f996045a90/31f46f6a-0bfc-4ecd-bee8-e46e4c2e5b44"
-					(reference "C31")
+					(reference "C30")
 					(unit 1)
 				)
@@
 		(dnp no)
 		(fields_autoplaced yes)
-		(property "Reference" "R56"
+		(property "Reference" "R54"
 			(at 190.5 109.2199 90)
 			(effects
@@
 			(project "minimal_ad74416h"
 				(path "/996c4afa-af57-455f-b0b6-e0f996045a90/31f46f6a-0bfc-4ecd-bee8-e46e4c2e5b44"
-					(reference "R56")
+					(reference "R54")
 					(unit 1)
 				)
@@
 		(dnp no)
 		(fields_autoplaced yes)
-		(property "Reference" "U8"
+		(property "Reference" "U3"
 			(at 89.4781 187.96 0)
 			(effects
@@
 			(project "minimal_ad74416h"
 				(path "/996c4afa-af57-455f-b0b6-e0f996045a90/31f46f6a-0bfc-4ecd-bee8-e46e4c2e5b44"
-					(reference "U8")
+					(reference "U3")
 					(unit 1)
 				)

Commit message: backup
Parts:
- renumbered R15 to R13, R11 to R14, R12 to R15
Changed lines of the file:
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@@
 		(on_board yes)
 		(dnp no)
-		(property "Reference" "R12"
+		(property "Reference" "R15"
 			(at 193.04 137.1599 90)
 			(effects
@@
 			(project "minimal_ad74416h"
 				(path "/996c4afa-af57-455f-b0b6-e0f996045a90/31f46f6a-0bfc-4ecd-bee8-e46e4c2e5b44"
-					(reference "R12")
+					(reference "R15")
 					(unit 1)
 				)
@@
 		(on_board yes)
 		(dnp no)
-		(property "Reference" "R11"
+		(property "Reference" "R14"
 			(at 203.2 137.1599 90)
 			(effects
@@
 			(project "minimal_ad74416h"
 				(path "/996c4afa-af57-455f-b0b6-e0f996045a90/31f46f6a-0bfc-4ecd-bee8-e46e4c2e5b44"
-					(reference "R11")
+					(reference "R14")
 					(unit 1)
 				)
@@
 		(on_board yes)
 		(dnp no)
-		(property "Reference" "R15"
+		(property "Reference" "R13"
 			(at 142.24 170.1799 90)
 			(effects
@@
 			(project "minimal_ad74416h"
 				(path "/996c4afa-af57-455f-b0b6-e0f996045a90/31f46f6a-0bfc-4ecd-bee8-e46e4c2e5b44"
-					(reference "R15")
+					(reference "R13")
 					(unit 1)
 				)

Commit message: backup
Parts:
- removed S1: 416131160802, dip_switches_footprints:416131160802, symbol UNITED_DIP_SWITCHES_DATA_BASE:S_416131160802
