File: minimal_ad74416h/AD74416H.kicad_sch (KiCad schematic)
At the start: 44 parts, among them U1 AD74416HBCPZ-RL7, U2 ADR4525BRZ, U3 U_74CBTLV3253BQ_115, U4 PCAL9555AHF_128

Commit message: backup
Parts:
- D1, D2, D3, D4, D5, D6: value 1.8 V -> 2.1 V
Changed lines of the file:
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@@
 			)
 		)
-		(property "Value" "1.8 V"
+		(property "Value" "2.1 V"
 			(at 173.99 218.8209 90)
 			(effects
@@
 			)
 		)
-		(property "Description" "Green LED SMD 1.8 V"
+		(property "Description" "Green LED SMD 2.1 V"
 			(at 165.1 215.9 0)
 			(show_name yes)
@@
 			)
 		)
-		(property "Value" "1.8 V"
+		(property "Value" "2.1 V"
 			(at 153.67 218.8209 90)
 			(effects
@@
 			)
 		)
-		(property "Description" "Green LED SMD 1.8 V"
+		(property "Description" "Green LED SMD 2.1 V"
 			(at 144.78 215.9 0)
 			(show_name yes)
@@
 			)
 		)
-		(property "Value" "1.8 V"
+		(property "Value" "2.1 V"
 			(at 133.35 218.8209 90)
 			(effects
@@
 			)
 		)
-		(property "Description" "Green LED SMD 1.8 V"
+		(property "Description" "Green LED SMD 2.1 V"
 			(at 124.46 215.9 0)
 			(show_name yes)
@@
 			)
 		)
-		(property "Value" "1.8 V"
+		(property "Value" "2.1 V"
 			(at 163.83 218.8209 90)
 			(effects
@@
 			)
 		)
-		(property "Description" "Green LED SMD 1.8 V"
+		(property "Description" "Green LED SMD 2.1 V"
 			(at 154.94 215.9 0)
 			(show_name yes)
@@
 			)
 		)
-		(property "Value" "1.8 V"
+		(property "Value" "2.1 V"
 			(at 143.51 218.8209 90)
 			(effects
@@
 			)
 		)
-		(property "Description" "Green LED SMD 1.8 V"
+		(property "Description" "Green LED SMD 2.1 V"
 			(at 134.62 215.9 0)
 			(show_name yes)
@@
 			)
 		)
-		(property "Value" "1.8 V"
+		(property "Value" "2.1 V"
 			(at 184.15 218.8209 90)
 			(effects
@@
 			)
 		)
-		(property "Description" "Green LED SMD 1.8 V"
+		(property "Description" "Green LED SMD 2.1 V"
 			(at 175.26 215.9 0)
 			(show_name yes)
